File: boards/carrier/sheets/uart_bridge.kicad_sch (KiCad schematic)
At the start: 7 parts, among them J1 TYPE-C-31-M-12, U1 CP2102N-A02-GQFN24R

Commit message: place: auto-NC every IC pin not handled by overrides/cluster/power-paths
Default policy reversed: instead of NC'ing only pins explicitly listed
in the refcircuit's no_external_required, NC every IC pin we didn't
explicitly wire. A pin is "handled" if any of: pin_net_overrides /
net_overrides claim it, the cluster pass placed a passive against it,
it's the IC's primary supply pin (power_input_net / power_output_net
standard names), or it's a GND-family pin _attach_ic_ground covers.

Drops pin_not_connected ERC errors from ~45 → ~5 across the carrier
without requiring refcircuits to explicitly catalogue every unused pin
on every IC's symbol. A small visual cost (X mark on otherwise-bare
pins) for a clean baseline; refcircuits can still add explicit pin
handling when they want a nicer rendering.

  Before: 89 errors
  After:  44 errors
Connections:
- no-connect marks 6 -> 21
Changed lines of the file:
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@@
 		(instances
 			(project "USB-UART Bridge (CP2102N → Zynq PS UART0)"
-				(path "/77122c87-1a10-4bfa-83db-8af671214bb9"
+				(path "/da1231e1-8c51-401b-87d3-d07829a91e2d"
 					(reference "U1")
 					(unit 1)
@@
 		(instances
 			(project "USB-UART Bridge (CP2102N → Zynq PS UART0)"
-				(path "/77122c87-1a10-4bfa-83db-8af671214bb9"
+				(path "/da1231e1-8c51-401b-87d3-d07829a91e2d"
 					(reference "C100")
 					(unit 1)
@@
 		(instances
 			(project "USB-UART Bridge (CP2102N → Zynq PS UART0)"
-				(path "/77122c87-1a10-4bfa-83db-8af671214bb9"
+				(path "/da1231e1-8c51-401b-87d3-d07829a91e2d"
 					(reference "#PWR100")
 					(unit 1)
@@
 		(instances
 			(project "USB-UART Bridge (CP2102N → Zynq PS UART0)"
-				(path "/77122c87-1a10-4bfa-83db-8af671214bb9"
+				(path "/da1231e1-8c51-401b-87d3-d07829a91e2d"
 					(reference "C101")
 					(unit 1)
@@
 		(instances
 			(project "USB-UART Bridge (CP2102N → Zynq PS UART0)"
-				(path "/77122c87-1a10-4bfa-83db-8af671214bb9"
+				(path "/da1231e1-8c51-401b-87d3-d07829a91e2d"
 					(reference "#PWR101")
 					(unit 1)
@@
 		(instances
 			(project "USB-UART Bridge (CP2102N → Zynq PS UART0)"
-				(path "/77122c87-1a10-4bfa-83db-8af671214bb9"
+				(path "/da1231e1-8c51-401b-87d3-d07829a91e2d"
 					(reference "C102")
 					(unit 1)
@@
 		(instances
 			(project "USB-UART Bridge (CP2102N → Zynq PS UART0)"
-				(path "/77122c87-1a10-4bfa-83db-8af671214bb9"
+				(path "/da1231e1-8c51-401b-87d3-d07829a91e2d"
 					(reference "#PWR102")
 					(unit 1)
@@
 		(instances
 			(project "USB-UART Bridge (CP2102N → Zynq PS UART0)"
-				(path "/77122c87-1a10-4bfa-83db-8af671214bb9"
+				(path "/da1231e1-8c51-401b-87d3-d07829a91e2d"
 					(reference "#PWR103")
 					(unit 1)
@@
 		(instances
 			(project "USB-UART Bridge (CP2102N → Zynq PS UART0)"
-				(path "/77122c87-1a10-4bfa-83db-8af671214bb9"
+				(path "/da1231e1-8c51-401b-87d3-d07829a91e2d"
 					(reference "#PWR104")
 					(unit 1)
@@
 		(instances
 			(project "USB-UART Bridge (CP2102N → Zynq PS UART0)"
-				(path "/77122c87-1a10-4bfa-83db-8af671214bb9"
+				(path "/da1231e1-8c51-401b-87d3-d07829a91e2d"
 					(reference "J1")
 					(unit 1)
@@
 		(instances
 			(project "USB-UART Bridge (CP2102N → Zynq PS UART0)"
-				(path "/77122c87-1a10-4bfa-83db-8af671214bb9"
+				(path "/da1231e1-8c51-401b-87d3-d07829a91e2d"
 					(reference "C103")
 					(unit 1)
@@
 		(instances
 			(project "USB-UART Bridge (CP2102N → Zynq PS UART0)"
-				(path "/77122c87-1a10-4bfa-83db-8af671214bb9"
+				(path "/da1231e1-8c51-401b-87d3-d07829a91e2d"
 					(reference "#PWR105")
 					(unit 1)
@@
 		(instances
 			(project "USB-UART Bridge (CP2102N → Zynq PS UART0)"
-				(path "/77122c87-1a10-4bfa-83db-8af671214bb9"
+				(path "/da1231e1-8c51-401b-87d3-d07829a91e2d"
 					(reference "C104")
 					(unit 1)
@@
 		(instances
 			(project "USB-UART Bridge (CP2102N → Zynq PS UART0)"
-				(path "/77122c87-1a10-4bfa-83db-8af671214bb9"
+				(path "/da1231e1-8c51-401b-87d3-d07829a91e2d"
 					(reference "#PWR106")
 					(unit 1)
@@
 		(instances
 			(project "USB-UART Bridge (CP2102N → Zynq PS UART0)"
-				(path "/77122c87-1a10-4bfa-83db-8af671214bb9"
+				(path "/da1231e1-8c51-401b-87d3-d07829a91e2d"
 					(reference "#PWR107")
 					(unit 1)
@@
 	)
 	(no_connect
+		(at 142.24 54.61)
+	)
+	(no_connect
 		(at 116.84 54.61)
 	)
@@
 	)
 	(no_connect
+		(at 132.08 31.75)
+	)
+	(no_connect
+		(at 127 31.75)
+	)
+	(no_connect
+		(at 116.84 36.83)
+	)
+	(no_connect
 		(at 119.38 82.55)
 	)
 	(no_connect
+		(at 142.24 74.93)
+	)
+	(no_connect
+		(at 142.24 72.39)
+	)
+	(no_connect
+		(at 142.24 69.85)
+	)
+	(no_connect
+		(at 142.24 67.31)
+	)
+	(no_connect
+		(at 142.24 62.23)
+	)
+	(no_connect
 		(at 139.7 82.55)
 	)
 	(no_connect
+		(at 142.24 59.69)
+	)
+	(no_connect
+		(at 142.24 44.45)
+	)
+	(no_connect
+		(at 142.24 41.91)
+	)
+	(no_connect
 		(at 142.24 39.37)
 	)
@@
 		(at 142.24 36.83)
 	)
+	(no_connect
+		(at 142.24 46.99)
+	)
+	(no_connect
+		(at 142.24 49.53)
+	)
+	(no_connect
+		(at 142.24 52.07)
+	)
 	(sheet_instances
