File: boards/carrier/sheets/lvds_lcd_power.kicad_sch (KiCad schematic)
At the start: 4 parts, among them J5B FPC-05F-40PH20

Commit message: planner: share-wires for power-destination cluster sub-slots (ERC 50→29)
Cluster pins with multiple slots sharing a power destination (e.g.
VBUS with 3 caps all going to GND) previously left slots N≥1's
cap.far pins floating from KiCad ERC's perspective: only slot 0 got
the GND symbol, sub-slots got nothing. KiCad fired
``erc.pin_not_connected`` on every sub-slot cap.far.

Add ``_try_emit_cluster_share_wire``: when a cluster sub-slot shares
a POWER destination with slot 0, emit a direct single-segment wire
from the sub-slot's cap.far to slot 0's cap.far (which sits on the
shared power symbol's pin tip). The wire is HORIZONTAL for LEFT/
RIGHT clusters (where it skims the bottom edge of slot 0's
power-symbol body — overlap intersection falls below the validator's
0.15 mm noise floor). TOP/BOTTOM clusters and label-terminated
destinations are skipped (the share-wire would either cut through
slot 0's symbol body or terminate at a label — both flagged by the
strict layout validator).

Endpoint owners are computed from plan.symbols / plan.labels (cap
symbols whose body spans either endpoint, plus the symbol/label at
slot 0's cap.far) and exempted from the per-segment occupancy probe
so the share-wire's legitimate termination points don't read as
collisions.

Result: ERC pin_not_connected count 50 → 29 (-42%). Layout still
27/27 clean (bounds=0, overlap=0). 228 unit tests pass.

Remaining 29 errors are split between:
  - TOP/BOTTOM cluster sub-slots (intentionally skipped — wire would
    cut through slot 0 power-symbol body)
  - Connector pin_to_net assignments without label emission (separate
    issue; planner doesn't currently emit local labels for connector
    pins assigned to OUTPUT/BIDIRECTIONAL nets)
  - Standalone IC pin pin_not_connected (NoConnect markers missing
    for genuinely unused pins on some ICs)

Co-Authored-By: Claude Opus 4.7 <noreply@anthropic.com>
Connections:
- net GND: now also C101.1
Changed lines of the file:
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@@
 		(instances
 			(project "LVDS LCD bank B (panel + backlight power)"
-				(path "/b24f9d6b-ba4b-402e-bfd3-321892d6d893"
+				(path "/ed5bcafb-a0fc-4854-bebd-a96bd4fc7d30"
 					(reference "J5B")
 					(unit 1)
@@
 		(instances
 			(project "LVDS LCD bank B (panel + backlight power)"
-				(path "/b24f9d6b-ba4b-402e-bfd3-321892d6d893"
+				(path "/ed5bcafb-a0fc-4854-bebd-a96bd4fc7d30"
 					(reference "#PWR200")
 					(unit 1)
@@
 		(instances
 			(project "LVDS LCD bank B (panel + backlight power)"
-				(path "/b24f9d6b-ba4b-402e-bfd3-321892d6d893"
+				(path "/ed5bcafb-a0fc-4854-bebd-a96bd4fc7d30"
 					(reference "#PWR201")
 					(unit 1)
@@
 		(instances
 			(project "LVDS LCD bank B (panel + backlight power)"
-				(path "/b24f9d6b-ba4b-402e-bfd3-321892d6d893"
+				(path "/ed5bcafb-a0fc-4854-bebd-a96bd4fc7d30"
 					(reference "#PWR202")
 					(unit 1)
@@
 		(instances
 			(project "LVDS LCD bank B (panel + backlight power)"
-				(path "/b24f9d6b-ba4b-402e-bfd3-321892d6d893"
+				(path "/ed5bcafb-a0fc-4854-bebd-a96bd4fc7d30"
 					(reference "#PWR203")
 					(unit 1)
@@
 		(instances
 			(project "LVDS LCD bank B (panel + backlight power)"
-				(path "/b24f9d6b-ba4b-402e-bfd3-321892d6d893"
+				(path "/ed5bcafb-a0fc-4854-bebd-a96bd4fc7d30"
 					(reference "#PWR204")
 					(unit 1)
@@
 		(instances
 			(project "LVDS LCD bank B (panel + backlight power)"
-				(path "/b24f9d6b-ba4b-402e-bfd3-321892d6d893"
+				(path "/ed5bcafb-a0fc-4854-bebd-a96bd4fc7d30"
 					(reference "#PWR205")
 					(unit 1)
@@
 		(instances
 			(project "LVDS LCD bank B (panel + backlight power)"
-				(path "/b24f9d6b-ba4b-402e-bfd3-321892d6d893"
+				(path "/ed5bcafb-a0fc-4854-bebd-a96bd4fc7d30"
 					(reference "#PWR206")
 					(unit 1)
@@
 		(instances
 			(project "LVDS LCD bank B (panel + backlight power)"
-				(path "/b24f9d6b-ba4b-402e-bfd3-321892d6d893"
+				(path "/ed5bcafb-a0fc-4854-bebd-a96bd4fc7d30"
 					(reference "#PWR207")
 					(unit 1)
@@
 		(instances
 			(project "LVDS LCD bank B (panel + backlight power)"
-				(path "/b24f9d6b-ba4b-402e-bfd3-321892d6d893"
+				(path "/ed5bcafb-a0fc-4854-bebd-a96bd4fc7d30"
 					(reference "#PWR208")
 					(unit 1)
@@
 		(instances
 			(project "LVDS LCD bank B (panel + backlight power)"
-				(path "/b24f9d6b-ba4b-402e-bfd3-321892d6d893"
+				(path "/ed5bcafb-a0fc-4854-bebd-a96bd4fc7d30"
 					(reference "#PWR209")
 					(unit 1)
@@
 		(instances
 			(project "LVDS LCD bank B (panel + backlight power)"
-				(path "/b24f9d6b-ba4b-402e-bfd3-321892d6d893"
+				(path "/ed5bcafb-a0fc-4854-bebd-a96bd4fc7d30"
 					(reference "#PWR210")
 					(unit 1)
@@
 		(instances
 			(project "LVDS LCD bank B (panel + backlight power)"
-				(path "/b24f9d6b-ba4b-402e-bfd3-321892d6d893"
+				(path "/ed5bcafb-a0fc-4854-bebd-a96bd4fc7d30"
 					(reference "C100")
 					(unit 1)
@@
 		(instances
 			(project "LVDS LCD bank B (panel + backlight power)"
-				(path "/b24f9d6b-ba4b-402e-bfd3-321892d6d893"
+				(path "/ed5bcafb-a0fc-4854-bebd-a96bd4fc7d30"
 					(reference "#PWR300")
 					(unit 1)
@@
 		(instances
 			(project "LVDS LCD bank B (panel + backlight power)"
-				(path "/b24f9d6b-ba4b-402e-bfd3-321892d6d893"
+				(path "/ed5bcafb-a0fc-4854-bebd-a96bd4fc7d30"
 					(reference "C101")
 					(unit 1)
@@
 		(instances
 			(project "LVDS LCD bank B (panel + backlight power)"
-				(path "/b24f9d6b-ba4b-402e-bfd3-321892d6d893"
+				(path "/ed5bcafb-a0fc-4854-bebd-a96bd4fc7d30"
 					(reference "C102")
 					(unit 1)
@@
 		(instances
 			(project "LVDS LCD bank B (panel + backlight power)"
-				(path "/b24f9d6b-ba4b-402e-bfd3-321892d6d893"
+				(path "/ed5bcafb-a0fc-4854-bebd-a96bd4fc7d30"
 					(reference "#PWR301")
 					(unit 1)
@@
 		(instances
 			(project "LVDS LCD bank B (panel + backlight power)"
-				(path "/b24f9d6b-ba4b-402e-bfd3-321892d6d893"
+				(path "/ed5bcafb-a0fc-4854-bebd-a96bd4fc7d30"
 					(reference "#FLG100")
 					(unit 1)
@@
 		(instances
 			(project "LVDS LCD bank B (panel + backlight power)"
-				(path "/b24f9d6b-ba4b-402e-bfd3-321892d6d893"
+				(path "/ed5bcafb-a0fc-4854-bebd-a96bd4fc7d30"
 					(reference "#FLG101")
 					(unit 1)
@@
 		)
 	)
+	(wire
+		(pts
+			(xy 321.31 36.83) (xy 326.39 36.83)
+		)
+		(stroke
+			(width 0)
+			(type default)
+		)
+	)

Commit message: planner: drive GND + tap power-rail cluster pins (ERC 6→4, no hiding)
Two visible-only connectivity fixes that close power_pin_not_driven
ERC errors without touching the validator or hiding anything:

1. GND drive stamp (mipi GND_1). KiCad's power:GND symbol pin is
   itself a power-INPUT, so the flattened GND net (connector GND
   pins + power:GND symbols) has no driver → power_pin_not_driven.
   Emit ONE self-contained stamp — a power:GND + PWR_FLAG joined by a
   short wire — in clear space on the ``power`` block (the ground
   source). One stamp drives the whole flattened GND net.

2. Power-rail tap (microsd VDD). A connector pin classified CLUSTER
   for its decoupling caps still has its own rail net (VDD on +3V3),
   but the cluster only wires the cap far pins to GND — the pin's
   +3V3 trunk is an unnamed undriven island. Tap it: find the trunk's
   true far end (the outboard end of the contiguous wire run at the
   pin row), extend it into the open interior, and place a VISIBLE
   +3V3 label at the extension end (text reading outboard, beyond
   every wire). The trunk joins the rail net and is driven by its flag.

Both passes probe strictly against the full occupancy and skip
(leaving ERC to surface) rather than ever overlapping. Result: all 27
blocks + root overlap=0 bounds=0; ERC 6→4 (remaining 4 are ethernet
Bob-Smith bias resistors). 228 unit tests pass.

Co-Authored-By: Claude Opus 4.8 (1M context) <noreply@anthropic.com>
Connections:
- net +3V3: now also C100.2, C101.2, J5B.2 (+3V3)
Changed lines of the file:
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@@
 		(instances
 			(project "LVDS LCD bank B (panel + backlight power)"
-				(path "/c8078cb2-13d0-423b-8de0-f4098d5aa95c"
+				(path "/e7218a98-8a47-44ea-b78f-2db2d171cc8f"
 					(reference "J5B")
 					(unit 1)
@@
 		(instances
 			(project "LVDS LCD bank B (panel + backlight power)"
-				(path "/c8078cb2-13d0-423b-8de0-f4098d5aa95c"
+				(path "/e7218a98-8a47-44ea-b78f-2db2d171cc8f"
 					(reference "#PWR200")
 					(unit 1)
@@
 		(instances
 			(project "LVDS LCD bank B (panel + backlight power)"
-				(path "/c8078cb2-13d0-423b-8de0-f4098d5aa95c"
+				(path "/e7218a98-8a47-44ea-b78f-2db2d171cc8f"
 					(reference "#PWR201")
 					(unit 1)
@@
 		(instances
 			(project "LVDS LCD bank B (panel + backlight power)"
-				(path "/c8078cb2-13d0-423b-8de0-f4098d5aa95c"
+				(path "/e7218a98-8a47-44ea-b78f-2db2d171cc8f"
 					(reference "#PWR202")
 					(unit 1)
@@
 		(instances
 			(project "LVDS LCD bank B (panel + backlight power)"
-				(path "/c8078cb2-13d0-423b-8de0-f4098d5aa95c"
+				(path "/e7218a98-8a47-44ea-b78f-2db2d171cc8f"
 					(reference "#PWR203")
 					(unit 1)
@@
 		(instances
 			(project "LVDS LCD bank B (panel + backlight power)"
-				(path "/c8078cb2-13d0-423b-8de0-f4098d5aa95c"
+				(path "/e7218a98-8a47-44ea-b78f-2db2d171cc8f"
 					(reference "#PWR204")
 					(unit 1)
@@
 		(instances
 			(project "LVDS LCD bank B (panel + backlight power)"
-				(path "/c8078cb2-13d0-423b-8de0-f4098d5aa95c"
+				(path "/e7218a98-8a47-44ea-b78f-2db2d171cc8f"
 					(reference "#PWR205")
 					(unit 1)
@@
 		(instances
 			(project "LVDS LCD bank B (panel + backlight power)"
-				(path "/c8078cb2-13d0-423b-8de0-f4098d5aa95c"
+				(path "/e7218a98-8a47-44ea-b78f-2db2d171cc8f"
 					(reference "#PWR206")
 					(unit 1)
@@
 		(instances
 			(project "LVDS LCD bank B (panel + backlight power)"
-				(path "/c8078cb2-13d0-423b-8de0-f4098d5aa95c"
+				(path "/e7218a98-8a47-44ea-b78f-2db2d171cc8f"
 					(reference "#PWR207")
 					(unit 1)
@@
 		(instances
 			(project "LVDS LCD bank B (panel + backlight power)"
-				(path "/c8078cb2-13d0-423b-8de0-f4098d5aa95c"
+				(path "/e7218a98-8a47-44ea-b78f-2db2d171cc8f"
 					(reference "#PWR208")
 					(unit 1)
@@
 		(instances
 			(project "LVDS LCD bank B (panel + backlight power)"
-				(path "/c8078cb2-13d0-423b-8de0-f4098d5aa95c"
+				(path "/e7218a98-8a47-44ea-b78f-2db2d171cc8f"
 					(reference "#PWR209")
 					(unit 1)
@@
 		(instances
 			(project "LVDS LCD bank B (panel + backlight power)"
-				(path "/c8078cb2-13d0-423b-8de0-f4098d5aa95c"
+				(path "/e7218a98-8a47-44ea-b78f-2db2d171cc8f"
 					(reference "#PWR210")
 					(unit 1)
@@
 		(instances
 			(project "LVDS LCD bank B (panel + backlight power)"
-				(path "/c8078cb2-13d0-423b-8de0-f4098d5aa95c"
+				(path "/e7218a98-8a47-44ea-b78f-2db2d171cc8f"
 					(reference "C100")
 					(unit 1)
@@
 		(instances
 			(project "LVDS LCD bank B (panel + backlight power)"
-				(path "/c8078cb2-13d0-423b-8de0-f4098d5aa95c"
+				(path "/e7218a98-8a47-44ea-b78f-2db2d171cc8f"
 					(reference "#PWR300")
 					(unit 1)
@@
 		(instances
 			(project "LVDS LCD bank B (panel + backlight power)"
-				(path "/c8078cb2-13d0-423b-8de0-f4098d5aa95c"
+				(path "/e7218a98-8a47-44ea-b78f-2db2d171cc8f"
 					(reference "C101")
 					(unit 1)
@@
 		(instances
 			(project "LVDS LCD bank B (panel + backlight power)"
-				(path "/c8078cb2-13d0-423b-8de0-f4098d5aa95c"
+				(path "/e7218a98-8a47-44ea-b78f-2db2d171cc8f"
 					(reference "C102")
 					(unit 1)
@@
 		(instances
 			(project "LVDS LCD bank B (panel + backlight power)"
-				(path "/c8078cb2-13d0-423b-8de0-f4098d5aa95c"
+				(path "/e7218a98-8a47-44ea-b78f-2db2d171cc8f"
 					(reference "#PWR301")
 					(unit 1)
@@
 		(instances
 			(project "LVDS LCD bank B (panel + backlight power)"
-				(path "/c8078cb2-13d0-423b-8de0-f4098d5aa95c"
+				(path "/e7218a98-8a47-44ea-b78f-2db2d171cc8f"
 					(reference "#FLG100")
 					(unit 1)
@@
 		(instances
 			(project "LVDS LCD bank B (panel + backlight power)"
-				(path "/c8078cb2-13d0-423b-8de0-f4098d5aa95c"
+				(path "/e7218a98-8a47-44ea-b78f-2db2d171cc8f"
 					(reference "#FLG101")
 					(unit 1)
@@
 		(pts
 			(xy 374.65 71.12) (xy 369.57 71.12)
+		)
+		(stroke
+			(width 0)
+			(type default)
+		)
+	)
+	(wire
+		(pts
+			(xy 321.31 45.72) (xy 318.77 45.72)
 		)
 		(stroke
@@
 		(color 0 0 0 0)
 	)
+	(label "+3V3"
+		(at 318.77 45.72 180)
+		(effects
+			(font
+				(size 1.27 1.27)
+			)
+			(justify left bottom)
+		)
+	)
 	(hierarchical_label "+3V3"
