File: boards/_iso/sheets/power.kicad_sch (KiCad schematic)
At the start: 15 parts, among them U1 TLV75733PDBVR, U2 TLV75725PDBVR, U3 TLV75718PDBVR

Commit message: Regenerate carrier (overlap=0 all 27, ERC 134->22) + STAGE_E_STATUS UPDATE 4
Co-Authored-By: Claude Opus 4.8 <noreply@anthropic.com>
Connections:
- net GND: no longer C100.2, C200.2, C300.2, R103.2, R203.2, R303.2, U1.1 (IN), U1.3 (EN), U2.1 (IN), U2.3 (EN), U3.1 (IN), U3.3 (EN)
- new net: R203.2, U2.3 (EN)
- new net: C300.2, U3.1 (IN)
- new net: R303.2, U3.3 (EN)
- new net: C100.2, U1.1 (IN)
- new net: R103.2, U1.3 (EN)
- new net: C200.2, U2.1 (IN)
