File: carrier/schematic/pmod.kicad_sch (KiCad schematic)
At the start: 22 parts, among them J1101 DS1024-2x6R2, J1102 DS1024-2x6R2

Commit message: carrier: pd_input GREEN (power-inlet sheet) — orientation-agnostic cluster elements (TVS in the +VIN bank), fully-labeled PORT islets accepted by the router (cable-flip pads labeled on both sides); board regenerated: 21 sheets, BOARD GATE PASS, goldens blessed (only pd_input new)
Co-Authored-By: Claude Fable 5 <noreply@anthropic.com>
Parts:
- removed C1101, C1103: 100n, Capacitor_SMD:C_0603_1608Metric, symbol Device:C
- removed C1102, C1104: 10u, Capacitor_SMD:C_0805_2012Metric, symbol Device:C
- removed J1101, J1102: DS1024-2x6R2, DS1024-2x6R2:DS1024-2x6R2, symbol DS1024-2x6R2:DS1024-2x6R2
- removed R1101, R1102, R1103, R1104, R1105, R1106, R1107, R1108, R1109, R1110, R1111, R1112, R1113, R1114, R1115, R1116: 200R, Resistor_SMD:R_0603_1608Metric, symbol Device:R
- added C1201, C1203: 100n, Capacitor_SMD:C_0603_1608Metric, symbol Device:C
- added C1202, C1204: 10u, Capacitor_SMD:C_0805_2012Metric, symbol Device:C
- added J1201, J1202: DS1024-2x6R2, DS1024-2x6R2:DS1024-2x6R2, symbol DS1024-2x6R2:DS1024-2x6R2
- added R1201, R1202, R1203, R1204, R1205, R1206, R1207, R1208, R1209, R1210, R1211, R1212, R1213, R1214, R1215, R1216: 200R, Resistor_SMD:R_0603_1608Metric, symbol Device:R
Connections:
- net +3V3_PMOD: now also C1201.1, C1202.1, C1203.1, C1204.1, J1201.11, J1201.12, J1202.11, J1202.12
- net GND: now also C1201.2, C1202.2, C1203.2, C1204.2, J1201.10, J1201.9, J1202.10, J1202.9
- net IO_L10_N_13: now also R1216.1
- net IO_L10_P_13: now also R1215.1
- net IO_L2_N_13: now also R1202.1
- net IO_L2_P_13: now also R1201.1
- net IO_L3_N_13: now also R1204.1
- net IO_L3_P_13: now also R1203.1
- net IO_L4_N_13: now also R1206.1
- net IO_L4_P_13: now also R1205.1
- net IO_L5P_13: now also R1207.1
- net IO_L5_N_13: now also R1208.1
- net IO_L7_N_13: now also R1210.1
- net IO_L7_P_13: now also R1209.1
- net IO_L8_N_13: now also R1212.1
- net IO_L8_P_13: now also R1211.1
- net IO_L9_DQS_N_13: now also R1214.1
- net IO_L9_DQS_P_13: now also R1213.1
- new net: J1201.8, R1208.2
- new net: J1202.5, R1211.2
- new net: J1201.1, R1201.2
- new net: J1201.2, R1205.2
- new net: J1201.3, R1202.2
- new net: J1201.4, R1206.2
- new net: J1201.5, R1203.2
- new net: J1201.6, R1207.2
- new net: J1201.7, R1204.2
- new net: J1202.1, R1209.2
- new net: J1202.2, R1213.2
- new net: J1202.3, R1210.2
- new net: J1202.4, R1214.2
- new net: J1202.6, R1215.2
- new net: J1202.7, R1212.2
- new net: J1202.8, R1216.2

Commit message: carrier: camera GREEN — port-to-port series columns (differential terminations as labeled columns; each net's fan label is the matching islet). Board regenerated: 22 sheets, BOARD GATE PASS, goldens blessed (only camera new). m1_rc PASS.
Co-Authored-By: Claude Fable 5 <noreply@anthropic.com>
Parts:
- removed C1201, C1203: 100n, Capacitor_SMD:C_0603_1608Metric, symbol Device:C
- removed C1202, C1204: 10u, Capacitor_SMD:C_0805_2012Metric, symbol Device:C
- removed J1201, J1202: DS1024-2x6R2, DS1024-2x6R2:DS1024-2x6R2, symbol DS1024-2x6R2:DS1024-2x6R2
- removed R1201, R1202, R1203, R1204, R1205, R1206, R1207, R1208, R1209, R1210, R1211, R1212, R1213, R1214, R1215, R1216: 200R, Resistor_SMD:R_0603_1608Metric, symbol Device:R
- added C1301, C1303: 100n, Capacitor_SMD:C_0603_1608Metric, symbol Device:C
- added C1302, C1304: 10u, Capacitor_SMD:C_0805_2012Metric, symbol Device:C
- added J1301, J1302: DS1024-2x6R2, DS1024-2x6R2:DS1024-2x6R2, symbol DS1024-2x6R2:DS1024-2x6R2
- added R1301, R1302, R1303, R1304, R1305, R1306, R1307, R1308, R1309, R1310, R1311, R1312, R1313, R1314, R1315, R1316: 200R, Resistor_SMD:R_0603_1608Metric, symbol Device:R
Connections:
- net +3V3_PMOD: now also C1301.1, C1302.1, C1303.1, C1304.1, J1301.11, J1301.12, J1302.11, J1302.12
- net GND: now also C1301.2, C1302.2, C1303.2, C1304.2, J1301.10, J1301.9, J1302.10, J1302.9
- net IO_L10_N_13: now also R1316.1
- net IO_L10_P_13: now also R1315.1
- net IO_L2_N_13: now also R1302.1
- net IO_L2_P_13: now also R1301.1
- net IO_L3_N_13: now also R1304.1
- net IO_L3_P_13: now also R1303.1
- net IO_L4_N_13: now also R1306.1
- net IO_L4_P_13: now also R1305.1
- net IO_L5P_13: now also R1307.1
- net IO_L5_N_13: now also R1308.1
- net IO_L7_N_13: now also R1310.1
- net IO_L7_P_13: now also R1309.1
- net IO_L8_N_13: now also R1312.1
- net IO_L8_P_13: now also R1311.1
- net IO_L9_DQS_N_13: now also R1314.1
- net IO_L9_DQS_P_13: now also R1313.1
- new net: J1301.3, R1302.2
- new net: J1302.1, R1309.2
- new net: J1302.8, R1316.2
- new net: J1301.1, R1301.2
- new net: J1301.2, R1305.2
- new net: J1301.4, R1306.2
- new net: J1301.5, R1303.2
- new net: J1301.6, R1307.2
- new net: J1301.7, R1304.2
- new net: J1301.8, R1308.2
- new net: J1302.2, R1313.2
- new net: J1302.4, R1314.2
- new net: J1302.3, R1310.2
- new net: J1302.5, R1311.2
- new net: J1302.6, R1315.2
- new net: J1302.7, R1312.2

Commit message: carrier: fmc GREEN — board regenerated: 23 sheets all-gates PASS, LINK PASS, BOARD GATE PASS; goldens blessed (fmc NEW; inspected drift: power_mon shunt rank now ONE row -> sheet demoted A3->A4, bringup_rails recenter + attach-column nudge, bringup_en_modules wider cap farm — all eyeballed clean). m1_rc PASS.
Co-Authored-By: Claude Fable 5 <noreply@anthropic.com>
Parts:
- removed C1301, C1303: 100n, Capacitor_SMD:C_0603_1608Metric, symbol Device:C
- removed C1302, C1304: 10u, Capacitor_SMD:C_0805_2012Metric, symbol Device:C
- removed J1301, J1302: DS1024-2x6R2, DS1024-2x6R2:DS1024-2x6R2, symbol DS1024-2x6R2:DS1024-2x6R2
- removed R1301, R1302, R1303, R1304, R1305, R1306, R1307, R1308, R1309, R1310, R1311, R1312, R1313, R1314, R1315, R1316: 200R, Resistor_SMD:R_0603_1608Metric, symbol Device:R
- added C1401, C1403: 100n, Capacitor_SMD:C_0603_1608Metric, symbol Device:C
- added C1402, C1404: 10u, Capacitor_SMD:C_0805_2012Metric, symbol Device:C
- added J1401, J1402: DS1024-2x6R2, DS1024-2x6R2:DS1024-2x6R2, symbol DS1024-2x6R2:DS1024-2x6R2
- added R1401, R1402, R1403, R1404, R1405, R1406, R1407, R1408, R1409, R1410, R1411, R1412, R1413, R1414, R1415, R1416: 200R, Resistor_SMD:R_0603_1608Metric, symbol Device:R
Connections:
- net +3V3_PMOD: now also C1401.1, C1402.1, C1403.1, C1404.1, J1401.11, J1401.12, J1402.11, J1402.12
- net GND: now also C1401.2, C1402.2, C1403.2, C1404.2, J1401.10, J1401.9, J1402.10, J1402.9
- net IO_L10_N_13: now also R1416.1
- net IO_L10_P_13: now also R1415.1
- net IO_L2_N_13: now also R1402.1
- net IO_L2_P_13: now also R1401.1
- net IO_L3_N_13: now also R1404.1
- net IO_L3_P_13: now also R1403.1
- net IO_L4_N_13: now also R1406.1
- net IO_L4_P_13: now also R1405.1
- net IO_L5P_13: now also R1407.1
- net IO_L5_N_13: now also R1408.1
- net IO_L7_N_13: now also R1410.1
- net IO_L7_P_13: now also R1409.1
- net IO_L8_N_13: now also R1412.1
- net IO_L8_P_13: now also R1411.1
- net IO_L9_DQS_N_13: now also R1414.1
- net IO_L9_DQS_P_13: now also R1413.1
- new net: J1402.1, R1409.2
- new net: J1402.6, R1415.2
- new net: J1402.4, R1414.2
- new net: J1402.3, R1410.2
- new net: J1402.5, R1411.2
- new net: J1401.1, R1401.2
- new net: J1401.2, R1405.2
- new net: J1401.3, R1402.2
- new net: J1401.4, R1406.2
- new net: J1401.5, R1403.2
- new net: J1401.6, R1407.2
- new net: J1401.7, R1404.2
- new net: J1401.8, R1408.2
- new net: J1402.2, R1413.2
- new net: J1402.7, R1412.2
- new net: J1402.8, R1416.2

Commit message: audit-fix(engine): harvest F1-F7,F9 — gate hardening + leak + guards
F1 selftest now exercises the VISUAL gate against geometry mutants (wire-cross
+ text-over-wire) — proven to bite (was never run on a mutant before).
F2 visual_gate catches different-net wire T-touch / butt-join shorts.
F3 netlist_gate no longer leaks tmp .net files (was 2671 stale).
F4 board uniquify guards the stride (widened 100->1000) against ref collision.
F5 hier-mode sheets now re-run through the per-sheet netlist gate.
F6 dead clause dropped; F7 stale zynq_eda docstring fixed; F9 eager inline-pin
validation. Source copied verbatim from the audit-fix worktree (6 files, proven
untouched on origin since its base); board regenerated fresh. All gates green,
selftest geo-mutants killed by the visual gate, goldens 23/23, m1_rc PASS.

Co-Authored-By: Claude Fable 5 <noreply@anthropic.com>
Parts:
- renumbered C1401 to C14001, C1402 to C14002, C1403 to C14003, C1404 to C14004, J1401 to J14001, J1402 to J14002, R1401 to R14001, R1402 to R14002, R1403 to R14003, R1404 to R14004, R1405 to R14005, R1406 to R14006, R1407 to R14007, R1408 to R14008, R1409 to R14009, R1410 to R14010, R1411 to R14011, R1412 to R14012, R1413 to R14013, R1414 to R14014, R1415 to R14015, R1416 to R14016

Commit message: DEF-6: netlist the HDMI-RX TMDS sink termination (new hdmi_rx_term sheet)
The HDMI-RX sink REQUIRES 8x 49.9 ohm/pair-to-AVCC source termination (a
7-series HR bank does not self-terminate TMDS_33) — without it HDMI RX simply
does not work. It had been carried for rounds as a docstring-only MANDATORY
layout note because the resistors belong at the FPGA-bank (receiver) end and
the connector-sheet placer could not anchor an off-sheet AVCC trunk. DEF-6
promotes it to a real, netlisted, gate-checked, BOM-counted network on its own
sheet hdmi_rx_term.py: 8x 49.9R (C114625) from HDMI_RX_{D2,D1,D0,CLK}_{P,N} to
AVCC = +3V3 (bank-33 VCCO IS +3V3, the correct TMDS_33 termination voltage).

LINK PASS (the 3-way TMDS merge with hdmi_rx + som_j2), powertree accepts the
~64 mA termination load, render clean (LAW 1), board PASS 26 sheets,
deterministic, selftest 44/44, m1 PASS.

The 100n/1u AVCC bypass is a documented layout note (not netlisted): the
placer has no pattern for a rail-to-rail cap with no host part on an IC-less
sheet (a tracked placer-robustness follow-up). Inserting the sheet
alphabetically re-stamps the per-sheet reference uniquification of the 15
downstream sheets (U11001->U12001 etc.) — deterministic, a known consequence
of the position-based hierarchy numbering.

Co-Authored-By: Claude Opus 4.8 <noreply@anthropic.com>
Parts:
- renumbered C14001 to C15001, C14002 to C15002, C14003 to C15003, C14004 to C15004, J14001 to J15001, J14002 to J15002, R14001 to R15001, R14002 to R15002, R14003 to R15003, R14004 to R15004, R14005 to R15005, R14006 to R15006, R14007 to R15007, R14008 to R15008, R14009 to R15009, R14010 to R15010, R14011 to R15011, R14012 to R15012, R14013 to R15013, R14014 to R15014, R14015 to R15015, R14016 to R15016
