File: carrier/schematic/debug_boot.kicad_sch (KiCad schematic)
At the start: 10 parts, among them J501 878311420, J502 HX_JN1.27-2x5, SW501 DIP-4, SW502 RESET

Commit message: carrier: camera GREEN — port-to-port series columns (differential terminations as labeled columns; each net's fan label is the matching islet). Board regenerated: 22 sheets, BOARD GATE PASS, goldens blessed (only camera new). m1_rc PASS.
Co-Authored-By: Claude Fable 5 <noreply@anthropic.com>
Parts:
- removed J501: 878311420, 878311420:878311420, symbol 878311420:878311420
- removed J502: HX_JN1.27-2x5, HX_JN1.27-2x5_TP_H4.9:HX_JN1.27-2x5_TP_H4.9, symbol HX_JN1.27-2x5_TP_H4.9:HX_JN1.27-2x5_TP_H4.9
- removed R501, R502: 4k7, Resistor_SMD:R_0603_1608Metric, symbol Device:R
- removed R503: 100R, Resistor_SMD:R_0603_1608Metric, symbol Device:R
- removed R504, R505, R506: 10k, Resistor_SMD:R_0603_1608Metric, symbol Device:R
- removed SW501: DIP-4, DSHP04TSGER:DSHP04TSGER, symbol DSHP04TSGER:DSHP04TSGER
- removed SW502: RESET, TS-1187A-B-A-B:TS-1187A-B-A-B, symbol TS-1187A-B-A-B:TS-1187A-B-A-B
- added J601: 878311420, 878311420:878311420, symbol 878311420:878311420
- added J602: HX_JN1.27-2x5, HX_JN1.27-2x5_TP_H4.9:HX_JN1.27-2x5_TP_H4.9, symbol HX_JN1.27-2x5_TP_H4.9:HX_JN1.27-2x5_TP_H4.9
- added R601, R602: 4k7, Resistor_SMD:R_0603_1608Metric, symbol Device:R
- added R603: 100R, Resistor_SMD:R_0603_1608Metric, symbol Device:R
- added R604, R605, R606: 10k, Resistor_SMD:R_0603_1608Metric, symbol Device:R
- added SW601: DIP-4, DSHP04TSGER:DSHP04TSGER, symbol DSHP04TSGER:DSHP04TSGER
- added SW602: RESET, TS-1187A-B-A-B:TS-1187A-B-A-B, symbol TS-1187A-B-A-B:TS-1187A-B-A-B
Connections:
- net +3V3: now also J601.2, R601.1, R602.1
- net +3V3_SC: now also J602.1, R603.1, R604.1, R605.1, R606.1
- net GND: now also J601.1, J601.11, J601.13, J601.3, J601.5, J601.7, J601.9, J602.3, J602.5, J602.9, SW601.5, SW601.6, SW601.7, SW602.3 (C), SW602.4 (D)
- net STM32_BOOT0: now also SW601.1
- net STM32_GPIO5: now also J602.4
- net STM32_GPIO6: now also J602.2
- net STM32_GPIO7: now also R604.2, SW601.2
- net STM32_GPIO8: now also R605.2, SW601.3
- net STM32_NRST: now also J602.10, SW602.1 (A), SW602.2 (B)
- net ZYNQ_TCK: now also J601.6
- net ZYNQ_TDI: now also J601.10, R602.2
- net ZYNQ_TDO: now also J601.8
- net ZYNQ_TMS: now also J601.4, R601.2
- new net: R606.2, SW601.4
- new net: R603.2, SW601.8
Changed lines of the file:
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@@
 		(property
 			"Reference"
-			"SW501"
+			"SW601"
 			(at 90.17 73.025 0)
 			(effects
@@
 				"Zynq_Carrier"
 				(path
-					"/5dc66003-6dff-4b2a-9031-15ab79ee8b4b/67653f37-b9c9-4d64-b6e1-f65d439758bf"
-					(reference "SW501")
+					"/f0293046-ef42-43e4-84be-baa87b4d212c/fe69304b-7994-4faa-a0a5-98ff64846006"
+					(reference "SW601")
 					(unit 1)
 				)
@@
 		(property
 			"Reference"
-			"R505"
+			"R605"
 			(at 54.712 72.39 0)
 			(effects
@@
 				"Zynq_Carrier"
 				(path
-					"/5dc66003-6dff-4b2a-9031-15ab79ee8b4b/67653f37-b9c9-4d64-b6e1-f65d439758bf"
-					(reference "R505")
+					"/f0293046-ef42-43e4-84be-baa87b4d212c/fe69304b-7994-4faa-a0a5-98ff64846006"
+					(reference "R605")
 					(unit 1)
 				)
@@
 		(property
 			"Reference"
-			"R504"
+			"R604"
 			(at 105.513 69.85 0)
 			(effects
@@
 				"Zynq_Carrier"
 				(path
-					"/5dc66003-6dff-4b2a-9031-15ab79ee8b4b/67653f37-b9c9-4d64-b6e1-f65d439758bf"
-					(reference "R504")
+					"/f0293046-ef42-43e4-84be-baa87b4d212c/fe69304b-7994-4faa-a0a5-98ff64846006"
+					(reference "R604")
 					(unit 1)
 				)
@@
 		(property
 			"Reference"
-			"R506"
+			"R606"
 			(at 130.912 69.85 0)
 			(effects
@@
 				"Zynq_Carrier"
 				(path
-					"/5dc66003-6dff-4b2a-9031-15ab79ee8b4b/67653f37-b9c9-4d64-b6e1-f65d439758bf"
-					(reference "R506")
+					"/f0293046-ef42-43e4-84be-baa87b4d212c/fe69304b-7994-4faa-a0a5-98ff64846006"
+					(reference "R606")
 					(unit 1)
 				)
@@
 		(property
 			"Reference"
-			"R503"
+			"R603"
 			(at 141.072 69.85 0)
 			(effects
@@
 				"Zynq_Carrier"
 				(path
-					"/5dc66003-6dff-4b2a-9031-15ab79ee8b4b/67653f37-b9c9-4d64-b6e1-f65d439758bf"
-					(reference "R503")
+					"/f0293046-ef42-43e4-84be-baa87b4d212c/fe69304b-7994-4faa-a0a5-98ff64846006"
+					(reference "R603")
 					(unit 1)
 				)
@@
 		(property
 			"Reference"
-			"SW502"
+			"SW602"
 			(at 177.8 75.565 0)
 			(effects
@@
 				"Zynq_Carrier"
 				(path
-					"/5dc66003-6dff-4b2a-9031-15ab79ee8b4b/67653f37-b9c9-4d64-b6e1-f65d439758bf"
-					(reference "SW502")
+					"/f0293046-ef42-43e4-84be-baa87b4d212c/fe69304b-7994-4faa-a0a5-98ff64846006"
+					(reference "SW602")
 					(unit 1)
 				)
@@
 		(property
 			"Reference"
-			"J502"
+			"J602"
 			(at 248.92 65.405 0)
 			(effects
@@
 				"Zynq_Carrier"
 				(path
-					"/5dc66003-6dff-4b2a-9031-15ab79ee8b4b/67653f37-b9c9-4d64-b6e1-f65d439758bf"
-					(reference "J502")
+					"/f0293046-ef42-43e4-84be-baa87b4d212c/fe69304b-7994-4faa-a0a5-98ff64846006"
+					(reference "J602")
 					(unit 1)
 				)
@@
 		(property
 			"Reference"
-			"J501"
+			"J601"
 			(at 90.17 95.885 0)
 			(effects
@@
 				"Zynq_Carrier"
 				(path
-					"/5dc66003-6dff-4b2a-9031-15ab79ee8b4b/67653f37-b9c9-4d64-b6e1-f65d439758bf"
-					(reference "J501")
+					"/f0293046-ef42-43e4-84be-baa87b4d212c/fe69304b-7994-4faa-a0a5-98ff64846006"
+					(reference "J601")
 					(unit 1)
 				)
@@
 		(property
 			"Reference"
-			"R501"
+			"R601"
 			(at 108.053 118.11 0)
 			(effects
@@
 				"Zynq_Carrier"
 				(path
-					"/5dc66003-6dff-4b2a-9031-15ab79ee8b4b/67653f37-b9c9-4d64-b6e1-f65d439758bf"
-					(reference "R501")
+					"/f0293046-ef42-43e4-84be-baa87b4d212c/fe69304b-7994-4faa-a0a5-98ff64846006"
+					(reference "R601")
 					(unit 1)
 				)
@@
 		(property
 			"Reference"
-			"R502"
+			"R602"
 			(at 161.393 118.11 0)
 			(effects
@@
 				"Zynq_Carrier"
 				(path
-					"/5dc66003-6dff-4b2a-9031-15ab79ee8b4b/67653f37-b9c9-4d64-b6e1-f65d439758bf"
-					(reference "R502")
+					"/f0293046-ef42-43e4-84be-baa87b4d212c/fe69304b-7994-4faa-a0a5-98ff64846006"
+					(reference "R602")
 					(unit 1)
 				)
@@
 		(property
 			"Reference"
-			"#PWR501"
+			"#PWR601"
 			(at 81.28 82.55 0)
 			(effects
@@
 				"Zynq_Carrier"
 				(path
-					"/5dc66003-6dff-4b2a-9031-15ab79ee8b4b/67653f37-b9c9-4d64-b6e1-f65d439758bf"
-					(reference "#PWR501")
+					"/f0293046-ef42-43e4-84be-baa87b4d212c/fe69304b-7994-4faa-a0a5-98ff64846006"
+					(reference "#PWR601")
 					(unit 1)
 				)
@@
 		(property
 			"Reference"
-			"#PWR502"
+			"#PWR602"
 			(at 52.07 67.31 0)
 			(effects
@@
 				"Zynq_Carrier"
 				(path
-					"/5dc66003-6dff-4b2a-9031-15ab79ee8b4b/67653f37-b9c9-4d64-b6e1-f65d439758bf"
-					(reference "#PWR502")
+					"/f0293046-ef42-43e4-84be-baa87b4d212c/fe69304b-7994-4faa-a0a5-98ff64846006"
+					(reference "#PWR602")
 					(unit 1)
 				)
@@
 		(property
 			"Reference"
-			"#PWR503"
+			"#PWR603"
 			(at 99.06 80.01 0)
 			(effects
@@
 				"Zynq_Carrier"
 				(path
-					"/5dc66003-6dff-4b2a-9031-15ab79ee8b4b/67653f37-b9c9-4d64-b6e1-f65d439758bf"
-					(reference "#PWR503")
+					"/f0293046-ef42-43e4-84be-baa87b4d212c/fe69304b-7994-4faa-a0a5-98ff64846006"
+					(reference "#PWR603")
 					(unit 1)
 				)
@@
 		(property
 			"Reference"
-			"#PWR504"
+			"#PWR604"
 			(at 102.87 64.77 0)
 			(effects
@@
 				"Zynq_Carrier"
 				(path
-					"/5dc66003-6dff-4b2a-9031-15ab79ee8b4b/67653f37-b9c9-4d64-b6e1-f65d439758bf"
-					(reference "#PWR504")
+					"/f0293046-ef42-43e4-84be-baa87b4d212c/fe69304b-7994-4faa-a0a5-98ff64846006"
+					(reference "#PWR604")
 					(unit 1)
 				)
@@
 		(property
 			"Reference"
-			"#PWR505"
+			"#PWR605"
 			(at 128.27 64.77 0)
 			(effects
@@
 				"Zynq_Carrier"
 				(path
-					"/5dc66003-6dff-4b2a-9031-15ab79ee8b4b/67653f37-b9c9-4d64-b6e1-f65d439758bf"
-					(reference "#PWR505")
+					"/f0293046-ef42-43e4-84be-baa87b4d212c/fe69304b-7994-4faa-a0a5-98ff64846006"
+					(reference "#PWR605")
 					(unit 1)
 				)
@@
 		(property
 			"Reference"
-			"#PWR506"
+			"#PWR606"
 			(at 138.43 64.77 0)
 			(effects
@@
 				"Zynq_Carrier"
 				(path
-					"/5dc66003-6dff-4b2a-9031-15ab79ee8b4b/67653f37-b9c9-4d64-b6e1-f65d439758bf"
-					(reference "#PWR506")
+					"/f0293046-ef42-43e4-84be-baa87b4d212c/fe69304b-7994-4faa-a0a5-98ff64846006"
+					(reference "#PWR606")
 					(unit 1)
 				)
@@
 		(property
 			"Reference"
-			"#PWR507"
+			"#PWR607"
 			(at 166.37 80.01 0)
 			(effects
@@
 				"Zynq_Carrier"
 				(path
-					"/5dc66003-6dff-4b2a-9031-15ab79ee8b4b/67653f37-b9c9-4d64-b6e1-f65d439758bf"
-					(reference "#PWR507")
+					"/f0293046-ef42-43e4-84be-baa87b4d212c/fe69304b-7994-4faa-a0a5-98ff64846006"
+					(reference "#PWR607")
 					(unit 1)
 				)
@@
 		(property
 			"Reference"
-			"#PWR508"
+			"#PWR608"
 			(at 257.81 62.23 0)
 			(effects
@@
 				"Zynq_Carrier"
 				(path
-					"/5dc66003-6dff-4b2a-9031-15ab79ee8b4b/67653f37-b9c9-4d64-b6e1-f65d439758bf"
-					(reference "#PWR508")
+					"/f0293046-ef42-43e4-84be-baa87b4d212c/fe69304b-7994-4faa-a0a5-98ff64846006"
+					(reference "#PWR608")
 					(unit 1)
 				)
@@
 		(property
 			"Reference"
-			"#PWR509"
+			"#PWR609"
 			(at 257.81 74.93 0)
 			(effects
@@
 				"Zynq_Carrier"
 				(path
-					"/5dc66003-6dff-4b2a-9031-15ab79ee8b4b/67653f37-b9c9-4d64-b6e1-f65d439758bf"
-					(reference "#PWR509")
+					"/f0293046-ef42-43e4-84be-baa87b4d212c/fe69304b-7994-4faa-a0a5-98ff64846006"
+					(reference "#PWR609")
 					(unit 1)
 				)
@@
 		(property
 			"Reference"
-			"#PWR510"
+			"#PWR610"
 			(at 260.35 82.55 0)
 			(effects
@@
 				"Zynq_Carrier"
 				(path
-					"/5dc66003-6dff-4b2a-9031-15ab79ee8b4b/67653f37-b9c9-4d64-b6e1-f65d439758bf"
-					(reference "#PWR510")
+					"/f0293046-ef42-43e4-84be-baa87b4d212c/fe69304b-7994-4faa-a0a5-98ff64846006"
+					(reference "#PWR610")
 					(unit 1)
 				)
@@
 		(property
 			"Reference"
-			"#PWR511"
+			"#PWR611"
 			(at 81.28 113.03 0)
 			(effects
@@
 				"Zynq_Carrier"
 				(path
-					"/5dc66003-6dff-4b2a-9031-15ab79ee8b4b/67653f37-b9c9-4d64-b6e1-f65d439758bf"
-					(reference "#PWR511")
+					"/f0293046-ef42-43e4-84be-baa87b4d212c/fe69304b-7994-4faa-a0a5-98ff64846006"
+					(reference "#PWR611")
 					(unit 1)
 				)
@@
 		(property
 			"Reference"
-			"#PWR512"
+			"#PWR612"
 			(at 99.06 118.11 0)
 			(effects
@@
 				"Zynq_Carrier"
 				(path
-					"/5dc66003-6dff-4b2a-9031-15ab79ee8b4b/67653f37-b9c9-4d64-b6e1-f65d439758bf"
-					(reference "#PWR512")
+					"/f0293046-ef42-43e4-84be-baa87b4d212c/fe69304b-7994-4faa-a0a5-98ff64846006"
+					(reference "#PWR612")
 					(unit 1)
 				)
@@
 		(property
 			"Reference"
-			"#PWR513"
+			"#PWR613"
 			(at 105.41 120.65 0)
 			(effects
@@
 				"Zynq_Carrier"
 				(path
-					"/5dc66003-6dff-4b2a-9031-15ab79ee8b4b/67653f37-b9c9-4d64-b6e1-f65d439758bf"
-					(reference "#PWR513")
+					"/f0293046-ef42-43e4-84be-baa87b4d212c/fe69304b-7994-4faa-a0a5-98ff64846006"
+					(reference "#PWR613")
 					(unit 1)
 				)
@@
 		(property
 			"Reference"
-			"#PWR514"
+			"#PWR614"
 			(at 158.75 120.65 0)
 			(effects
@@
 				"Zynq_Carrier"
 				(path
-					"/5dc66003-6dff-4b2a-9031-15ab79ee8b4b/67653f37-b9c9-4d64-b6e1-f65d439758bf"
-					(reference "#PWR514")
-					(unit 1)
-				)
+					"/f0293046-ef42-43e4-84be-baa87b4d212c/fe69304b-7994-4faa-a0a5-98ff64846006"
+					(reference "#PWR614")
+					(unit 1)
+				)

Commit message: audit-fix(engine): harvest F1-F7,F9 — gate hardening + leak + guards
F1 selftest now exercises the VISUAL gate against geometry mutants (wire-cross
+ text-over-wire) — proven to bite (was never run on a mutant before).
F2 visual_gate catches different-net wire T-touch / butt-join shorts.
F3 netlist_gate no longer leaks tmp .net files (was 2671 stale).
F4 board uniquify guards the stride (widened 100->1000) against ref collision.
F5 hier-mode sheets now re-run through the per-sheet netlist gate.
F6 dead clause dropped; F7 stale zynq_eda docstring fixed; F9 eager inline-pin
validation. Source copied verbatim from the audit-fix worktree (6 files, proven
untouched on origin since its base); board regenerated fresh. All gates green,
selftest geo-mutants killed by the visual gate, goldens 23/23, m1_rc PASS.

Co-Authored-By: Claude Fable 5 <noreply@anthropic.com>
Parts:
- renumbered J601 to J6001, J602 to J6002, R601 to R6001, R602 to R6002, R603 to R6003, R604 to R6004, R605 to R6005, R606 to R6006, SW601 to SW6001, SW602 to SW6002
Changed lines of the file:
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@@
 		(property
 			"Reference"
-			"SW601"
+			"SW6001"
 			(at 90.17 73.025 0)
 			(effects
@@
 				(path
 					"/c2797150-7a6e-556a-82f5-fdda13c31368/f595abbb-cfb6-58c9-833d-958a6d6e62ca"
-					(reference "SW601")
+					(reference "SW6001")
 					(unit 1)
 				)
@@
 		(property
 			"Reference"
-			"R605"
+			"R6005"
 			(at 54.712 72.39 0)
 			(effects
@@
 				(path
 					"/c2797150-7a6e-556a-82f5-fdda13c31368/f595abbb-cfb6-58c9-833d-958a6d6e62ca"
-					(reference "R605")
+					(reference "R6005")
 					(unit 1)
 				)
@@
 		(property
 			"Reference"
-			"R604"
+			"R6004"
 			(at 105.513 69.85 0)
 			(effects
@@
 				(path
 					"/c2797150-7a6e-556a-82f5-fdda13c31368/f595abbb-cfb6-58c9-833d-958a6d6e62ca"
-					(reference "R604")
+					(reference "R6004")
 					(unit 1)
 				)
@@
 		(property
 			"Reference"
-			"R606"
+			"R6006"
 			(at 130.912 69.85 0)
 			(effects
@@
 				(path
 					"/c2797150-7a6e-556a-82f5-fdda13c31368/f595abbb-cfb6-58c9-833d-958a6d6e62ca"
-					(reference "R606")
+					(reference "R6006")
 					(unit 1)
 				)
@@
 		(property
 			"Reference"
-			"R603"
+			"R6003"
 			(at 141.072 69.85 0)
 			(effects
@@
 				(path
 					"/c2797150-7a6e-556a-82f5-fdda13c31368/f595abbb-cfb6-58c9-833d-958a6d6e62ca"
-					(reference "R603")
+					(reference "R6003")
 					(unit 1)
 				)
@@
 		(property
 			"Reference"
-			"SW602"
+			"SW6002"
 			(at 177.8 75.565 0)
 			(effects
@@
 				(path
 					"/c2797150-7a6e-556a-82f5-fdda13c31368/f595abbb-cfb6-58c9-833d-958a6d6e62ca"
-					(reference "SW602")
+					(reference "SW6002")
 					(unit 1)
 				)
@@
 		(property
 			"Reference"
-			"J602"
+			"J6002"
 			(at 248.92 65.405 0)
 			(effects
@@
 				(path
 					"/c2797150-7a6e-556a-82f5-fdda13c31368/f595abbb-cfb6-58c9-833d-958a6d6e62ca"
-					(reference "J602")
+					(reference "J6002")
 					(unit 1)
 				)
@@
 		(property
 			"Reference"
-			"J601"
+			"J6001"
 			(at 90.17 95.885 0)
 			(effects
@@
 				(path
 					"/c2797150-7a6e-556a-82f5-fdda13c31368/f595abbb-cfb6-58c9-833d-958a6d6e62ca"
-					(reference "J601")
+					(reference "J6001")
 					(unit 1)
 				)
@@
 		(property
 			"Reference"
-			"R601"
+			"R6001"
 			(at 108.053 118.11 0)
 			(effects
@@
 				(path
 					"/c2797150-7a6e-556a-82f5-fdda13c31368/f595abbb-cfb6-58c9-833d-958a6d6e62ca"
-					(reference "R601")
+					(reference "R6001")
 					(unit 1)
 				)
@@
 		(property
 			"Reference"
-			"R602"
+			"R6002"
 			(at 161.393 118.11 0)
 			(effects
@@
 				(path
 					"/c2797150-7a6e-556a-82f5-fdda13c31368/f595abbb-cfb6-58c9-833d-958a6d6e62ca"
-					(reference "R602")
+					(reference "R6002")
 					(unit 1)
 				)
@@
 		(property
 			"Reference"
-			"#PWR601"
+			"#PWR6001"
 			(at 81.28 82.55 0)
 			(effects
@@
 				(path
 					"/c2797150-7a6e-556a-82f5-fdda13c31368/f595abbb-cfb6-58c9-833d-958a6d6e62ca"
-					(reference "#PWR601")
+					(reference "#PWR6001")
 					(unit 1)
 				)
@@
 		(property
 			"Reference"
-			"#PWR602"
+			"#PWR6002"
 			(at 52.07 67.31 0)
 			(effects
@@
 				(path
 					"/c2797150-7a6e-556a-82f5-fdda13c31368/f595abbb-cfb6-58c9-833d-958a6d6e62ca"
-					(reference "#PWR602")
+					(reference "#PWR6002")
 					(unit 1)
 				)
@@
 		(property
 			"Reference"
-			"#PWR603"
+			"#PWR6003"
 			(at 99.06 80.01 0)
 			(effects
@@
 				(path
 					"/c2797150-7a6e-556a-82f5-fdda13c31368/f595abbb-cfb6-58c9-833d-958a6d6e62ca"
-					(reference "#PWR603")
+					(reference "#PWR6003")
 					(unit 1)
 				)
@@
 		(property
 			"Reference"
-			"#PWR604"
+			"#PWR6004"
 			(at 102.87 64.77 0)
 			(effects
@@
 				(path
 					"/c2797150-7a6e-556a-82f5-fdda13c31368/f595abbb-cfb6-58c9-833d-958a6d6e62ca"
-					(reference "#PWR604")
+					(reference "#PWR6004")
 					(unit 1)
 				)
@@
 		(property
 			"Reference"
-			"#PWR605"
+			"#PWR6005"
 			(at 128.27 64.77 0)
 			(effects
@@
 				(path
 					"/c2797150-7a6e-556a-82f5-fdda13c31368/f595abbb-cfb6-58c9-833d-958a6d6e62ca"
-					(reference "#PWR605")
+					(reference "#PWR6005")
 					(unit 1)
 				)
@@
 		(property
 			"Reference"
-			"#PWR606"
+			"#PWR6006"
 			(at 138.43 64.77 0)
 			(effects
@@
 				(path
 					"/c2797150-7a6e-556a-82f5-fdda13c31368/f595abbb-cfb6-58c9-833d-958a6d6e62ca"
-					(reference "#PWR606")
+					(reference "#PWR6006")
 					(unit 1)
 				)
@@
 		(property
 			"Reference"
-			"#PWR607"
+			"#PWR6007"
 			(at 166.37 80.01 0)
 			(effects
@@
 				(path
 					"/c2797150-7a6e-556a-82f5-fdda13c31368/f595abbb-cfb6-58c9-833d-958a6d6e62ca"
-					(reference "#PWR607")
+					(reference "#PWR6007")
 					(unit 1)
 				)
@@
 		(property
 			"Reference"
-			"#PWR608"
+			"#PWR6008"
 			(at 257.81 62.23 0)
 			(effects
@@
 				(path
 					"/c2797150-7a6e-556a-82f5-fdda13c31368/f595abbb-cfb6-58c9-833d-958a6d6e62ca"
-					(reference "#PWR608")
+					(reference "#PWR6008")
 					(unit 1)
 				)
@@
 		(property
 			"Reference"
-			"#PWR609"
+			"#PWR6009"
 			(at 257.81 74.93 0)
 			(effects
@@
 				(path
 					"/c2797150-7a6e-556a-82f5-fdda13c31368/f595abbb-cfb6-58c9-833d-958a6d6e62ca"
-					(reference "#PWR609")
+					(reference "#PWR6009")
 					(unit 1)
 				)
@@
 		(property
 			"Reference"
-			"#PWR610"
+			"#PWR6010"
 			(at 260.35 82.55 0)
 			(effects
@@
 				(path
 					"/c2797150-7a6e-556a-82f5-fdda13c31368/f595abbb-cfb6-58c9-833d-958a6d6e62ca"
-					(reference "#PWR610")
+					(reference "#PWR6010")
 					(unit 1)
 				)
@@
 		(property
 			"Reference"
-			"#PWR611"
+			"#PWR6011"
 			(at 81.28 113.03 0)
 			(effects
@@
 				(path
 					"/c2797150-7a6e-556a-82f5-fdda13c31368/f595abbb-cfb6-58c9-833d-958a6d6e62ca"
-					(reference "#PWR611")
+					(reference "#PWR6011")
 					(unit 1)
 				)
@@
 		(property
 			"Reference"
-			"#PWR612"
+			"#PWR6012"
 			(at 99.06 118.11 0)
 			(effects
@@
 				(path
 					"/c2797150-7a6e-556a-82f5-fdda13c31368/f595abbb-cfb6-58c9-833d-958a6d6e62ca"
-					(reference "#PWR612")
+					(reference "#PWR6012")
 					(unit 1)
 				)
@@
 		(property
 			"Reference"
-			"#PWR613"
+			"#PWR6013"
 			(at 105.41 120.65 0)
 			(effects
@@
 				(path
 					"/c2797150-7a6e-556a-82f5-fdda13c31368/f595abbb-cfb6-58c9-833d-958a6d6e62ca"
-					(reference "#PWR613")
+					(reference "#PWR6013")
 					(unit 1)
 				)
@@
 		(property
 			"Reference"
-			"#PWR614"
+			"#PWR6014"
 			(at 158.75 120.65 0)
 			(effects
@@
 				(path
 					"/c2797150-7a6e-556a-82f5-fdda13c31368/f595abbb-cfb6-58c9-833d-958a6d6e62ca"
-					(reference "#PWR614")
-					(unit 1)
-				)
+					(reference "#PWR6014")
+					(unit 1)
+				)

Commit message: genpolish: TITLE-1 — populate the schematic title block on every sheet
Every sheet rendered a blank Title/Rev/Date — the clearest 'not a real
schematic' tell. emit() now writes a (title_block ...) after the paper node:
title = the sheet circuit's title, company "Zynq SoM Carrier", and a
"<sheet> — generated by schgen (do not hand-edit)" comment. NO date node — a
wall-clock date would break byte-determinism; the content-derived fields keep
every rebuild identical. Verified on A4 (usb_pd) and the dense A3 (power): the
block fills the standard reserved corner with zero drawing overlap. All 26
sheets, goldens re-blessed, board PASS + deterministic, selftest 53/53, m1,
pytest 147.

Co-Authored-By: Claude Opus 4.8 <noreply@anthropic.com>
Other:
- company: (none) -> Zynq SoM Carrier
- title: (none) -> JTAG + SWD headers, boot-request DIP, reset
Changed lines of the file:
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@@
 	(generator_version "1.0")
 	(paper "A4")
+	(title_block
+		(title "JTAG + SWD headers, boot-request DIP, reset")
+		(company "Zynq SoM Carrier")
+		(comment 1 "debug_boot — generated by schgen (do not hand-edit)")
+	)
 	(wire
 		(pts
