File: carrier/schematic/microsd.kicad_sch (KiCad schematic)
At the start: 14 parts, among them J1201 TF-01A, U1201 TXS02612RTWR, U1202 TPD6E001RSER

Commit message: carrier: wave-2 consolidated regeneration — ALL round-4 gates live (POWER TREE 12 regulators / TESTPOINTS 43+9 / SPICE 14 checks incl. the caught CP2102N abs-max fix), LINK 0/0, goldens 23/23, byte-deterministic
Co-Authored-By: Claude Fable 5 <noreply@anthropic.com>
Changed lines of the file:
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@@
-	(wire
-		(pts
-			(xy 105.41 218.44)
-			(xy 105.41 220.98)
-		)
-		(stroke
-			(width 0)
-			(type default)
-		)
-	)
 	(wire
 		(pts
@@
 				"Zynq_Carrier"
 				(path
-					"/210e47c2-a83b-45be-ae0a-d7b3f3834bfa/82483d64-bb32-47a8-a892-d0113c6d7170"
+					"/c2797150-7a6e-556a-82f5-fdda13c31368/d897b633-e4e1-5c36-ba27-9e08872325fa"
 					(reference "U1201")
 					(unit 1)
@@
 				"Zynq_Carrier"
 				(path
-					"/210e47c2-a83b-45be-ae0a-d7b3f3834bfa/82483d64-bb32-47a8-a892-d0113c6d7170"
+					"/c2797150-7a6e-556a-82f5-fdda13c31368/d897b633-e4e1-5c36-ba27-9e08872325fa"
 					(reference "J1201")
 					(unit 1)
@@
 				"Zynq_Carrier"
 				(path
-					"/210e47c2-a83b-45be-ae0a-d7b3f3834bfa/82483d64-bb32-47a8-a892-d0113c6d7170"
+					"/c2797150-7a6e-556a-82f5-fdda13c31368/d897b633-e4e1-5c36-ba27-9e08872325fa"
 					(reference "R1206")
 					(unit 1)
@@
 				"Zynq_Carrier"
 				(path
-					"/210e47c2-a83b-45be-ae0a-d7b3f3834bfa/82483d64-bb32-47a8-a892-d0113c6d7170"
+					"/c2797150-7a6e-556a-82f5-fdda13c31368/d897b633-e4e1-5c36-ba27-9e08872325fa"
 					(reference "C1201")
 					(unit 1)
@@
 				"Zynq_Carrier"
 				(path
-					"/210e47c2-a83b-45be-ae0a-d7b3f3834bfa/82483d64-bb32-47a8-a892-d0113c6d7170"
+					"/c2797150-7a6e-556a-82f5-fdda13c31368/d897b633-e4e1-5c36-ba27-9e08872325fa"
 					(reference "C1202")
 					(unit 1)
@@
 				"Zynq_Carrier"
 				(path
-					"/210e47c2-a83b-45be-ae0a-d7b3f3834bfa/82483d64-bb32-47a8-a892-d0113c6d7170"
+					"/c2797150-7a6e-556a-82f5-fdda13c31368/d897b633-e4e1-5c36-ba27-9e08872325fa"
 					(reference "C1203")
 					(unit 1)
@@
 				"Zynq_Carrier"
 				(path
-					"/210e47c2-a83b-45be-ae0a-d7b3f3834bfa/82483d64-bb32-47a8-a892-d0113c6d7170"
+					"/c2797150-7a6e-556a-82f5-fdda13c31368/d897b633-e4e1-5c36-ba27-9e08872325fa"
 					(reference "U1202")
 					(unit 1)
@@
 				"Zynq_Carrier"
 				(path
-					"/210e47c2-a83b-45be-ae0a-d7b3f3834bfa/82483d64-bb32-47a8-a892-d0113c6d7170"
+					"/c2797150-7a6e-556a-82f5-fdda13c31368/d897b633-e4e1-5c36-ba27-9e08872325fa"
 					(reference "R1201")
 					(unit 1)
@@
 				"Zynq_Carrier"
 				(path
-					"/210e47c2-a83b-45be-ae0a-d7b3f3834bfa/82483d64-bb32-47a8-a892-d0113c6d7170"
+					"/c2797150-7a6e-556a-82f5-fdda13c31368/d897b633-e4e1-5c36-ba27-9e08872325fa"
 					(reference "R1202")
 					(unit 1)
@@
 				"Zynq_Carrier"
 				(path
-					"/210e47c2-a83b-45be-ae0a-d7b3f3834bfa/82483d64-bb32-47a8-a892-d0113c6d7170"
+					"/c2797150-7a6e-556a-82f5-fdda13c31368/d897b633-e4e1-5c36-ba27-9e08872325fa"
 					(reference "R1203")
 					(unit 1)
@@
 				"Zynq_Carrier"
 				(path
-					"/210e47c2-a83b-45be-ae0a-d7b3f3834bfa/82483d64-bb32-47a8-a892-d0113c6d7170"
+					"/c2797150-7a6e-556a-82f5-fdda13c31368/d897b633-e4e1-5c36-ba27-9e08872325fa"
 					(reference "R1204")
 					(unit 1)
@@
 				"Zynq_Carrier"
 				(path
-					"/210e47c2-a83b-45be-ae0a-d7b3f3834bfa/82483d64-bb32-47a8-a892-d0113c6d7170"
+					"/c2797150-7a6e-556a-82f5-fdda13c31368/d897b633-e4e1-5c36-ba27-9e08872325fa"
 					(reference "R1205")
 					(unit 1)
@@
 				"Zynq_Carrier"
 				(path
-					"/210e47c2-a83b-45be-ae0a-d7b3f3834bfa/82483d64-bb32-47a8-a892-d0113c6d7170"
+					"/c2797150-7a6e-556a-82f5-fdda13c31368/d897b633-e4e1-5c36-ba27-9e08872325fa"
 					(reference "TP1201")
 					(unit 1)
@@
 				"Zynq_Carrier"
 				(path
-					"/210e47c2-a83b-45be-ae0a-d7b3f3834bfa/82483d64-bb32-47a8-a892-d0113c6d7170"
+					"/c2797150-7a6e-556a-82f5-fdda13c31368/d897b633-e4e1-5c36-ba27-9e08872325fa"
 					(reference "TP1202")
 					(unit 1)
@@
 				"Zynq_Carrier"
 				(path
-					"/210e47c2-a83b-45be-ae0a-d7b3f3834bfa/82483d64-bb32-47a8-a892-d0113c6d7170"
+					"/c2797150-7a6e-556a-82f5-fdda13c31368/d897b633-e4e1-5c36-ba27-9e08872325fa"
 					(reference "#PWR1201")
 					(unit 1)
@@
 				"Zynq_Carrier"
 				(path
-					"/210e47c2-a83b-45be-ae0a-d7b3f3834bfa/82483d64-bb32-47a8-a892-d0113c6d7170"
+					"/c2797150-7a6e-556a-82f5-fdda13c31368/d897b633-e4e1-5c36-ba27-9e08872325fa"
 					(reference "#PWR1202")
 					(unit 1)
@@
 				"Zynq_Carrier"
 				(path
-					"/210e47c2-a83b-45be-ae0a-d7b3f3834bfa/82483d64-bb32-47a8-a892-d0113c6d7170"
+					"/c2797150-7a6e-556a-82f5-fdda13c31368/d897b633-e4e1-5c36-ba27-9e08872325fa"
 					(reference "#PWR1203")
 					(unit 1)
@@
 				"Zynq_Carrier"
 				(path
-					"/210e47c2-a83b-45be-ae0a-d7b3f3834bfa/82483d64-bb32-47a8-a892-d0113c6d7170"
+					"/c2797150-7a6e-556a-82f5-fdda13c31368/d897b633-e4e1-5c36-ba27-9e08872325fa"
 					(reference "#PWR1204")
 					(unit 1)
@@
 				"Zynq_Carrier"
 				(path
-					"/210e47c2-a83b-45be-ae0a-d7b3f3834bfa/82483d64-bb32-47a8-a892-d0113c6d7170"
+					"/c2797150-7a6e-556a-82f5-fdda13c31368/d897b633-e4e1-5c36-ba27-9e08872325fa"
 					(reference "#PWR1205")
 					(unit 1)
@@
 				"Zynq_Carrier"
 				(path
-					"/210e47c2-a83b-45be-ae0a-d7b3f3834bfa/82483d64-bb32-47a8-a892-d0113c6d7170"
+					"/c2797150-7a6e-556a-82f5-fdda13c31368/d897b633-e4e1-5c36-ba27-9e08872325fa"
 					(reference "#PWR1206")
 					(unit 1)
@@
 				"Zynq_Carrier"
 				(path
-					"/210e47c2-a83b-45be-ae0a-d7b3f3834bfa/82483d64-bb32-47a8-a892-d0113c6d7170"
+					"/c2797150-7a6e-556a-82f5-fdda13c31368/d897b633-e4e1-5c36-ba27-9e08872325fa"
 					(reference "#PWR1207")
 					(unit 1)
@@
 				"Zynq_Carrier"
 				(path
-					"/210e47c2-a83b-45be-ae0a-d7b3f3834bfa/82483d64-bb32-47a8-a892-d0113c6d7170"
+					"/c2797150-7a6e-556a-82f5-fdda13c31368/d897b633-e4e1-5c36-ba27-9e08872325fa"
 					(reference "#PWR1208")
 					(unit 1)
@@
 				"Zynq_Carrier"
 				(path
-					"/210e47c2-a83b-45be-ae0a-d7b3f3834bfa/82483d64-bb32-47a8-a892-d0113c6d7170"
+					"/c2797150-7a6e-556a-82f5-fdda13c31368/d897b633-e4e1-5c36-ba27-9e08872325fa"
 					(reference "#PWR1209")
 					(unit 1)
@@
 				"Zynq_Carrier"
 				(path
-					"/210e47c2-a83b-45be-ae0a-d7b3f3834bfa/82483d64-bb32-47a8-a892-d0113c6d7170"
+					"/c2797150-7a6e-556a-82f5-fdda13c31368/d897b633-e4e1-5c36-ba27-9e08872325fa"
 					(reference "#PWR1210")
 					(unit 1)
@@
 				"Zynq_Carrier"
 				(path
-					"/210e47c2-a83b-45be-ae0a-d7b3f3834bfa/82483d64-bb32-47a8-a892-d0113c6d7170"
+					"/c2797150-7a6e-556a-82f5-fdda13c31368/d897b633-e4e1-5c36-ba27-9e08872325fa"
 					(reference "#PWR1211")
 					(unit 1)
@@
 				"Zynq_Carrier"
 				(path
-					"/210e47c2-a83b-45be-ae0a-d7b3f3834bfa/82483d64-bb32-47a8-a892-d0113c6d7170"
+					"/c2797150-7a6e-556a-82f5-fdda13c31368/d897b633-e4e1-5c36-ba27-9e08872325fa"
 					(reference "#PWR1212")
 					(unit 1)
@@
 				"Zynq_Carrier"
 				(path
-					"/210e47c2-a83b-45be-ae0a-d7b3f3834bfa/82483d64-bb32-47a8-a892-d0113c6d7170"
+					"/c2797150-7a6e-556a-82f5-fdda13c31368/d897b633-e4e1-5c36-ba27-9e08872325fa"
 					(reference "#PWR1213")
 					(unit 1)
@@
 				"Zynq_Carrier"
 				(path
-					"/210e47c2-a83b-45be-ae0a-d7b3f3834bfa/82483d64-bb32-47a8-a892-d0113c6d7170"
+					"/c2797150-7a6e-556a-82f5-fdda13c31368/d897b633-e4e1-5c36-ba27-9e08872325fa"
 					(reference "#PWR1214")
 					(unit 1)
 				)
-			)
-		)
-	)
-	(symbol
-		(lib_id "power:+1V8")
-		(at 105.41 218.44 0)
-		(unit 1)
-		(exclude_from_sim no)
-		(in_bom yes)
-		(on_board yes)
-		(dnp no)
-		(property
-			"Reference"
-			"#PWR1215"
-			(at 105.41 215.9 0)
-			(effects
-				(font
-					(size 1.27 1.27)
-				)
-				(hide yes)
-			)
-		)
-		(property
-			"Value"
-			"+1V8"
-			(at 105.41 214.884 0)
-			(effects
-				(font
-					(size 1.27 1.27)
-				)
-			)
-		)
-		(property
-			"Footprint"
-			""
-			(at 105.41 218.44 0)
-			(effects
-				(font
-					(size 1.27 1.27)
-				)
-				(hide yes)
-			)
-		)
-		(property
-			"Datasheet"
-			""
-			(at 105.41 218.44 0)
-			(effects
-				(font
-					(size 1.27 1.27)
-				)
-				(hide yes)
-			)
-		)
-		(pin
-			"1"
-		)
-		(instances
-			(project
-				"Zynq_Carrier"
-				(path
-					"/210e47c2-a83b-45be-ae0a-d7b3f3834bfa/82483d64-bb32-47a8-a892-d0113c6d7170"
-					(reference "#PWR1215")
-					(unit 1)
-				)
-			)
-		)
-	)
-	(symbol
-		(lib_id "power:PWR_FLAG")
-		(at 105.41 220.98 180)
-		(unit 1)
-		(exclude_from_sim no)
-		(in_bom yes)
-		(on_board yes)
-		(dnp no)
-		(property
-			"Reference"
-			"#FLG1201"
-			(at 105.41 218.44 0)
-			(effects
-				(font
-					(size 1.27 1.27)
-				)
-				(hide yes)
-			)
-		)
-		(property
-			"Value"
-			"PWR_FLAG"
-			(at 105.41 223.52 0)
-			(effects
-				(font
-					(size 1.27 1.27)
-				)
-				(hide yes)
-			)
-		)
-		(property
-			"Footprint"
-			""
-			(at 105.41 220.98 0)
-			(effects
-				(font
-					(size 1.27 1.27)
-				)
-				(hide yes)
-			)
-		)
-		(property
-			"Datasheet"
-			""
-			(at 105.41 220.98 0)
-			(effects
-				(font
-					(size 1.27 1.27)
-				)
-				(hide yes)
-			)
-		)
-		(pin
-			"1"
-		)
-		(instances
-			(project
-				"Zynq_Carrier"
-				(path
-					"/210e47c2-a83b-45be-ae0a-d7b3f3834bfa/82483d64-bb32-47a8-a892-d0113c6d7170"
-					(reference "#FLG1201")
-					(unit 1)
-				)

Commit message: audit-fix(engine): harvest F1-F7,F9 — gate hardening + leak + guards
F1 selftest now exercises the VISUAL gate against geometry mutants (wire-cross
+ text-over-wire) — proven to bite (was never run on a mutant before).
F2 visual_gate catches different-net wire T-touch / butt-join shorts.
F3 netlist_gate no longer leaks tmp .net files (was 2671 stale).
F4 board uniquify guards the stride (widened 100->1000) against ref collision.
F5 hier-mode sheets now re-run through the per-sheet netlist gate.
F6 dead clause dropped; F7 stale zynq_eda docstring fixed; F9 eager inline-pin
validation. Source copied verbatim from the audit-fix worktree (6 files, proven
untouched on origin since its base); board regenerated fresh. All gates green,
selftest geo-mutants killed by the visual gate, goldens 23/23, m1_rc PASS.

Co-Authored-By: Claude Fable 5 <noreply@anthropic.com>
Parts:
- renumbered C1201 to C12001, C1202 to C12002, C1203 to C12003, J1201 to J12001, R1201 to R12001, R1202 to R12002, R1203 to R12003, R1204 to R12004, R1205 to R12005, R1206 to R12006, TP1201 to TP12001, TP1202 to TP12002, U1201 to U12001, U1202 to U12002
Changed lines of the file:
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@@
 		(property
 			"Reference"
-			"U1201"
+			"U12001"
 			(at 179.07 65.405 0)
 			(effects
@@
 				(path
 					"/c2797150-7a6e-556a-82f5-fdda13c31368/d897b633-e4e1-5c36-ba27-9e08872325fa"
-					(reference "U1201")
+					(reference "U12001")
 					(unit 1)
 				)
@@
 		(property
 			"Reference"
-			"J1201"
+			"J12001"
 			(at 269.24 73.025 0)
 			(effects
@@
 				(path
 					"/c2797150-7a6e-556a-82f5-fdda13c31368/d897b633-e4e1-5c36-ba27-9e08872325fa"
-					(reference "J1201")
+					(reference "J12001")
 					(unit 1)
 				)
@@
 		(property
 			"Reference"
-			"R1206"
+			"R12006"
 			(at 284.583 80.01 0)
 			(effects
@@
 				(path
 					"/c2797150-7a6e-556a-82f5-fdda13c31368/d897b633-e4e1-5c36-ba27-9e08872325fa"
-					(reference "R1206")
+					(reference "R12006")
 					(unit 1)
 				)
@@
 		(property
 			"Reference"
-			"C1201"
+			"C12001"
 			(at 134.469 132.08 0)
 			(effects
@@
 				(path
 					"/c2797150-7a6e-556a-82f5-fdda13c31368/d897b633-e4e1-5c36-ba27-9e08872325fa"
-					(reference "C1201")
+					(reference "C12001")
 					(unit 1)
 				)
@@
 		(property
 			"Reference"
-			"C1202"
+			"C12002"
 			(at 144.628 132.08 0)
 			(effects
@@
 				(path
 					"/c2797150-7a6e-556a-82f5-fdda13c31368/d897b633-e4e1-5c36-ba27-9e08872325fa"
-					(reference "C1202")
+					(reference "C12002")
 					(unit 1)
 				)
@@
 		(property
 			"Reference"
-			"C1203"
+			"C12003"
 			(at 154.788 132.08 0)
 			(effects
@@
 				(path
 					"/c2797150-7a6e-556a-82f5-fdda13c31368/d897b633-e4e1-5c36-ba27-9e08872325fa"
-					(reference "C1203")
+					(reference "C12003")
 					(unit 1)
 				)
@@
 		(property
 			"Reference"
-			"U1202"
+			"U12002"
 			(at 153.67 150.495 0)
 			(effects
@@
 				(path
 					"/c2797150-7a6e-556a-82f5-fdda13c31368/d897b633-e4e1-5c36-ba27-9e08872325fa"
-					(reference "U1202")
+					(reference "U12002")
 					(unit 1)
 				)
@@
 		(property
 			"Reference"
-			"R1201"
+			"R12001"
 			(at 113.132 203.2 0)
 			(effects
@@
 				(path
 					"/c2797150-7a6e-556a-82f5-fdda13c31368/d897b633-e4e1-5c36-ba27-9e08872325fa"
-					(reference "R1201")
+					(reference "R12001")
 					(unit 1)
 				)
@@
 		(property
 			"Reference"
-			"R1202"
+			"R12002"
 			(at 132.183 203.2 0)
 			(effects
@@
 				(path
 					"/c2797150-7a6e-556a-82f5-fdda13c31368/d897b633-e4e1-5c36-ba27-9e08872325fa"
-					(reference "R1202")
+					(reference "R12002")
 					(unit 1)
 				)
@@
 		(property
 			"Reference"
-			"R1203"
+			"R12003"
 			(at 151.232 203.2 0)
 			(effects
@@
 				(path
 					"/c2797150-7a6e-556a-82f5-fdda13c31368/d897b633-e4e1-5c36-ba27-9e08872325fa"
-					(reference "R1203")
+					(reference "R12003")
 					(unit 1)
 				)
@@
 		(property
 			"Reference"
-			"R1204"
+			"R12004"
 			(at 170.282 203.2 0)
 			(effects
@@
 				(path
 					"/c2797150-7a6e-556a-82f5-fdda13c31368/d897b633-e4e1-5c36-ba27-9e08872325fa"
-					(reference "R1204")
+					(reference "R12004")
 					(unit 1)
 				)
@@
 		(property
 			"Reference"
-			"R1205"
+			"R12005"
 			(at 189.332 203.2 0)
 			(effects
@@
 				(path
 					"/c2797150-7a6e-556a-82f5-fdda13c31368/d897b633-e4e1-5c36-ba27-9e08872325fa"
-					(reference "R1205")
+					(reference "R12005")
 					(unit 1)
 				)
@@
 		(property
 			"Reference"
-			"TP1201"
+			"TP12001"
 			(at 108.402 235.712 0)
 			(effects
@@
 				(path
 					"/c2797150-7a6e-556a-82f5-fdda13c31368/d897b633-e4e1-5c36-ba27-9e08872325fa"
-					(reference "TP1201")
+					(reference "TP12001")
 					(unit 1)
 				)
@@
 		(property
 			"Reference"
-			"TP1202"
+			"TP12002"
 			(at 124.912 235.712 0)
 			(effects
@@
 				(path
 					"/c2797150-7a6e-556a-82f5-fdda13c31368/d897b633-e4e1-5c36-ba27-9e08872325fa"
-					(reference "TP1202")
+					(reference "TP12002")
 					(unit 1)
 				)
@@
 		(property
 			"Reference"
-			"#PWR1201"
+			"#PWR12001"
 			(at 187.96 102.87 0)
 			(effects
@@
 				(path
 					"/c2797150-7a6e-556a-82f5-fdda13c31368/d897b633-e4e1-5c36-ba27-9e08872325fa"
-					(reference "#PWR1201")
+					(reference "#PWR12001")
 					(unit 1)
 				)
@@
 		(property
 			"Reference"
-			"#PWR1202"
+			"#PWR12002"
 			(at 173.99 59.69 0)
 			(effects
@@
 				(path
 					"/c2797150-7a6e-556a-82f5-fdda13c31368/d897b633-e4e1-5c36-ba27-9e08872325fa"
-					(reference "#PWR1202")
+					(reference "#PWR12002")
 					(unit 1)
 				)
@@
 		(property
 			"Reference"
-			"#PWR1203"
+			"#PWR12003"
 			(at 163.83 59.69 0)
 			(effects
@@
 				(path
 					"/c2797150-7a6e-556a-82f5-fdda13c31368/d897b633-e4e1-5c36-ba27-9e08872325fa"
-					(reference "#PWR1203")
+					(reference "#PWR12003")
 					(unit 1)
 				)
@@
 		(property
 			"Reference"
-			"#PWR1204"
+			"#PWR12004"
 			(at 171.45 115.57 0)
 			(effects
@@
 				(path
 					"/c2797150-7a6e-556a-82f5-fdda13c31368/d897b633-e4e1-5c36-ba27-9e08872325fa"
-					(reference "#PWR1204")
+					(reference "#PWR12004")
 					(unit 1)
 				)
@@
 		(property
 			"Reference"
-			"#PWR1205"
+			"#PWR12005"
 			(at 281.94 74.93 0)
 			(effects
@@
 				(path
 					"/c2797150-7a6e-556a-82f5-fdda13c31368/d897b633-e4e1-5c36-ba27-9e08872325fa"
-					(reference "#PWR1205")
+					(reference "#PWR12005")
 					(unit 1)
 				)
@@
 		(property
 			"Reference"
-			"#PWR1206"
+			"#PWR12006"
 			(at 257.81 67.31 0)
 			(effects
@@
 				(path
 					"/c2797150-7a6e-556a-82f5-fdda13c31368/d897b633-e4e1-5c36-ba27-9e08872325fa"
-					(reference "#PWR1206")
+					(reference "#PWR12006")
 					(unit 1)
 				)
@@
 		(property
 			"Reference"
-			"#PWR1207"
+			"#PWR12007"
 			(at 257.81 105.41 0)
 			(effects
@@
 				(path
 					"/c2797150-7a6e-556a-82f5-fdda13c31368/d897b633-e4e1-5c36-ba27-9e08872325fa"
-					(reference "#PWR1207")
+					(reference "#PWR12007")
 					(unit 1)
 				)
@@
 		(property
 			"Reference"
-			"#PWR1208"
+			"#PWR12008"
 			(at 130.81 134.62 0)
 			(effects
@@
 				(path
 					"/c2797150-7a6e-556a-82f5-fdda13c31368/d897b633-e4e1-5c36-ba27-9e08872325fa"
-					(reference "#PWR1208")
+					(reference "#PWR12008")
 					(unit 1)
 				)
@@
 		(property
 			"Reference"
-			"#PWR1209"
+			"#PWR12009"
 			(at 130.81 127 0)
 			(effects
@@
 				(path
 					"/c2797150-7a6e-556a-82f5-fdda13c31368/d897b633-e4e1-5c36-ba27-9e08872325fa"
-					(reference "#PWR1209")
+					(reference "#PWR12009")
 					(unit 1)
 				)
@@
 		(property
 			"Reference"
-			"#PWR1210"
+			"#PWR12010"
 			(at 140.97 134.62 0)
 			(effects
@@
 				(path
 					"/c2797150-7a6e-556a-82f5-fdda13c31368/d897b633-e4e1-5c36-ba27-9e08872325fa"
-					(reference "#PWR1210")
+					(reference "#PWR12010")
 					(unit 1)
 				)
@@
 		(property
 			"Reference"
-			"#PWR1211"
+			"#PWR12011"
 			(at 151.13 134.62 0)
 			(effects
@@
 				(path
 					"/c2797150-7a6e-556a-82f5-fdda13c31368/d897b633-e4e1-5c36-ba27-9e08872325fa"
-					(reference "#PWR1211")
+					(reference "#PWR12011")
 					(unit 1)
 				)
@@
 		(property
 			"Reference"
-			"#PWR1212"
+			"#PWR12012"
 			(at 146.05 124.46 0)
 			(effects
@@
 				(path
 					"/c2797150-7a6e-556a-82f5-fdda13c31368/d897b633-e4e1-5c36-ba27-9e08872325fa"
-					(reference "#PWR1212")
+					(reference "#PWR12012")
 					(unit 1)
 				)
@@
 		(property
 			"Reference"
-			"#PWR1213"
+			"#PWR12013"
 			(at 149.86 180.34 0)
 			(effects
@@
 				(path
 					"/c2797150-7a6e-556a-82f5-fdda13c31368/d897b633-e4e1-5c36-ba27-9e08872325fa"
-					(reference "#PWR1213")
+					(reference "#PWR12013")
 					(unit 1)
 				)
@@
 		(property
 			"Reference"
-			"#PWR1214"
+			"#PWR12014"
 			(at 148.59 195.58 0)
 			(effects
@@
 				(path
 					"/c2797150-7a6e-556a-82f5-fdda13c31368/d897b633-e4e1-5c36-ba27-9e08872325fa"
-					(reference "#PWR1214")
-					(unit 1)
-				)
+					(reference "#PWR12014")
+					(unit 1)
+				)
