File: carrier/schematic/microsd.kicad_sch (KiCad schematic)
At the start: 15 parts, among them J13001 TF-01A, U13001 TXS02612RTWR, U13002 TPD6E001RSER

Commit message: board: four board-management HW blocks on a manually-gated +3V3_AUX (BOARDHW)
The four services the carrier was missing — all behind ONE manual power enable
(C1) on two new sheets split so neither defeats the placer's rail-stub router:

  board_aux       — the gate + I2C isolator (infrastructure)
  board_services  — ID-EEPROM + RTC + watchdog + QWIIC (the peripherals)

WHAT LANDED
  * 24AA025E48 (C129895)  ID-EEPROM with a factory EUI-48 **MAC** for the
      LAN8720/RJ45 — strapped 0x51 (0x50 is the FMC EEPROM).
  * RV-3028-C7 (C3019759) I2C RTC, integrated DTCXO (no crystal), CR1220 coin
      cell (KH-CR1220-2) with auto-switchover, 0x52.
  * TPS3823-33 (C7719)    supervisor + windowed watchdog.
  * ZX-SH1.0-4PWT (C7430446)  QWIIC / STEMMA-QT expansion (gated 3V3 + the
      isolated AUX I2C).
  * SY6280 gate + DSHP04 DIP + PCA9306 isolator complete the infrastructure.

CONSTRAINTS (the user's three standing requirements)
  C1 manual enable "like the previous": +3V3_AUX is a SY6280 load switch whose
     EN is a default-OFF DSHP04 DIP (100k pulldown) — the same gated-module
     idiom, self-contained so it touches none of the dense rail/EN sheets.
  C2 "no watchdog reset during power-up": THREE independent guards — (1) the
     supervisor's VDD is the default-OFF +3V3_AUX, so it is UNPOWERED through
     power-up; (2) the TPS3823 disables its watchdog while WDI floats, and WDI
     is driven only by the PL (WATCHDOG_KICK, Hi-Z until the fabric is up); (3)
     RESET# is a firmware-mediated PL EVENT (J3.31), never a rail/POR line.
  C3 Zynq-agnostic: the only SoM-side signals (the 2 watchdog lines) ride PL
     bank-35 IO by their contract net names (IO_L16_N/P_35 -> J3.29/31); xdc.py
     emits the constraints live — nothing hard-codes the Zynq part.

LAW 0 (electrical integrity): the peripherals sit on the GATED rail but their
bus is the always-on STM32_I2C2 management bus. A PCA9306 bridges them with EN
tied to +3V3_AUX, so the switch OPENS whenever the rail is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
Parts:
- renumbered C13001 to C15001, C13002 to C15002, C13003 to C15003, C13004 to C15004, J13001 to J15001, R13001 to R15001, R13002 to R15002, R13003 to R15003, R13004 to R15004, R13005 to R15005, R13006 to R15006, TP13001 to TP15001, TP13002 to TP15002, U13001 to U15001, U13002 to U15002
Changed lines of the file:
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@@
 		(property
 			"Reference"
-			"U13001"
+			"U15001"
 			(at 181.61 65.405 0)
 			(effects
@@
 				(path
 					"/c2797150-7a6e-556a-82f5-fdda13c31368/d897b633-e4e1-5c36-ba27-9e08872325fa"
-					(reference "U13001")
+					(reference "U15001")
 					(unit 1)
 				)
@@
 		(property
 			"Reference"
-			"J13001"
+			"J15001"
 			(at 271.78 73.025 0)
 			(effects
@@
 				(path
 					"/c2797150-7a6e-556a-82f5-fdda13c31368/d897b633-e4e1-5c36-ba27-9e08872325fa"
-					(reference "J13001")
+					(reference "J15001")
 					(unit 1)
 				)
@@
 		(property
 			"Reference"
-			"R13006"
+			"R15006"
 			(at 287.123 80.01 0)
 			(effects
@@
 				(path
 					"/c2797150-7a6e-556a-82f5-fdda13c31368/d897b633-e4e1-5c36-ba27-9e08872325fa"
-					(reference "R13006")
+					(reference "R15006")
 					(unit 1)
 				)
@@
 		(property
 			"Reference"
-			"C13001"
+			"C15001"
 			(at 126.849 132.08 0)
 			(effects
@@
 				(path
 					"/c2797150-7a6e-556a-82f5-fdda13c31368/d897b633-e4e1-5c36-ba27-9e08872325fa"
-					(reference "C13001")
+					(reference "C15001")
 					(unit 1)
 				)
@@
 		(property
 			"Reference"
-			"C13002"
+			"C15002"
 			(at 137.009 132.08 0)
 			(effects
@@
 				(path
 					"/c2797150-7a6e-556a-82f5-fdda13c31368/d897b633-e4e1-5c36-ba27-9e08872325fa"
-					(reference "C13002")
+					(reference "C15002")
 					(unit 1)
 				)
@@
 		(property
 			"Reference"
-			"C13003"
+			"C15003"
 			(at 147.169 132.08 0)
 			(effects
@@
 				(path
 					"/c2797150-7a6e-556a-82f5-fdda13c31368/d897b633-e4e1-5c36-ba27-9e08872325fa"
-					(reference "C13003")
+					(reference "C15003")
 					(unit 1)
 				)
@@
 		(property
 			"Reference"
-			"C13004"
+			"C15004"
 			(at 157.329 132.08 0)
 			(effects
@@
 				(path
 					"/c2797150-7a6e-556a-82f5-fdda13c31368/d897b633-e4e1-5c36-ba27-9e08872325fa"
-					(reference "C13004")
+					(reference "C15004")
 					(unit 1)
 				)
@@
 		(property
 			"Reference"
-			"U13002"
+			"U15002"
 			(at 151.13 150.495 0)
 			(effects
@@
 				(path
 					"/c2797150-7a6e-556a-82f5-fdda13c31368/d897b633-e4e1-5c36-ba27-9e08872325fa"
-					(reference "U13002")
+					(reference "U15002")
 					(unit 1)
 				)
@@
 		(property
 			"Reference"
-			"R13001"
+			"R15001"
 			(at 110.593 203.2 0)
 			(effects
@@
 				(path
 					"/c2797150-7a6e-556a-82f5-fdda13c31368/d897b633-e4e1-5c36-ba27-9e08872325fa"
-					(reference "R13001")
+					(reference "R15001")
 					(unit 1)
 				)
@@
 		(property
 			"Reference"
-			"R13002"
+			"R15002"
 			(at 129.643 203.2 0)
 			(effects
@@
 				(path
 					"/c2797150-7a6e-556a-82f5-fdda13c31368/d897b633-e4e1-5c36-ba27-9e08872325fa"
-					(reference "R13002")
+					(reference "R15002")
 					(unit 1)
 				)
@@
 		(property
 			"Reference"
-			"R13003"
+			"R15003"
 			(at 148.693 203.2 0)
 			(effects
@@
 				(path
 					"/c2797150-7a6e-556a-82f5-fdda13c31368/d897b633-e4e1-5c36-ba27-9e08872325fa"
-					(reference "R13003")
+					(reference "R15003")
 					(unit 1)
 				)
@@
 		(property
 			"Reference"
-			"R13004"
+			"R15004"
 			(at 167.743 203.2 0)
 			(effects
@@
 				(path
 					"/c2797150-7a6e-556a-82f5-fdda13c31368/d897b633-e4e1-5c36-ba27-9e08872325fa"
-					(reference "R13004")
+					(reference "R15004")
 					(unit 1)
 				)
@@
 		(property
 			"Reference"
-			"R13005"
+			"R15005"
 			(at 186.792 203.2 0)
 			(effects
@@
 				(path
 					"/c2797150-7a6e-556a-82f5-fdda13c31368/d897b633-e4e1-5c36-ba27-9e08872325fa"
-					(reference "R13005")
+					(reference "R15005")
 					(unit 1)
 				)
@@
 		(property
 			"Reference"
-			"TP13001"
+			"TP15001"
 			(at 105.862 235.712 0)
 			(effects
@@
 				(path
 					"/c2797150-7a6e-556a-82f5-fdda13c31368/d897b633-e4e1-5c36-ba27-9e08872325fa"
-					(reference "TP13001")
+					(reference "TP15001")
 					(unit 1)
 				)
@@
 		(property
 			"Reference"
-			"TP13002"
+			"TP15002"
 			(at 122.372 235.712 0)
 			(effects
@@
 				(path
 					"/c2797150-7a6e-556a-82f5-fdda13c31368/d897b633-e4e1-5c36-ba27-9e08872325fa"
-					(reference "TP13002")
+					(reference "TP15002")
 					(unit 1)
 				)
@@
 		(property
 			"Reference"
-			"#PWR13001"
+			"#PWR15001"
 			(at 190.5 102.87 0)
 			(effects
@@
 				(path
 					"/c2797150-7a6e-556a-82f5-fdda13c31368/d897b633-e4e1-5c36-ba27-9e08872325fa"
-					(reference "#PWR13001")
+					(reference "#PWR15001")
 					(unit 1)
 				)
@@
 		(property
 			"Reference"
-			"#PWR13002"
+			"#PWR15002"
 			(at 176.53 59.69 0)
 			(effects
@@
 				(path
 					"/c2797150-7a6e-556a-82f5-fdda13c31368/d897b633-e4e1-5c36-ba27-9e08872325fa"
-					(reference "#PWR13002")
+					(reference "#PWR15002")
 					(unit 1)
 				)
@@
 		(property
 			"Reference"
-			"#PWR13003"
+			"#PWR15003"
 			(at 166.37 59.69 0)
 			(effects
@@
 				(path
 					"/c2797150-7a6e-556a-82f5-fdda13c31368/d897b633-e4e1-5c36-ba27-9e08872325fa"
-					(reference "#PWR13003")
+					(reference "#PWR15003")
 					(unit 1)
 				)
@@
 		(property
 			"Reference"
-			"#PWR13004"
+			"#PWR15004"
 			(at 173.99 115.57 0)
 			(effects
@@
 				(path
 					"/c2797150-7a6e-556a-82f5-fdda13c31368/d897b633-e4e1-5c36-ba27-9e08872325fa"
-					(reference "#PWR13004")
+					(reference "#PWR15004")
 					(unit 1)
 				)
@@
 		(property
 			"Reference"
-			"#PWR13005"
+			"#PWR15005"
 			(at 284.48 74.93 0)
 			(effects
@@
 				(path
 					"/c2797150-7a6e-556a-82f5-fdda13c31368/d897b633-e4e1-5c36-ba27-9e08872325fa"
-					(reference "#PWR13005")
+					(reference "#PWR15005")
 					(unit 1)
 				)
@@
 		(property
 			"Reference"
-			"#PWR13006"
+			"#PWR15006"
 			(at 260.35 67.31 0)
 			(effects
@@
 				(path
 					"/c2797150-7a6e-556a-82f5-fdda13c31368/d897b633-e4e1-5c36-ba27-9e08872325fa"
-					(reference "#PWR13006")
+					(reference "#PWR15006")
 					(unit 1)
 				)
@@
 		(property
 			"Reference"
-			"#PWR13007"
+			"#PWR15007"
 			(at 260.35 105.41 0)
 			(effects
@@
 				(path
 					"/c2797150-7a6e-556a-82f5-fdda13c31368/d897b633-e4e1-5c36-ba27-9e08872325fa"
-					(reference "#PWR13007")
+					(reference "#PWR15007")
 					(unit 1)
 				)
@@
 		(property
 			"Reference"
-			"#PWR13008"
+			"#PWR15008"
 			(at 123.19 134.62 0)
 			(effects
@@
 				(path
 					"/c2797150-7a6e-556a-82f5-fdda13c31368/d897b633-e4e1-5c36-ba27-9e08872325fa"
-					(reference "#PWR13008")
+					(reference "#PWR15008")
 					(unit 1)
 				)
@@
 		(property
 			"Reference"
-			"#PWR13009"
+			"#PWR15009"
 			(at 123.19 127 0)
 			(effects
@@
 				(path
 					"/c2797150-7a6e-556a-82f5-fdda13c31368/d897b633-e4e1-5c36-ba27-9e08872325fa"
-					(reference "#PWR13009")
+					(reference "#PWR15009")
 					(unit 1)
 				)
@@
 		(property
 			"Reference"
-			"#PWR13010"
+			"#PWR15010"
 			(at 133.35 134.62 0)
 			(effects
@@
 				(path
 					"/c2797150-7a6e-556a-82f5-fdda13c31368/d897b633-e4e1-5c36-ba27-9e08872325fa"
-					(reference "#PWR13010")
+					(reference "#PWR15010")
 					(unit 1)
 				)
@@
 		(property
 			"Reference"
-			"#PWR13011"
+			"#PWR15011"
 			(at 143.51 134.62 0)
 			(effects
@@
 				(path
 					"/c2797150-7a6e-556a-82f5-fdda13c31368/d897b633-e4e1-5c36-ba27-9e08872325fa"
-					(reference "#PWR13011")
+					(reference "#PWR15011")
 					(unit 1)
 				)
@@
 		(property
 			"Reference"
-			"#PWR13012"
+			"#PWR15012"
 			(at 153.67 134.62 0)
 			(effects
@@
 				(path
 					"/c2797150-7a6e-556a-82f5-fdda13c31368/d897b633-e4e1-5c36-ba27-9e08872325fa"
-					(reference "#PWR13012")
+					(reference "#PWR15012")
 					(unit 1)
 				)
@@
 		(property
 			"Reference"
-			"#PWR13013"
+			"#PWR15013"
 			(at 143.51 124.46 0)
 			(effects
@@
 				(path
 					"/c2797150-7a6e-556a-82f5-fdda13c31368/d897b633-e4e1-5c36-ba27-9e08872325fa"
-					(reference "#PWR13013")
+					(reference "#PWR15013")
 					(unit 1)
 				)
@@
 		(property
 			"Reference"
-			"#PWR13014"
+			"#PWR15014"
 			(at 147.32 144.78 0)
 			(effects
@@
 				(path
 					"/c2797150-7a6e-556a-82f5-fdda13c31368/d897b633-e4e1-5c36-ba27-9e08872325fa"
-					(reference "#PWR13014")
+					(reference "#PWR15014")
 					(unit 1)
 				)
@@
 		(property
 			"Reference"
-			"#PWR13015"
+			"#PWR15015"
 			(at 147.32 180.34 0)
 			(effects
@@
 				(path
 					"/c2797150-7a6e-556a-82f5-fdda13c31368/d897b633-e4e1-5c36-ba27-9e08872325fa"
-					(reference "#PWR13015")
+					(reference "#PWR15015")
 					(unit 1)
 				)
@@
 		(property
 			"Reference"
-			"#PWR13016"
+			"#PWR15016"
 			(at 146.05 195.58 0)
 			(effects
@@
 				(path
 					"/c2797150-7a6e-556a-82f5-fdda13c31368/d897b633-e4e1-5c36-ba27-9e08872325fa"
-					(reference "#PWR13016")
-					(unit 1)
-				)
+					(reference "#PWR15016")
+					(unit 1)
+				)
