File: carrier/schematic/ethernet.kicad_sch (KiCad schematic)
At the start: 10 parts, among them T701 HX5008NLT

Commit message: ethernet: 2kV BOB-SMITH (PLAN round 5) — genuine 1nF/2kV X7R 1206 on all 5 barrier caps
The first live-match C1588 was a 50 V 0603 part: fine at DC, USELESS as
the IEC hi-pot barrier the docstring promised. Replaced with C9196 —
FH/Fenghua 1206B102K202NT, LIVE-verified on the JLC parts API 2026-06-12
(the API attribute line itself reads '1nF 2kV X7R +/-10% 1206'): JLC
BASIC, stock 1,369,013, $0.036 @ 1. Alternates documented in the sheet
docstring: Walsin 1206B102K202 C77494 (21k, Ext), Walsin CT C303946
(2.5k), FH 1808B102K202NT C81332 (29.7k, Ext) if 1808 creepage is later
preferred. Round-5 said 'x4' but C5 — the single BS_COMMON->CHASSIS_GND
element that IS the isolation barrier — had the same 50 V bug; all FIVE
upgraded (noted honestly in the docstring). Footprint 0603 -> 1206.

PLAN: mechanical-debt Bob-Smith flag marked RESOLVED; added a
RECONCILIATION note to the concurrent wave-3 adoption (its USBOTG_FLT_N
-> P12 claim and 'no free DIP' assumption are stale against the committed
round-5 netlists: P12/P13 are the 5V-gate vetoes, SW6 has the HDMI_TX_5V
position — binding agent must read the generated header, not prose).

Render verified byte-stable: goldens 23/23 MATCH (value text unchanged;
only LCSC/footprint fields moved). Full regression: schgen board exit 0,
selftest 40/40 mutants killed + byte-determinism PASS, m1_rc PASS.

Co-Authored-By: Claude Fable 5 <noreply@anthropic.com>
Parts:
- C701, C702, C703, C704, C705: footprint Capacitor_SMD:C_0603_1608Metric -> Capacitor_SMD:C_1206_3225Metric; LCSC C1588 -> C9196
Changed lines of the file:
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@@
 		(property
 			"Footprint"
-			"Capacitor_SMD:C_0603_1608Metric"
+			"Capacitor_SMD:C_1206_3225Metric"
 			(at 133.35 120.65 0)
 			(effects
@@
 		(property
 			"LCSC"
-			"C1588"
+			"C9196"
 			(at 133.35 120.65 0)
 			(effects
@@
 		(property
 			"Footprint"
-			"Capacitor_SMD:C_0603_1608Metric"
+			"Capacitor_SMD:C_1206_3225Metric"
 			(at 148.59 120.65 0)
 			(effects
@@
 		(property
 			"LCSC"
-			"C1588"
+			"C9196"
 			(at 148.59 120.65 0)
 			(effects
@@
 		(property
 			"Footprint"
-			"Capacitor_SMD:C_0603_1608Metric"
+			"Capacitor_SMD:C_1206_3225Metric"
 			(at 163.83 120.65 0)
 			(effects
@@
 		(property
 			"LCSC"
-			"C1588"
+			"C9196"
 			(at 163.83 120.65 0)
 			(effects
@@
 		(property
 			"Footprint"
-			"Capacitor_SMD:C_0603_1608Metric"
+			"Capacitor_SMD:C_1206_3225Metric"
 			(at 179.07 120.65 0)
 			(effects
@@
 		(property
 			"LCSC"
-			"C1588"
+			"C9196"
 			(at 179.07 120.65 0)
 			(effects
@@
 		(property
 			"Footprint"
-			"Capacitor_SMD:C_0603_1608Metric"
+			"Capacitor_SMD:C_1206_3225Metric"
 			(at 189.23 128.27 0)
 			(effects
@@
 		(property
 			"LCSC"
-			"C1588"
+			"C9196"
 			(at 189.23 128.27 0)
 			(effects

Commit message: audit-fix(engine): harvest F1-F7,F9 — gate hardening + leak + guards
F1 selftest now exercises the VISUAL gate against geometry mutants (wire-cross
+ text-over-wire) — proven to bite (was never run on a mutant before).
F2 visual_gate catches different-net wire T-touch / butt-join shorts.
F3 netlist_gate no longer leaks tmp .net files (was 2671 stale).
F4 board uniquify guards the stride (widened 100->1000) against ref collision.
F5 hier-mode sheets now re-run through the per-sheet netlist gate.
F6 dead clause dropped; F7 stale zynq_eda docstring fixed; F9 eager inline-pin
validation. Source copied verbatim from the audit-fix worktree (6 files, proven
untouched on origin since its base); board regenerated fresh. All gates green,
selftest geo-mutants killed by the visual gate, goldens 23/23, m1_rc PASS.

Co-Authored-By: Claude Fable 5 <noreply@anthropic.com>
Parts:
- renumbered C701 to C7001, C702 to C7002, C703 to C7003, C704 to C7004, C705 to C7005, R701 to R7001, R702 to R7002, R703 to R7003, R704 to R7004, T701 to T7001
Changed lines of the file:
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@@
 		(property
 			"Reference"
-			"T701"
+			"T7001"
 			(at 175.26 51.435 0)
 			(effects
@@
 				(path
 					"/c2797150-7a6e-556a-82f5-fdda13c31368/4d664980-e58b-5403-9b49-c54d6ca52225"
-					(reference "T701")
+					(reference "T7001")
 					(unit 1)
 				)
@@
 		(property
 			"Reference"
-			"R701"
+			"R7001"
 			(at 123.088 111.76 0)
 			(effects
@@
 				(path
 					"/c2797150-7a6e-556a-82f5-fdda13c31368/4d664980-e58b-5403-9b49-c54d6ca52225"
-					(reference "R701")
+					(reference "R7001")
 					(unit 1)
 				)
@@
 		(property
 			"Reference"
-			"C701"
+			"C7001"
 			(at 137.008 119.38 0)
 			(effects
@@
 				(path
 					"/c2797150-7a6e-556a-82f5-fdda13c31368/4d664980-e58b-5403-9b49-c54d6ca52225"
-					(reference "C701")
+					(reference "C7001")
 					(unit 1)
 				)
@@
 		(property
 			"Reference"
-			"R702"
+			"R7002"
 			(at 138.328 111.76 0)
 			(effects
@@
 				(path
 					"/c2797150-7a6e-556a-82f5-fdda13c31368/4d664980-e58b-5403-9b49-c54d6ca52225"
-					(reference "R702")
+					(reference "R7002")
 					(unit 1)
 				)
@@
 		(property
 			"Reference"
-			"C702"
+			"C7002"
 			(at 152.249 119.38 0)
 			(effects
@@
 				(path
 					"/c2797150-7a6e-556a-82f5-fdda13c31368/4d664980-e58b-5403-9b49-c54d6ca52225"
-					(reference "C702")
+					(reference "C7002")
 					(unit 1)
 				)
@@
 		(property
 			"Reference"
-			"R703"
+			"R7003"
 			(at 153.567 111.76 0)
 			(effects
@@
 				(path
 					"/c2797150-7a6e-556a-82f5-fdda13c31368/4d664980-e58b-5403-9b49-c54d6ca52225"
-					(reference "R703")
+					(reference "R7003")
 					(unit 1)
 				)
@@
 		(property
 			"Reference"
-			"C703"
+			"C7003"
 			(at 167.488 119.38 0)
 			(effects
@@
 				(path
 					"/c2797150-7a6e-556a-82f5-fdda13c31368/4d664980-e58b-5403-9b49-c54d6ca52225"
-					(reference "C703")
+					(reference "C7003")
 					(unit 1)
 				)
@@
 		(property
 			"Reference"
-			"R704"
+			"R7004"
 			(at 168.808 111.76 0)
 			(effects
@@
 				(path
 					"/c2797150-7a6e-556a-82f5-fdda13c31368/4d664980-e58b-5403-9b49-c54d6ca52225"
-					(reference "R704")
+					(reference "R7004")
 					(unit 1)
 				)
@@
 		(property
 			"Reference"
-			"C704"
+			"C7004"
 			(at 182.728 119.38 0)
 			(effects
@@
 				(path
 					"/c2797150-7a6e-556a-82f5-fdda13c31368/4d664980-e58b-5403-9b49-c54d6ca52225"
-					(reference "C704")
+					(reference "C7004")
 					(unit 1)
 				)
@@
 		(property
 			"Reference"
-			"C705"
+			"C7005"
 			(at 192.888 127 0)
 			(effects
@@
 				(path
 					"/c2797150-7a6e-556a-82f5-fdda13c31368/4d664980-e58b-5403-9b49-c54d6ca52225"
-					(reference "C705")
+					(reference "C7005")
 					(unit 1)
 				)
@@
 		(property
 			"Reference"
-			"#PWR701"
+			"#PWR7001"
 			(at 184.15 101.6 0)
 			(effects
@@
 				(path
 					"/c2797150-7a6e-556a-82f5-fdda13c31368/4d664980-e58b-5403-9b49-c54d6ca52225"
-					(reference "#PWR701")
+					(reference "#PWR7001")
 					(unit 1)
 				)
@@
 		(property
 			"Reference"
-			"#PWR702"
+			"#PWR7002"
 			(at 189.23 129.54 0)
 			(effects
@@
 				(path
 					"/c2797150-7a6e-556a-82f5-fdda13c31368/4d664980-e58b-5403-9b49-c54d6ca52225"
-					(reference "#PWR702")
+					(reference "#PWR7002")
 					(unit 1)
 				)
@@
 		(property
 			"Reference"
-			"#PWR703"
+			"#PWR7003"
 			(at 92.71 142.24 0)
 			(effects
@@
 				(path
 					"/c2797150-7a6e-556a-82f5-fdda13c31368/4d664980-e58b-5403-9b49-c54d6ca52225"
-					(reference "#PWR703")
+					(reference "#PWR7003")
 					(unit 1)
 				)
@@
 		(property
 			"Reference"
-			"#FLG701"
+			"#FLG7001"
 			(at 92.71 139.7 0)
 			(effects
@@
 				(path
 					"/c2797150-7a6e-556a-82f5-fdda13c31368/4d664980-e58b-5403-9b49-c54d6ca52225"
-					(reference "#FLG701")
-					(unit 1)
-				)
+					(reference "#FLG7001")
+					(unit 1)
+				)

Commit message: genpolish: TITLE-1 — populate the schematic title block on every sheet
Every sheet rendered a blank Title/Rev/Date — the clearest 'not a real
schematic' tell. emit() now writes a (title_block ...) after the paper node:
title = the sheet circuit's title, company "Zynq SoM Carrier", and a
"<sheet> — generated by schgen (do not hand-edit)" comment. NO date node — a
wall-clock date would break byte-determinism; the content-derived fields keep
every rebuild identical. Verified on A4 (usb_pd) and the dense A3 (power): the
block fills the standard reserved corner with zero drawing overlap. All 26
sheets, goldens re-blessed, board PASS + deterministic, selftest 53/53, m1,
pytest 147.

Co-Authored-By: Claude Opus 4.8 <noreply@anthropic.com>
Other:
- company: (none) -> Zynq SoM Carrier
- title: (none) -> Ethernet: HX5008NLT magnetics + Bob-Smith
Changed lines of the file:
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@@
 	(generator_version "1.0")
 	(paper "A4")
+	(title_block
+		(title "Ethernet: HX5008NLT magnetics + Bob-Smith")
+		(company "Zynq SoM Carrier")
+		(comment 1 "ethernet — generated by schgen (do not hand-edit)")
+	)
 	(wire
 		(pts

Commit message: sourcing: regen ethernet.kicad_sch + manifest for the ALT_LCSC property
Follow-up to the SOURCING commit: ALT_LCSC IS emitted as a hidden symbol
property (so the schematic itself documents the committed second source — a
bonus), so the previous commit's "byte-identical" claim was wrong and it left
the regenerated ethernet.kicad_sch + manifest.json uncommitted. This commits
them, so a fresh board build reproduces the committed tree (determinism).
Render unaffected (hidden property) — 26 goldens match; BOM unchanged
(ALT_LCSC is not a BOM column); board PASS.

Co-Authored-By: Claude Opus 4.8 <noreply@anthropic.com>
Parts:
- T7001: ALT_LCSC (none) -> C47575004
Changed lines of the file:
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@@
+			)
+		)
+		(property
+			"ALT_LCSC"
+			"C47575004"
+			(at 148.59 76.2 0)
+			(effects
+				(font
+					(size 1.27 1.27)
+				)
+				(hide yes)
 			)
 		)

Commit message: board: four board-management HW blocks on a manually-gated +3V3_AUX (BOARDHW)
The four services the carrier was missing — all behind ONE manual power enable
(C1) on two new sheets split so neither defeats the placer's rail-stub router:

  board_aux       — the gate + I2C isolator (infrastructure)
  board_services  — ID-EEPROM + RTC + watchdog + QWIIC (the peripherals)

WHAT LANDED
  * 24AA025E48 (C129895)  ID-EEPROM with a factory EUI-48 **MAC** for the
      LAN8720/RJ45 — strapped 0x51 (0x50 is the FMC EEPROM).
  * RV-3028-C7 (C3019759) I2C RTC, integrated DTCXO (no crystal), CR1220 coin
      cell (KH-CR1220-2) with auto-switchover, 0x52.
  * TPS3823-33 (C7719)    supervisor + windowed watchdog.
  * ZX-SH1.0-4PWT (C7430446)  QWIIC / STEMMA-QT expansion (gated 3V3 + the
      isolated AUX I2C).
  * SY6280 gate + DSHP04 DIP + PCA9306 isolator complete the infrastructure.

CONSTRAINTS (the user's three standing requirements)
  C1 manual enable "like the previous": +3V3_AUX is a SY6280 load switch whose
     EN is a default-OFF DSHP04 DIP (100k pulldown) — the same gated-module
     idiom, self-contained so it touches none of the dense rail/EN sheets.
  C2 "no watchdog reset during power-up": THREE independent guards — (1) the
     supervisor's VDD is the default-OFF +3V3_AUX, so it is UNPOWERED through
     power-up; (2) the TPS3823 disables its watchdog while WDI floats, and WDI
     is driven only by the PL (WATCHDOG_KICK, Hi-Z until the fabric is up); (3)
     RESET# is a firmware-mediated PL EVENT (J3.31), never a rail/POR line.
  C3 Zynq-agnostic: the only SoM-side signals (the 2 watchdog lines) ride PL
     bank-35 IO by their contract net names (IO_L16_N/P_35 -> J3.29/31); xdc.py
     emits the constraints live — nothing hard-codes the Zynq part.

LAW 0 (electrical integrity): the peripherals sit on the GATED rail but their
bus is the always-on STM32_I2C2 management bus. A PCA9306 bridges them with EN
tied to +3V3_AUX, so the switch OPENS whenever the rail is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
Parts:
- renumbered C7001 to C9001, C7002 to C9002, C7003 to C9003, C7004 to C9004, C7005 to C9005, R7001 to R9001, R7002 to R9002, R7003 to R9003, R7004 to R9004, T7001 to T9001
Changed lines of the file:
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@@
 		(property
 			"Reference"
-			"T7001"
+			"T9001"
 			(at 175.26 51.435 0)
 			(effects
@@
 				(path
 					"/c2797150-7a6e-556a-82f5-fdda13c31368/4d664980-e58b-5403-9b49-c54d6ca52225"
-					(reference "T7001")
+					(reference "T9001")
 					(unit 1)
 				)
@@
 		(property
 			"Reference"
-			"R7001"
+			"R9001"
 			(at 123.088 111.76 0)
 			(effects
@@
 				(path
 					"/c2797150-7a6e-556a-82f5-fdda13c31368/4d664980-e58b-5403-9b49-c54d6ca52225"
-					(reference "R7001")
+					(reference "R9001")
 					(unit 1)
 				)
@@
 		(property
 			"Reference"
-			"C7001"
+			"C9001"
 			(at 137.008 119.38 0)
 			(effects
@@
 				(path
 					"/c2797150-7a6e-556a-82f5-fdda13c31368/4d664980-e58b-5403-9b49-c54d6ca52225"
-					(reference "C7001")
+					(reference "C9001")
 					(unit 1)
 				)
@@
 		(property
 			"Reference"
-			"R7002"
+			"R9002"
 			(at 138.328 111.76 0)
 			(effects
@@
 				(path
 					"/c2797150-7a6e-556a-82f5-fdda13c31368/4d664980-e58b-5403-9b49-c54d6ca52225"
-					(reference "R7002")
+					(reference "R9002")
 					(unit 1)
 				)
@@
 		(property
 			"Reference"
-			"C7002"
+			"C9002"
 			(at 152.249 119.38 0)
 			(effects
@@
 				(path
 					"/c2797150-7a6e-556a-82f5-fdda13c31368/4d664980-e58b-5403-9b49-c54d6ca52225"
-					(reference "C7002")
+					(reference "C9002")
 					(unit 1)
 				)
@@
 		(property
 			"Reference"
-			"R7003"
+			"R9003"
 			(at 153.567 111.76 0)
 			(effects
@@
 				(path
 					"/c2797150-7a6e-556a-82f5-fdda13c31368/4d664980-e58b-5403-9b49-c54d6ca52225"
-					(reference "R7003")
+					(reference "R9003")
 					(unit 1)
 				)
@@
 		(property
 			"Reference"
-			"C7003"
+			"C9003"
 			(at 167.488 119.38 0)
 			(effects
@@
 				(path
 					"/c2797150-7a6e-556a-82f5-fdda13c31368/4d664980-e58b-5403-9b49-c54d6ca52225"
-					(reference "C7003")
+					(reference "C9003")
 					(unit 1)
 				)
@@
 		(property
 			"Reference"
-			"R7004"
+			"R9004"
 			(at 168.808 111.76 0)
 			(effects
@@
 				(path
 					"/c2797150-7a6e-556a-82f5-fdda13c31368/4d664980-e58b-5403-9b49-c54d6ca52225"
-					(reference "R7004")
+					(reference "R9004")
 					(unit 1)
 				)
@@
 		(property
 			"Reference"
-			"C7004"
+			"C9004"
 			(at 182.728 119.38 0)
 			(effects
@@
 				(path
 					"/c2797150-7a6e-556a-82f5-fdda13c31368/4d664980-e58b-5403-9b49-c54d6ca52225"
-					(reference "C7004")
+					(reference "C9004")
 					(unit 1)
 				)
@@
 		(property
 			"Reference"
-			"C7005"
+			"C9005"
 			(at 192.888 127 0)
 			(effects
@@
 				(path
 					"/c2797150-7a6e-556a-82f5-fdda13c31368/4d664980-e58b-5403-9b49-c54d6ca52225"
-					(reference "C7005")
+					(reference "C9005")
 					(unit 1)
 				)
@@
 		(property
 			"Reference"
-			"#PWR7001"
+			"#PWR9001"
 			(at 184.15 101.6 0)
 			(effects
@@
 				(path
 					"/c2797150-7a6e-556a-82f5-fdda13c31368/4d664980-e58b-5403-9b49-c54d6ca52225"
-					(reference "#PWR7001")
+					(reference "#PWR9001")
 					(unit 1)
 				)
@@
 		(property
 			"Reference"
-			"#PWR7002"
+			"#PWR9002"
 			(at 189.23 129.54 0)
 			(effects
@@
 				(path
 					"/c2797150-7a6e-556a-82f5-fdda13c31368/4d664980-e58b-5403-9b49-c54d6ca52225"
-					(reference "#PWR7002")
+					(reference "#PWR9002")
 					(unit 1)
 				)
@@
 		(property
 			"Reference"
-			"#PWR7003"
+			"#PWR9003"
 			(at 92.71 142.24 0)
 			(effects
@@
 				(path
 					"/c2797150-7a6e-556a-82f5-fdda13c31368/4d664980-e58b-5403-9b49-c54d6ca52225"
-					(reference "#PWR7003")
+					(reference "#PWR9003")
 					(unit 1)
 				)
@@
 		(property
 			"Reference"
-			"#FLG7001"
+			"#FLG9001"
 			(at 92.71 139.7 0)
 			(effects
@@
 				(path
 					"/c2797150-7a6e-556a-82f5-fdda13c31368/4d664980-e58b-5403-9b49-c54d6ca52225"
-					(reference "#FLG7001")
-					(unit 1)
-				)
+					(reference "#FLG9001")
+					(unit 1)
+				)

Commit message: audit fixes: QWIIC ESD on its own sheet + firmware I2C-map completeness
Acting on a multi-agent adversarial re-audit of the 28-sheet board. Each
finding was independently re-verified before action — two confident "HIGH"
findings were FALSE POSITIVES whose proposed fixes would have INTRODUCED bugs,
and are documented-rejected, not applied:

  * "DSHP04 switches in parallel" — wrong. The footprint pads prove the pairing
    by physical opposition (switch n = pads n & 9-n): switch 1 = pads 1&8 is the
    only one on EN_AUX; the other even pins (2/4/6) are NC, identical to the
    proven bringup_rails SW6 idiom. The proposed "fix" (pins 1+2) wires two
    DIFFERENT switches and would leave EN_AUX permanently pulled down — the rail
    could never enable.
  * "PCA9306 EN floats when AUX is off" — wrong. A 100k to a 0 V rail pulls EN
    to 0 V (disabled), which is exactly TI's recommended "isolate when the gated
    side is unpowered" connection. No float.

REAL findings actioned:

1. QWIIC connector lacked ESD (every other external connector has it). Moved the
   QWIIC out of board_services onto its own sheet board_qwiic (the carrier's
   connectors-get-their-own-sheet idiom — rj45_connector, usb_uart_connector)
   and added a USBLC6-2SC6 low-cap ESD array at the connector (1<->6 / 3<->4
   passthrough, clamp ref +3V3_AUX). The dedicated sheet also keeps both sheets
   sparse enough for the rail-stub router. board_services drops to 9 parts.

2. schgen/firmware.py loaded only 7 sheets, so the SC-firmware contract + its
   I2C address-collision check were BLIND to the new devices. Added board_aux/
   board_services to SOURCES and three address rows: FMC-EEPROM 0x50, ID-EEPROM
   0x51 (DERIVED from the 24AA025E48 A1/A0 straps, so a mis-strap to 0x50 now
   trips the collision check against the FMC EEPROM), RTC 0x52. The firmware can
   now address the EUI-48 MAC EEPROM and the RTC. 114 -> 117 #defines.

3. board_services docstring clarified (EEPROM/RTC are on the PCA9306-i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
Parts:
- renumbered C9001 to C10001, C9002 to C10002, C9003 to C10003, C9004 to C10004, C9005 to C10005, R9001 to R10001, R9002 to R10002, R9003 to R10003, R9004 to R10004, T9001 to T10001
Changed lines of the file:
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@@
 		(property
 			"Reference"
-			"T9001"
+			"T10001"
 			(at 175.26 51.435 0)
 			(effects
@@
 				(path
 					"/c2797150-7a6e-556a-82f5-fdda13c31368/4d664980-e58b-5403-9b49-c54d6ca52225"
-					(reference "T9001")
+					(reference "T10001")
 					(unit 1)
 				)
@@
 		(property
 			"Reference"
-			"R9001"
+			"R10001"
 			(at 123.088 111.76 0)
 			(effects
@@
 				(path
 					"/c2797150-7a6e-556a-82f5-fdda13c31368/4d664980-e58b-5403-9b49-c54d6ca52225"
-					(reference "R9001")
+					(reference "R10001")
 					(unit 1)
 				)
@@
 		(property
 			"Reference"
-			"C9001"
+			"C10001"
 			(at 137.008 119.38 0)
 			(effects
@@
 				(path
 					"/c2797150-7a6e-556a-82f5-fdda13c31368/4d664980-e58b-5403-9b49-c54d6ca52225"
-					(reference "C9001")
+					(reference "C10001")
 					(unit 1)
 				)
@@
 		(property
 			"Reference"
-			"R9002"
+			"R10002"
 			(at 138.328 111.76 0)
 			(effects
@@
 				(path
 					"/c2797150-7a6e-556a-82f5-fdda13c31368/4d664980-e58b-5403-9b49-c54d6ca52225"
-					(reference "R9002")
+					(reference "R10002")
 					(unit 1)
 				)
@@
 		(property
 			"Reference"
-			"C9002"
+			"C10002"
 			(at 152.249 119.38 0)
 			(effects
@@
 				(path
 					"/c2797150-7a6e-556a-82f5-fdda13c31368/4d664980-e58b-5403-9b49-c54d6ca52225"
-					(reference "C9002")
+					(reference "C10002")
 					(unit 1)
 				)
@@
 		(property
 			"Reference"
-			"R9003"
+			"R10003"
 			(at 153.567 111.76 0)
 			(effects
@@
 				(path
 					"/c2797150-7a6e-556a-82f5-fdda13c31368/4d664980-e58b-5403-9b49-c54d6ca52225"
-					(reference "R9003")
+					(reference "R10003")
 					(unit 1)
 				)
@@
 		(property
 			"Reference"
-			"C9003"
+			"C10003"
 			(at 167.488 119.38 0)
 			(effects
@@
 				(path
 					"/c2797150-7a6e-556a-82f5-fdda13c31368/4d664980-e58b-5403-9b49-c54d6ca52225"
-					(reference "C9003")
+					(reference "C10003")
 					(unit 1)
 				)
@@
 		(property
 			"Reference"
-			"R9004"
+			"R10004"
 			(at 168.808 111.76 0)
 			(effects
@@
 				(path
 					"/c2797150-7a6e-556a-82f5-fdda13c31368/4d664980-e58b-5403-9b49-c54d6ca52225"
-					(reference "R9004")
+					(reference "R10004")
 					(unit 1)
 				)
@@
 		(property
 			"Reference"
-			"C9004"
+			"C10004"
 			(at 182.728 119.38 0)
 			(effects
@@
 				(path
 					"/c2797150-7a6e-556a-82f5-fdda13c31368/4d664980-e58b-5403-9b49-c54d6ca52225"
-					(reference "C9004")
+					(reference "C10004")
 					(unit 1)
 				)
@@
 		(property
 			"Reference"
-			"C9005"
+			"C10005"
 			(at 192.888 127 0)
 			(effects
@@
 				(path
 					"/c2797150-7a6e-556a-82f5-fdda13c31368/4d664980-e58b-5403-9b49-c54d6ca52225"
-					(reference "C9005")
+					(reference "C10005")
 					(unit 1)
 				)
@@
 		(property
 			"Reference"
-			"#PWR9001"
+			"#PWR10001"
 			(at 184.15 101.6 0)
 			(effects
@@
 				(path
 					"/c2797150-7a6e-556a-82f5-fdda13c31368/4d664980-e58b-5403-9b49-c54d6ca52225"
-					(reference "#PWR9001")
+					(reference "#PWR10001")
 					(unit 1)
 				)
@@
 		(property
 			"Reference"
-			"#PWR9002"
+			"#PWR10002"
 			(at 189.23 129.54 0)
 			(effects
@@
 				(path
 					"/c2797150-7a6e-556a-82f5-fdda13c31368/4d664980-e58b-5403-9b49-c54d6ca52225"
-					(reference "#PWR9002")
+					(reference "#PWR10002")
 					(unit 1)
 				)
@@
 		(property
 			"Reference"
-			"#PWR9003"
+			"#PWR10003"
 			(at 92.71 142.24 0)
 			(effects
@@
 				(path
 					"/c2797150-7a6e-556a-82f5-fdda13c31368/4d664980-e58b-5403-9b49-c54d6ca52225"
-					(reference "#PWR9003")
+					(reference "#PWR10003")
 					(unit 1)
 				)
@@
 		(property
 			"Reference"
-			"#FLG9001"
+			"#FLG10001"
 			(at 92.71 139.7 0)
 			(effects
@@
 				(path
 					"/c2797150-7a6e-556a-82f5-fdda13c31368/4d664980-e58b-5403-9b49-c54d6ca52225"
-					(reference "#FLG9001")
-					(unit 1)
-				)
+					(reference "#FLG10001")
+					(unit 1)
+				)
