File: carrier/schematic/power_mon.kicad_sch (KiCad schematic)
At the start: 10 parts, among them U1601 INA3221AIRGVR, U1602 INA3221AIRGVR

Commit message: audit-fix(engine): harvest F1-F7,F9 — gate hardening + leak + guards
F1 selftest now exercises the VISUAL gate against geometry mutants (wire-cross
+ text-over-wire) — proven to bite (was never run on a mutant before).
F2 visual_gate catches different-net wire T-touch / butt-join shorts.
F3 netlist_gate no longer leaks tmp .net files (was 2671 stale).
F4 board uniquify guards the stride (widened 100->1000) against ref collision.
F5 hier-mode sheets now re-run through the per-sheet netlist gate.
F6 dead clause dropped; F7 stale zynq_eda docstring fixed; F9 eager inline-pin
validation. Source copied verbatim from the audit-fix worktree (6 files, proven
untouched on origin since its base); board regenerated fresh. All gates green,
selftest geo-mutants killed by the visual gate, goldens 23/23, m1_rc PASS.

Co-Authored-By: Claude Fable 5 <noreply@anthropic.com>
Parts:
- renumbered C1601 to C16001, C1602 to C16002, C1603 to C16003, R1601 to R16001, RS1601 to RS16001, RS1602 to RS16002, RS1603 to RS16003, RS1604 to RS16004, U1601 to U16001, U1602 to U16002

Commit message: DEF-6: netlist the HDMI-RX TMDS sink termination (new hdmi_rx_term sheet)
The HDMI-RX sink REQUIRES 8x 49.9 ohm/pair-to-AVCC source termination (a
7-series HR bank does not self-terminate TMDS_33) — without it HDMI RX simply
does not work. It had been carried for rounds as a docstring-only MANDATORY
layout note because the resistors belong at the FPGA-bank (receiver) end and
the connector-sheet placer could not anchor an off-sheet AVCC trunk. DEF-6
promotes it to a real, netlisted, gate-checked, BOM-counted network on its own
sheet hdmi_rx_term.py: 8x 49.9R (C114625) from HDMI_RX_{D2,D1,D0,CLK}_{P,N} to
AVCC = +3V3 (bank-33 VCCO IS +3V3, the correct TMDS_33 termination voltage).

LINK PASS (the 3-way TMDS merge with hdmi_rx + som_j2), powertree accepts the
~64 mA termination load, render clean (LAW 1), board PASS 26 sheets,
deterministic, selftest 44/44, m1 PASS.

The 100n/1u AVCC bypass is a documented layout note (not netlisted): the
placer has no pattern for a rail-to-rail cap with no host part on an IC-less
sheet (a tracked placer-robustness follow-up). Inserting the sheet
alphabetically re-stamps the per-sheet reference uniquification of the 15
downstream sheets (U11001->U12001 etc.) — deterministic, a known consequence
of the position-based hierarchy numbering.

Co-Authored-By: Claude Opus 4.8 <noreply@anthropic.com>
Parts:
- renumbered C16001 to C17001, C16002 to C17002, C16003 to C17003, R16001 to R17001, RS16001 to RS17001, RS16002 to RS17002, RS16003 to RS17003, RS16004 to RS17004, U16001 to U17001, U16002 to U17002

Commit message: genpolish: TITLE-1 — populate the schematic title block on every sheet
Every sheet rendered a blank Title/Rev/Date — the clearest 'not a real
schematic' tell. emit() now writes a (title_block ...) after the paper node:
title = the sheet circuit's title, company "Zynq SoM Carrier", and a
"<sheet> — generated by schgen (do not hand-edit)" comment. NO date node — a
wall-clock date would break byte-determinism; the content-derived fields keep
every rebuild identical. Verified on A4 (usb_pd) and the dense A3 (power): the
block fills the standard reserved corner with zero drawing overlap. All 26
sheets, goldens re-blessed, board PASS + deterministic, selftest 53/53, m1,
pytest 147.

Co-Authored-By: Claude Opus 4.8 <noreply@anthropic.com>
Other:
- company: (none) -> Zynq SoM Carrier
- title: (none) -> Rail telemetry: 2x INA3221 + shunts (I2C 0x40/41)
Changed lines of the file:
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@@
 	(generator_version "1.0")
 	(paper "A4")
+	(title_block
+		(title "Rail telemetry: 2x INA3221 + shunts (I2C 0x40/41)")
+		(company "Zynq SoM Carrier")
+		(comment 1 "power_mon — generated by schgen (do not hand-edit)")
+	)
 	(wire
 		(pts

Commit message: board: four board-management HW blocks on a manually-gated +3V3_AUX (BOARDHW)
The four services the carrier was missing — all behind ONE manual power enable
(C1) on two new sheets split so neither defeats the placer's rail-stub router:

  board_aux       — the gate + I2C isolator (infrastructure)
  board_services  — ID-EEPROM + RTC + watchdog + QWIIC (the peripherals)

WHAT LANDED
  * 24AA025E48 (C129895)  ID-EEPROM with a factory EUI-48 **MAC** for the
      LAN8720/RJ45 — strapped 0x51 (0x50 is the FMC EEPROM).
  * RV-3028-C7 (C3019759) I2C RTC, integrated DTCXO (no crystal), CR1220 coin
      cell (KH-CR1220-2) with auto-switchover, 0x52.
  * TPS3823-33 (C7719)    supervisor + windowed watchdog.
  * ZX-SH1.0-4PWT (C7430446)  QWIIC / STEMMA-QT expansion (gated 3V3 + the
      isolated AUX I2C).
  * SY6280 gate + DSHP04 DIP + PCA9306 isolator complete the infrastructure.

CONSTRAINTS (the user's three standing requirements)
  C1 manual enable "like the previous": +3V3_AUX is a SY6280 load switch whose
     EN is a default-OFF DSHP04 DIP (100k pulldown) — the same gated-module
     idiom, self-contained so it touches none of the dense rail/EN sheets.
  C2 "no watchdog reset during power-up": THREE independent guards — (1) the
     supervisor's VDD is the default-OFF +3V3_AUX, so it is UNPOWERED through
     power-up; (2) the TPS3823 disables its watchdog while WDI floats, and WDI
     is driven only by the PL (WATCHDOG_KICK, Hi-Z until the fabric is up); (3)
     RESET# is a firmware-mediated PL EVENT (J3.31), never a rail/POR line.
  C3 Zynq-agnostic: the only SoM-side signals (the 2 watchdog lines) ride PL
     bank-35 IO by their contract net names (IO_L16_N/P_35 -> J3.29/31); xdc.py
     emits the constraints live — nothing hard-codes the Zynq part.

LAW 0 (electrical integrity): the peripherals sit on the GATED rail but their
bus is the always-on STM32_I2C2 management bus. A PCA9306 bridges them with EN
tied to +3V3_AUX, so the switch OPENS whenever the rail is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
Parts:
- renumbered C17001 to C19001, C17002 to C19002, C17003 to C19003, R17001 to R19001, RS17001 to RS19001, RS17002 to RS19002, RS17003 to RS19003, RS17004 to RS19004, U17001 to U19001, U17002 to U19002

Commit message: audit fixes: QWIIC ESD on its own sheet + firmware I2C-map completeness
Acting on a multi-agent adversarial re-audit of the 28-sheet board. Each
finding was independently re-verified before action — two confident "HIGH"
findings were FALSE POSITIVES whose proposed fixes would have INTRODUCED bugs,
and are documented-rejected, not applied:

  * "DSHP04 switches in parallel" — wrong. The footprint pads prove the pairing
    by physical opposition (switch n = pads n & 9-n): switch 1 = pads 1&8 is the
    only one on EN_AUX; the other even pins (2/4/6) are NC, identical to the
    proven bringup_rails SW6 idiom. The proposed "fix" (pins 1+2) wires two
    DIFFERENT switches and would leave EN_AUX permanently pulled down — the rail
    could never enable.
  * "PCA9306 EN floats when AUX is off" — wrong. A 100k to a 0 V rail pulls EN
    to 0 V (disabled), which is exactly TI's recommended "isolate when the gated
    side is unpowered" connection. No float.

REAL findings actioned:

1. QWIIC connector lacked ESD (every other external connector has it). Moved the
   QWIIC out of board_services onto its own sheet board_qwiic (the carrier's
   connectors-get-their-own-sheet idiom — rj45_connector, usb_uart_connector)
   and added a USBLC6-2SC6 low-cap ESD array at the connector (1<->6 / 3<->4
   passthrough, clamp ref +3V3_AUX). The dedicated sheet also keeps both sheets
   sparse enough for the rail-stub router. board_services drops to 9 parts.

2. schgen/firmware.py loaded only 7 sheets, so the SC-firmware contract + its
   I2C address-collision check were BLIND to the new devices. Added board_aux/
   board_services to SOURCES and three address rows: FMC-EEPROM 0x50, ID-EEPROM
   0x51 (DERIVED from the 24AA025E48 A1/A0 straps, so a mis-strap to 0x50 now
   trips the collision check against the FMC EEPROM), RTC 0x52. The firmware can
   now address the EUI-48 MAC EEPROM and the RTC. 114 -> 117 #defines.

3. board_services docstring clarified (EEPROM/RTC are on the PCA9306-i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
Parts:
- renumbered C19001 to C20001, C19002 to C20002, C19003 to C20003, R19001 to R20001, RS19001 to RS20001, RS19002 to RS20002, RS19003 to RS20003, RS19004 to RS20004, U19001 to U20001, U19002 to U20002
