File: carrier/schematic/usb_uart_connector.kicad_sch (KiCad schematic)
At the start: 5 parts, among them J23001 TYPE-C-31-M-12, U23001 USBLC6-2SC6

Commit message: DEF-6: netlist the HDMI-RX TMDS sink termination (new hdmi_rx_term sheet)
The HDMI-RX sink REQUIRES 8x 49.9 ohm/pair-to-AVCC source termination (a
7-series HR bank does not self-terminate TMDS_33) — without it HDMI RX simply
does not work. It had been carried for rounds as a docstring-only MANDATORY
layout note because the resistors belong at the FPGA-bank (receiver) end and
the connector-sheet placer could not anchor an off-sheet AVCC trunk. DEF-6
promotes it to a real, netlisted, gate-checked, BOM-counted network on its own
sheet hdmi_rx_term.py: 8x 49.9R (C114625) from HDMI_RX_{D2,D1,D0,CLK}_{P,N} to
AVCC = +3V3 (bank-33 VCCO IS +3V3, the correct TMDS_33 termination voltage).

LINK PASS (the 3-way TMDS merge with hdmi_rx + som_j2), powertree accepts the
~64 mA termination load, render clean (LAW 1), board PASS 26 sheets,
deterministic, selftest 44/44, m1 PASS.

The 100n/1u AVCC bypass is a documented layout note (not netlisted): the
placer has no pattern for a rail-to-rail cap with no host part on an IC-less
sheet (a tracked placer-robustness follow-up). Inserting the sheet
alphabetically re-stamps the per-sheet reference uniquification of the 15
downstream sheets (U11001->U12001 etc.) — deterministic, a known consequence
of the position-based hierarchy numbering.

Co-Authored-By: Claude Opus 4.8 <noreply@anthropic.com>
Parts:
- renumbered C23001 to C24001, J23001 to J24001, R23001 to R24001, R23002 to R24002, U23001 to U24001
Changed lines of the file:
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@@
 		(property
 			"Reference"
-			"U23001"
+			"U24001"
 			(at 106.68 86.995 0)
 			(effects
@@
 				(path
 					"/c2797150-7a6e-556a-82f5-fdda13c31368/f0a0a553-8394-53c5-ba0e-a6588fc1d256"
-					(reference "U23001")
+					(reference "U24001")
 					(unit 1)
 				)
@@
 		(property
 			"Reference"
-			"J23001"
+			"J24001"
 			(at 186.69 69.215 0)
 			(effects
@@
 				(path
 					"/c2797150-7a6e-556a-82f5-fdda13c31368/f0a0a553-8394-53c5-ba0e-a6588fc1d256"
-					(reference "J23001")
+					(reference "J24001")
 					(unit 1)
 				)
@@
 		(property
 			"Reference"
-			"R23002"
+			"R24002"
 			(at 155.043 83.82 0)
 			(effects
@@
 				(path
 					"/c2797150-7a6e-556a-82f5-fdda13c31368/f0a0a553-8394-53c5-ba0e-a6588fc1d256"
-					(reference "R23002")
+					(reference "R24002")
 					(unit 1)
 				)
@@
 		(property
 			"Reference"
-			"R23001"
+			"R24001"
 			(at 205.843 99.06 0)
 			(effects
@@
 				(path
 					"/c2797150-7a6e-556a-82f5-fdda13c31368/f0a0a553-8394-53c5-ba0e-a6588fc1d256"
-					(reference "R23001")
+					(reference "R24001")
 					(unit 1)
 				)
@@
 		(property
 			"Reference"
-			"C23001"
+			"C24001"
 			(at 192.889 120.65 0)
 			(effects
@@
 				(path
 					"/c2797150-7a6e-556a-82f5-fdda13c31368/f0a0a553-8394-53c5-ba0e-a6588fc1d256"
-					(reference "C23001")
+					(reference "C24001")
 					(unit 1)
 				)
@@
 		(property
 			"Reference"
-			"#PWR23001"
+			"#PWR24001"
 			(at 115.57 91.44 0)
 			(effects
@@
 				(path
 					"/c2797150-7a6e-556a-82f5-fdda13c31368/f0a0a553-8394-53c5-ba0e-a6588fc1d256"
-					(reference "#PWR23001")
+					(reference "#PWR24001")
 					(unit 1)
 				)
@@
 		(property
 			"Reference"
-			"#PWR23002"
+			"#PWR24002"
 			(at 163.83 86.36 0)
 			(effects
@@
 				(path
 					"/c2797150-7a6e-556a-82f5-fdda13c31368/f0a0a553-8394-53c5-ba0e-a6588fc1d256"
-					(reference "#PWR23002")
+					(reference "#PWR24002")
 					(unit 1)
 				)
@@
 		(property
 			"Reference"
-			"#PWR23003"
+			"#PWR24003"
 			(at 152.4 78.74 0)
 			(effects
@@
 				(path
 					"/c2797150-7a6e-556a-82f5-fdda13c31368/f0a0a553-8394-53c5-ba0e-a6588fc1d256"
-					(reference "#PWR23003")
+					(reference "#PWR24003")
 					(unit 1)
 				)
@@
 		(property
 			"Reference"
-			"#PWR23004"
+			"#PWR24004"
 			(at 203.2 101.6 0)
 			(effects
@@
 				(path
 					"/c2797150-7a6e-556a-82f5-fdda13c31368/f0a0a553-8394-53c5-ba0e-a6588fc1d256"
-					(reference "#PWR23004")
+					(reference "#PWR24004")
 					(unit 1)
 				)
@@
 		(property
 			"Reference"
-			"#PWR23005"
+			"#PWR24005"
 			(at 182.88 58.42 0)
 			(effects
@@
 				(path
 					"/c2797150-7a6e-556a-82f5-fdda13c31368/f0a0a553-8394-53c5-ba0e-a6588fc1d256"
-					(reference "#PWR23005")
+					(reference "#PWR24005")
 					(unit 1)
 				)
@@
 		(property
 			"Reference"
-			"#PWR23006"
+			"#PWR24006"
 			(at 189.23 123.19 0)
 			(effects
@@
 				(path
 					"/c2797150-7a6e-556a-82f5-fdda13c31368/f0a0a553-8394-53c5-ba0e-a6588fc1d256"
-					(reference "#PWR23006")
-					(unit 1)
-				)
+					(reference "#PWR24006")
+					(unit 1)
+				)

Commit message: genpolish: TITLE-1 — populate the schematic title block on every sheet
Every sheet rendered a blank Title/Rev/Date — the clearest 'not a real
schematic' tell. emit() now writes a (title_block ...) after the paper node:
title = the sheet circuit's title, company "Zynq SoM Carrier", and a
"<sheet> — generated by schgen (do not hand-edit)" comment. NO date node — a
wall-clock date would break byte-determinism; the content-derived fields keep
every rebuild identical. Verified on A4 (usb_pd) and the dense A3 (power): the
block fills the standard reserved corner with zero drawing overlap. All 26
sheets, goldens re-blessed, board PASS + deterministic, selftest 53/53, m1,
pytest 147.

Co-Authored-By: Claude Opus 4.8 <noreply@anthropic.com>
Other:
- company: (none) -> Zynq SoM Carrier
- title: (none) -> USB-C UFP console port -> CP2102N
Changed lines of the file:
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@@
 	(generator_version "1.0")
 	(paper "A4")
+	(title_block
+		(title "USB-C UFP console port -> CP2102N")
+		(company "Zynq SoM Carrier")
+		(comment 1 "usb_uart_connector — generated by schgen (do not hand-edit)")
+	)
 	(wire
 		(pts

Commit message: board: four board-management HW blocks on a manually-gated +3V3_AUX (BOARDHW)
The four services the carrier was missing — all behind ONE manual power enable
(C1) on two new sheets split so neither defeats the placer's rail-stub router:

  board_aux       — the gate + I2C isolator (infrastructure)
  board_services  — ID-EEPROM + RTC + watchdog + QWIIC (the peripherals)

WHAT LANDED
  * 24AA025E48 (C129895)  ID-EEPROM with a factory EUI-48 **MAC** for the
      LAN8720/RJ45 — strapped 0x51 (0x50 is the FMC EEPROM).
  * RV-3028-C7 (C3019759) I2C RTC, integrated DTCXO (no crystal), CR1220 coin
      cell (KH-CR1220-2) with auto-switchover, 0x52.
  * TPS3823-33 (C7719)    supervisor + windowed watchdog.
  * ZX-SH1.0-4PWT (C7430446)  QWIIC / STEMMA-QT expansion (gated 3V3 + the
      isolated AUX I2C).
  * SY6280 gate + DSHP04 DIP + PCA9306 isolator complete the infrastructure.

CONSTRAINTS (the user's three standing requirements)
  C1 manual enable "like the previous": +3V3_AUX is a SY6280 load switch whose
     EN is a default-OFF DSHP04 DIP (100k pulldown) — the same gated-module
     idiom, self-contained so it touches none of the dense rail/EN sheets.
  C2 "no watchdog reset during power-up": THREE independent guards — (1) the
     supervisor's VDD is the default-OFF +3V3_AUX, so it is UNPOWERED through
     power-up; (2) the TPS3823 disables its watchdog while WDI floats, and WDI
     is driven only by the PL (WATCHDOG_KICK, Hi-Z until the fabric is up); (3)
     RESET# is a firmware-mediated PL EVENT (J3.31), never a rail/POR line.
  C3 Zynq-agnostic: the only SoM-side signals (the 2 watchdog lines) ride PL
     bank-35 IO by their contract net names (IO_L16_N/P_35 -> J3.29/31); xdc.py
     emits the constraints live — nothing hard-codes the Zynq part.

LAW 0 (electrical integrity): the peripherals sit on the GATED rail but their
bus is the always-on STM32_I2C2 management bus. A PCA9306 bridges them with EN
tied to +3V3_AUX, so the switch OPENS whenever the rail is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
Parts:
- renumbered C24001 to C26001, J24001 to J26001, R24001 to R26001, R24002 to R26002, U24001 to U26001
Changed lines of the file:
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@@
 		(property
 			"Reference"
-			"U24001"
+			"U26001"
 			(at 106.68 86.995 0)
 			(effects
@@
 				(path
 					"/c2797150-7a6e-556a-82f5-fdda13c31368/f0a0a553-8394-53c5-ba0e-a6588fc1d256"
-					(reference "U24001")
+					(reference "U26001")
 					(unit 1)
 				)
@@
 		(property
 			"Reference"
-			"J24001"
+			"J26001"
 			(at 186.69 69.215 0)
 			(effects
@@
 				(path
 					"/c2797150-7a6e-556a-82f5-fdda13c31368/f0a0a553-8394-53c5-ba0e-a6588fc1d256"
-					(reference "J24001")
+					(reference "J26001")
 					(unit 1)
 				)
@@
 		(property
 			"Reference"
-			"R24002"
+			"R26002"
 			(at 155.043 83.82 0)
 			(effects
@@
 				(path
 					"/c2797150-7a6e-556a-82f5-fdda13c31368/f0a0a553-8394-53c5-ba0e-a6588fc1d256"
-					(reference "R24002")
+					(reference "R26002")
 					(unit 1)
 				)
@@
 		(property
 			"Reference"
-			"R24001"
+			"R26001"
 			(at 205.843 99.06 0)
 			(effects
@@
 				(path
 					"/c2797150-7a6e-556a-82f5-fdda13c31368/f0a0a553-8394-53c5-ba0e-a6588fc1d256"
-					(reference "R24001")
+					(reference "R26001")
 					(unit 1)
 				)
@@
 		(property
 			"Reference"
-			"C24001"
+			"C26001"
 			(at 192.889 120.65 0)
 			(effects
@@
 				(path
 					"/c2797150-7a6e-556a-82f5-fdda13c31368/f0a0a553-8394-53c5-ba0e-a6588fc1d256"
-					(reference "C24001")
+					(reference "C26001")
 					(unit 1)
 				)
@@
 		(property
 			"Reference"
-			"#PWR24001"
+			"#PWR26001"
 			(at 115.57 91.44 0)
 			(effects
@@
 				(path
 					"/c2797150-7a6e-556a-82f5-fdda13c31368/f0a0a553-8394-53c5-ba0e-a6588fc1d256"
-					(reference "#PWR24001")
+					(reference "#PWR26001")
 					(unit 1)
 				)
@@
 		(property
 			"Reference"
-			"#PWR24002"
+			"#PWR26002"
 			(at 163.83 86.36 0)
 			(effects
@@
 				(path
 					"/c2797150-7a6e-556a-82f5-fdda13c31368/f0a0a553-8394-53c5-ba0e-a6588fc1d256"
-					(reference "#PWR24002")
+					(reference "#PWR26002")
 					(unit 1)
 				)
@@
 		(property
 			"Reference"
-			"#PWR24003"
+			"#PWR26003"
 			(at 152.4 78.74 0)
 			(effects
@@
 				(path
 					"/c2797150-7a6e-556a-82f5-fdda13c31368/f0a0a553-8394-53c5-ba0e-a6588fc1d256"
-					(reference "#PWR24003")
+					(reference "#PWR26003")
 					(unit 1)
 				)
@@
 		(property
 			"Reference"
-			"#PWR24004"
+			"#PWR26004"
 			(at 203.2 101.6 0)
 			(effects
@@
 				(path
 					"/c2797150-7a6e-556a-82f5-fdda13c31368/f0a0a553-8394-53c5-ba0e-a6588fc1d256"
-					(reference "#PWR24004")
+					(reference "#PWR26004")
 					(unit 1)
 				)
@@
 		(property
 			"Reference"
-			"#PWR24005"
+			"#PWR26005"
 			(at 182.88 58.42 0)
 			(effects
@@
 				(path
 					"/c2797150-7a6e-556a-82f5-fdda13c31368/f0a0a553-8394-53c5-ba0e-a6588fc1d256"
-					(reference "#PWR24005")
+					(reference "#PWR26005")
 					(unit 1)
 				)
@@
 		(property
 			"Reference"
-			"#PWR24006"
+			"#PWR26006"
 			(at 189.23 123.19 0)
 			(effects
@@
 				(path
 					"/c2797150-7a6e-556a-82f5-fdda13c31368/f0a0a553-8394-53c5-ba0e-a6588fc1d256"
-					(reference "#PWR24006")
-					(unit 1)
-				)
+					(reference "#PWR26006")
+					(unit 1)
+				)

Commit message: audit fixes: QWIIC ESD on its own sheet + firmware I2C-map completeness
Acting on a multi-agent adversarial re-audit of the 28-sheet board. Each
finding was independently re-verified before action — two confident "HIGH"
findings were FALSE POSITIVES whose proposed fixes would have INTRODUCED bugs,
and are documented-rejected, not applied:

  * "DSHP04 switches in parallel" — wrong. The footprint pads prove the pairing
    by physical opposition (switch n = pads n & 9-n): switch 1 = pads 1&8 is the
    only one on EN_AUX; the other even pins (2/4/6) are NC, identical to the
    proven bringup_rails SW6 idiom. The proposed "fix" (pins 1+2) wires two
    DIFFERENT switches and would leave EN_AUX permanently pulled down — the rail
    could never enable.
  * "PCA9306 EN floats when AUX is off" — wrong. A 100k to a 0 V rail pulls EN
    to 0 V (disabled), which is exactly TI's recommended "isolate when the gated
    side is unpowered" connection. No float.

REAL findings actioned:

1. QWIIC connector lacked ESD (every other external connector has it). Moved the
   QWIIC out of board_services onto its own sheet board_qwiic (the carrier's
   connectors-get-their-own-sheet idiom — rj45_connector, usb_uart_connector)
   and added a USBLC6-2SC6 low-cap ESD array at the connector (1<->6 / 3<->4
   passthrough, clamp ref +3V3_AUX). The dedicated sheet also keeps both sheets
   sparse enough for the rail-stub router. board_services drops to 9 parts.

2. schgen/firmware.py loaded only 7 sheets, so the SC-firmware contract + its
   I2C address-collision check were BLIND to the new devices. Added board_aux/
   board_services to SOURCES and three address rows: FMC-EEPROM 0x50, ID-EEPROM
   0x51 (DERIVED from the 24AA025E48 A1/A0 straps, so a mis-strap to 0x50 now
   trips the collision check against the FMC EEPROM), RTC 0x52. The firmware can
   now address the EUI-48 MAC EEPROM and the RTC. 114 -> 117 #defines.

3. board_services docstring clarified (EEPROM/RTC are on the PCA9306-i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
Parts:
- renumbered C26001 to C27001, J26001 to J27001, R26001 to R27001, R26002 to R27002, U26001 to U27001
Changed lines of the file:
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@@
 		(property
 			"Reference"
-			"U26001"
+			"U27001"
 			(at 106.68 86.995 0)
 			(effects
@@
 				(path
 					"/c2797150-7a6e-556a-82f5-fdda13c31368/f0a0a553-8394-53c5-ba0e-a6588fc1d256"
-					(reference "U26001")
+					(reference "U27001")
 					(unit 1)
 				)
@@
 		(property
 			"Reference"
-			"J26001"
+			"J27001"
 			(at 186.69 69.215 0)
 			(effects
@@
 				(path
 					"/c2797150-7a6e-556a-82f5-fdda13c31368/f0a0a553-8394-53c5-ba0e-a6588fc1d256"
-					(reference "J26001")
+					(reference "J27001")
 					(unit 1)
 				)
@@
 		(property
 			"Reference"
-			"R26002"
+			"R27002"
 			(at 155.043 83.82 0)
 			(effects
@@
 				(path
 					"/c2797150-7a6e-556a-82f5-fdda13c31368/f0a0a553-8394-53c5-ba0e-a6588fc1d256"
-					(reference "R26002")
+					(reference "R27002")
 					(unit 1)
 				)
@@
 		(property
 			"Reference"
-			"R26001"
+			"R27001"
 			(at 205.843 99.06 0)
 			(effects
@@
 				(path
 					"/c2797150-7a6e-556a-82f5-fdda13c31368/f0a0a553-8394-53c5-ba0e-a6588fc1d256"
-					(reference "R26001")
+					(reference "R27001")
 					(unit 1)
 				)
@@
 		(property
 			"Reference"
-			"C26001"
+			"C27001"
 			(at 192.889 120.65 0)
 			(effects
@@
 				(path
 					"/c2797150-7a6e-556a-82f5-fdda13c31368/f0a0a553-8394-53c5-ba0e-a6588fc1d256"
-					(reference "C26001")
+					(reference "C27001")
 					(unit 1)
 				)
@@
 		(property
 			"Reference"
-			"#PWR26001"
+			"#PWR27001"
 			(at 115.57 91.44 0)
 			(effects
@@
 				(path
 					"/c2797150-7a6e-556a-82f5-fdda13c31368/f0a0a553-8394-53c5-ba0e-a6588fc1d256"
-					(reference "#PWR26001")
+					(reference "#PWR27001")
 					(unit 1)
 				)
@@
 		(property
 			"Reference"
-			"#PWR26002"
+			"#PWR27002"
 			(at 163.83 86.36 0)
 			(effects
@@
 				(path
 					"/c2797150-7a6e-556a-82f5-fdda13c31368/f0a0a553-8394-53c5-ba0e-a6588fc1d256"
-					(reference "#PWR26002")
+					(reference "#PWR27002")
 					(unit 1)
 				)
@@
 		(property
 			"Reference"
-			"#PWR26003"
+			"#PWR27003"
 			(at 152.4 78.74 0)
 			(effects
@@
 				(path
 					"/c2797150-7a6e-556a-82f5-fdda13c31368/f0a0a553-8394-53c5-ba0e-a6588fc1d256"
-					(reference "#PWR26003")
+					(reference "#PWR27003")
 					(unit 1)
 				)
@@
 		(property
 			"Reference"
-			"#PWR26004"
+			"#PWR27004"
 			(at 203.2 101.6 0)
 			(effects
@@
 				(path
 					"/c2797150-7a6e-556a-82f5-fdda13c31368/f0a0a553-8394-53c5-ba0e-a6588fc1d256"
-					(reference "#PWR26004")
+					(reference "#PWR27004")
 					(unit 1)
 				)
@@
 		(property
 			"Reference"
-			"#PWR26005"
+			"#PWR27005"
 			(at 182.88 58.42 0)
 			(effects
@@
 				(path
 					"/c2797150-7a6e-556a-82f5-fdda13c31368/f0a0a553-8394-53c5-ba0e-a6588fc1d256"
-					(reference "#PWR26005")
+					(reference "#PWR27005")
 					(unit 1)
 				)
@@
 		(property
 			"Reference"
-			"#PWR26006"
+			"#PWR27006"
 			(at 189.23 123.19 0)
 			(effects
@@
 				(path
 					"/c2797150-7a6e-556a-82f5-fdda13c31368/f0a0a553-8394-53c5-ba0e-a6588fc1d256"
-					(reference "#PWR26006")
-					(unit 1)
-				)
+					(reference "#PWR27006")
+					(unit 1)
+				)
