File: carrier/schematic/bringup_en.kicad_sch (KiCad schematic)
At the start: 15 parts, among them U101 SN74LVC1G08, U102 SN74LVC1G08, U103 SN74LVC1G08

Commit message: audit-fix(engine): harvest F1-F7,F9 — gate hardening + leak + guards
F1 selftest now exercises the VISUAL gate against geometry mutants (wire-cross
+ text-over-wire) — proven to bite (was never run on a mutant before).
F2 visual_gate catches different-net wire T-touch / butt-join shorts.
F3 netlist_gate no longer leaks tmp .net files (was 2671 stale).
F4 board uniquify guards the stride (widened 100->1000) against ref collision.
F5 hier-mode sheets now re-run through the per-sheet netlist gate.
F6 dead clause dropped; F7 stale zynq_eda docstring fixed; F9 eager inline-pin
validation. Source copied verbatim from the audit-fix worktree (6 files, proven
untouched on origin since its base); board regenerated fresh. All gates green,
selftest geo-mutants killed by the visual gate, goldens 23/23, m1_rc PASS.

Co-Authored-By: Claude Fable 5 <noreply@anthropic.com>
Parts:
- renumbered C101 to C1001, C102 to C1002, C103 to C1003, R101 to R1001, R102 to R1002, R103 to R1003, R104 to R1004, R105 to R1005, R106 to R1006, TP101 to TP1001, TP102 to TP1002, TP103 to TP1003, U101 to U1001, U102 to U1002, U103 to U1003

Commit message: genpolish: TITLE-1 — populate the schematic title block on every sheet
Every sheet rendered a blank Title/Rev/Date — the clearest 'not a real
schematic' tell. emit() now writes a (title_block ...) after the paper node:
title = the sheet circuit's title, company "Zynq SoM Carrier", and a
"<sheet> — generated by schgen (do not hand-edit)" comment. NO date node — a
wall-clock date would break byte-determinism; the content-derived fields keep
every rebuild identical. Verified on A4 (usb_pd) and the dense A3 (power): the
block fills the standard reserved corner with zero drawing overlap. All 26
sheets, goldens re-blessed, board PASS + deterministic, selftest 53/53, m1,
pytest 147.

Co-Authored-By: Claude Opus 4.8 <noreply@anthropic.com>
Other:
- company: (none) -> Zynq SoM Carrier
- title: (none) -> Bring-up EN cells: 3x SN74LVC1G08 rail DIP-AND-override
Changed lines of the file:
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@@
 	(generator_version "1.0")
 	(paper "A4")
+	(title_block
+		(title "Bring-up EN cells: 3x SN74LVC1G08 rail DIP-AND-override")
+		(company "Zynq SoM Carrier")
+		(comment 1 "bringup_en — generated by schgen (do not hand-edit)")
+	)
 	(wire
 		(pts

Commit message: board: four board-management HW blocks on a manually-gated +3V3_AUX (BOARDHW)
The four services the carrier was missing — all behind ONE manual power enable
(C1) on two new sheets split so neither defeats the placer's rail-stub router:

  board_aux       — the gate + I2C isolator (infrastructure)
  board_services  — ID-EEPROM + RTC + watchdog + QWIIC (the peripherals)

WHAT LANDED
  * 24AA025E48 (C129895)  ID-EEPROM with a factory EUI-48 **MAC** for the
      LAN8720/RJ45 — strapped 0x51 (0x50 is the FMC EEPROM).
  * RV-3028-C7 (C3019759) I2C RTC, integrated DTCXO (no crystal), CR1220 coin
      cell (KH-CR1220-2) with auto-switchover, 0x52.
  * TPS3823-33 (C7719)    supervisor + windowed watchdog.
  * ZX-SH1.0-4PWT (C7430446)  QWIIC / STEMMA-QT expansion (gated 3V3 + the
      isolated AUX I2C).
  * SY6280 gate + DSHP04 DIP + PCA9306 isolator complete the infrastructure.

CONSTRAINTS (the user's three standing requirements)
  C1 manual enable "like the previous": +3V3_AUX is a SY6280 load switch whose
     EN is a default-OFF DSHP04 DIP (100k pulldown) — the same gated-module
     idiom, self-contained so it touches none of the dense rail/EN sheets.
  C2 "no watchdog reset during power-up": THREE independent guards — (1) the
     supervisor's VDD is the default-OFF +3V3_AUX, so it is UNPOWERED through
     power-up; (2) the TPS3823 disables its watchdog while WDI floats, and WDI
     is driven only by the PL (WATCHDOG_KICK, Hi-Z until the fabric is up); (3)
     RESET# is a firmware-mediated PL EVENT (J3.31), never a rail/POR line.
  C3 Zynq-agnostic: the only SoM-side signals (the 2 watchdog lines) ride PL
     bank-35 IO by their contract net names (IO_L16_N/P_35 -> J3.29/31); xdc.py
     emits the constraints live — nothing hard-codes the Zynq part.

LAW 0 (electrical integrity): the peripherals sit on the GATED rail but their
bus is the always-on STM32_I2C2 management bus. A PCA9306 bridges them with EN
tied to +3V3_AUX, so the switch OPENS whenever the rail is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
Parts:
- renumbered C1001 to C3001, C1002 to C3002, C1003 to C3003, R1001 to R3001, R1002 to R3002, R1003 to R3003, R1004 to R3004, R1005 to R3005, R1006 to R3006, TP1001 to TP3001, TP1002 to TP3002, TP1003 to TP3003, U1001 to U3001, U1002 to U3002, U1003 to U3003

Commit message: audit fixes: QWIIC ESD on its own sheet + firmware I2C-map completeness
Acting on a multi-agent adversarial re-audit of the 28-sheet board. Each
finding was independently re-verified before action — two confident "HIGH"
findings were FALSE POSITIVES whose proposed fixes would have INTRODUCED bugs,
and are documented-rejected, not applied:

  * "DSHP04 switches in parallel" — wrong. The footprint pads prove the pairing
    by physical opposition (switch n = pads n & 9-n): switch 1 = pads 1&8 is the
    only one on EN_AUX; the other even pins (2/4/6) are NC, identical to the
    proven bringup_rails SW6 idiom. The proposed "fix" (pins 1+2) wires two
    DIFFERENT switches and would leave EN_AUX permanently pulled down — the rail
    could never enable.
  * "PCA9306 EN floats when AUX is off" — wrong. A 100k to a 0 V rail pulls EN
    to 0 V (disabled), which is exactly TI's recommended "isolate when the gated
    side is unpowered" connection. No float.

REAL findings actioned:

1. QWIIC connector lacked ESD (every other external connector has it). Moved the
   QWIIC out of board_services onto its own sheet board_qwiic (the carrier's
   connectors-get-their-own-sheet idiom — rj45_connector, usb_uart_connector)
   and added a USBLC6-2SC6 low-cap ESD array at the connector (1<->6 / 3<->4
   passthrough, clamp ref +3V3_AUX). The dedicated sheet also keeps both sheets
   sparse enough for the rail-stub router. board_services drops to 9 parts.

2. schgen/firmware.py loaded only 7 sheets, so the SC-firmware contract + its
   I2C address-collision check were BLIND to the new devices. Added board_aux/
   board_services to SOURCES and three address rows: FMC-EEPROM 0x50, ID-EEPROM
   0x51 (DERIVED from the 24AA025E48 A1/A0 straps, so a mis-strap to 0x50 now
   trips the collision check against the FMC EEPROM), RTC 0x52. The firmware can
   now address the EUI-48 MAC EEPROM and the RTC. 114 -> 117 #defines.

3. board_services docstring clarified (EEPROM/RTC are on the PCA9306-i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
Parts:
- renumbered C3001 to C4001, C3002 to C4002, C3003 to C4003, R3001 to R4001, R3002 to R4002, R3003 to R4003, R3004 to R4004, R3005 to R4005, R3006 to R4006, TP3001 to TP4001, TP3002 to TP4002, TP3003 to TP4003, U3001 to U4001, U3002 to U4002, U3003 to U4003
Changed lines of the file:
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@@
 		(property
 			"Reference"
-			"U3001"
+			"U4001"
 			(at 115.548 51.435 0)
 			(effects
@@
 				(path
 					"/c2797150-7a6e-556a-82f5-fdda13c31368/9b6d3467-85dc-5090-91f7-911c52154366"
-					(reference "U3001")
+					(reference "U4001")
 					(unit 1)
 				)
@@
 		(property
 			"Reference"
-			"R3001"
+			"R4001"
 			(at 92.812 48.26 0)
 			(effects
@@
 				(path
 					"/c2797150-7a6e-556a-82f5-fdda13c31368/9b6d3467-85dc-5090-91f7-911c52154366"
-					(reference "R3001")
+					(reference "R4001")
 					(unit 1)
 				)
@@
 		(property
 			"Reference"
-			"R3002"
+			"R4002"
 			(at 67.412 48.26 0)
 			(effects
@@
 				(path
 					"/c2797150-7a6e-556a-82f5-fdda13c31368/9b6d3467-85dc-5090-91f7-911c52154366"
-					(reference "R3002")
+					(reference "R4002")
 					(unit 1)
 				)
@@
 		(property
 			"Reference"
-			"U3002"
+			"U4002"
 			(at 227.308 51.435 0)
 			(effects
@@
 				(path
 					"/c2797150-7a6e-556a-82f5-fdda13c31368/9b6d3467-85dc-5090-91f7-911c52154366"
-					(reference "U3002")
+					(reference "U4002")
 					(unit 1)
 				)
@@
 		(property
 			"Reference"
-			"R3003"
+			"R4003"
 			(at 204.572 48.26 0)
 			(effects
@@
 				(path
 					"/c2797150-7a6e-556a-82f5-fdda13c31368/9b6d3467-85dc-5090-91f7-911c52154366"
-					(reference "R3003")
+					(reference "R4003")
 					(unit 1)
 				)
@@
 		(property
 			"Reference"
-			"R3004"
+			"R4004"
 			(at 179.173 48.26 0)
 			(effects
@@
 				(path
 					"/c2797150-7a6e-556a-82f5-fdda13c31368/9b6d3467-85dc-5090-91f7-911c52154366"
-					(reference "R3004")
+					(reference "R4004")
 					(unit 1)
 				)
@@
 		(property
 			"Reference"
-			"U3003"
+			"U4003"
 			(at 115.548 86.995 0)
 			(effects
@@
 				(path
 					"/c2797150-7a6e-556a-82f5-fdda13c31368/9b6d3467-85dc-5090-91f7-911c52154366"
-					(reference "U3003")
+					(reference "U4003")
 					(unit 1)
 				)
@@
 		(property
 			"Reference"
-			"R3005"
+			"R4005"
 			(at 92.812 83.82 0)
 			(effects
@@
 				(path
 					"/c2797150-7a6e-556a-82f5-fdda13c31368/9b6d3467-85dc-5090-91f7-911c52154366"
-					(reference "R3005")
+					(reference "R4005")
 					(unit 1)
 				)
@@
 		(property
 			"Reference"
-			"R3006"
+			"R4006"
 			(at 67.412 83.82 0)
 			(effects
@@
 				(path
 					"/c2797150-7a6e-556a-82f5-fdda13c31368/9b6d3467-85dc-5090-91f7-911c52154366"
-					(reference "R3006")
+					(reference "R4006")
 					(unit 1)
 				)
@@
 		(property
 			"Reference"
-			"C3001"
+			"C4001"
 			(at 78.589 120.65 0)
 			(effects
@@
 				(path
 					"/c2797150-7a6e-556a-82f5-fdda13c31368/9b6d3467-85dc-5090-91f7-911c52154366"
-					(reference "C3001")
+					(reference "C4001")
 					(unit 1)
 				)
@@
 		(property
 			"Reference"
-			"C3002"
+			"C4002"
 			(at 88.749 120.65 0)
 			(effects
@@
 				(path
 					"/c2797150-7a6e-556a-82f5-fdda13c31368/9b6d3467-85dc-5090-91f7-911c52154366"
-					(reference "C3002")
+					(reference "C4002")
 					(unit 1)
 				)
@@
 		(property
 			"Reference"
-			"C3003"
+			"C4003"
 			(at 98.909 120.65 0)
 			(effects
@@
 				(path
 					"/c2797150-7a6e-556a-82f5-fdda13c31368/9b6d3467-85dc-5090-91f7-911c52154366"
-					(reference "C3003")
+					(reference "C4003")
 					(unit 1)
 				)
@@
 		(property
 			"Reference"
-			"TP3001"
+			"TP4001"
 			(at 47.442 155.702 0)
 			(effects
@@
 				(path
 					"/c2797150-7a6e-556a-82f5-fdda13c31368/9b6d3467-85dc-5090-91f7-911c52154366"
-					(reference "TP3001")
+					(reference "TP4001")
 					(unit 1)
 				)
@@
 		(property
 			"Reference"
-			"TP3002"
+			"TP4002"
 			(at 61.412 155.702 0)
 			(effects
@@
 				(path
 					"/c2797150-7a6e-556a-82f5-fdda13c31368/9b6d3467-85dc-5090-91f7-911c52154366"
-					(reference "TP3002")
+					(reference "TP4002")
 					(unit 1)
 				)
@@
 		(property
 			"Reference"
-			"TP3003"
+			"TP4003"
 			(at 75.382 155.702 0)
 			(effects
@@
 				(path
 					"/c2797150-7a6e-556a-82f5-fdda13c31368/9b6d3467-85dc-5090-91f7-911c52154366"
-					(reference "TP3003")
+					(reference "TP4003")
 					(unit 1)
 				)
@@
 		(property
 			"Reference"
-			"#PWR3001"
+			"#PWR4001"
 			(at 90.17 43.18 0)
 			(effects
@@
 				(path
 					"/c2797150-7a6e-556a-82f5-fdda13c31368/9b6d3467-85dc-5090-91f7-911c52154366"
-					(reference "#PWR3001")
+					(reference "#PWR4001")
 					(unit 1)
 				)
@@
 		(property
 			"Reference"
-			"#PWR3002"
+			"#PWR4002"
 			(at 64.77 43.18 0)
 			(effects
@@
 				(path
 					"/c2797150-7a6e-556a-82f5-fdda13c31368/9b6d3467-85dc-5090-91f7-911c52154366"
-					(reference "#PWR3002")
+					(reference "#PWR4002")
 					(unit 1)
 				)
@@
 		(property
 			"Reference"
-			"#PWR3003"
+			"#PWR4003"
 			(at 113.03 43.18 0)
 			(effects
@@
 				(path
 					"/c2797150-7a6e-556a-82f5-fdda13c31368/9b6d3467-85dc-5090-91f7-911c52154366"
-					(reference "#PWR3003")
+					(reference "#PWR4003")
 					(unit 1)
 				)
@@
 		(property
 			"Reference"
-			"#PWR3004"
+			"#PWR4004"
 			(at 113.03 68.58 0)
 			(effects
@@
 				(path
 					"/c2797150-7a6e-556a-82f5-fdda13c31368/9b6d3467-85dc-5090-91f7-911c52154366"
-					(reference "#PWR3004")
+					(reference "#PWR4004")
 					(unit 1)
 				)
@@
 		(property
 			"Reference"
-			"#PWR3005"
+			"#PWR4005"
 			(at 201.93 43.18 0)
 			(effects
@@
 				(path
 					"/c2797150-7a6e-556a-82f5-fdda13c31368/9b6d3467-85dc-5090-91f7-911c52154366"
-					(reference "#PWR3005")
+					(reference "#PWR4005")
 					(unit 1)
 				)
@@
 		(property
 			"Reference"
-			"#PWR3006"
+			"#PWR4006"
 			(at 176.53 43.18 0)
 			(effects
@@
 				(path
 					"/c2797150-7a6e-556a-82f5-fdda13c31368/9b6d3467-85dc-5090-91f7-911c52154366"
-					(reference "#PWR3006")
+					(reference "#PWR4006")
 					(unit 1)
 				)
@@
 		(property
 			"Reference"
-			"#PWR3007"
+			"#PWR4007"
 			(at 224.79 43.18 0)
 			(effects
@@
 				(path
 					"/c2797150-7a6e-556a-82f5-fdda13c31368/9b6d3467-85dc-5090-91f7-911c52154366"
-					(reference "#PWR3007")
+					(reference "#PWR4007")
 					(unit 1)
 				)
@@
 		(property
 			"Reference"
-			"#PWR3008"
+			"#PWR4008"
 			(at 224.79 68.58 0)
 			(effects
@@
 				(path
 					"/c2797150-7a6e-556a-82f5-fdda13c31368/9b6d3467-85dc-5090-91f7-911c52154366"
-					(reference "#PWR3008")
+					(reference "#PWR4008")
 					(unit 1)
 				)
@@
 		(property
 			"Reference"
-			"#PWR3009"
+			"#PWR4009"
 			(at 90.17 78.74 0)
 			(effects
@@
 				(path
 					"/c2797150-7a6e-556a-82f5-fdda13c31368/9b6d3467-85dc-5090-91f7-911c52154366"
-					(reference "#PWR3009")
+					(reference "#PWR4009")
 					(unit 1)
 				)
@@
 		(property
 			"Reference"
-			"#PWR3010"
+			"#PWR4010"
 			(at 64.77 78.74 0)
 			(effects
@@
 				(path
 					"/c2797150-7a6e-556a-82f5-fdda13c31368/9b6d3467-85dc-5090-91f7-911c52154366"
-					(reference "#PWR3010")
+					(reference "#PWR4010")
 					(unit 1)
 				)
@@
 		(property
 			"Reference"
-			"#PWR3011"
+			"#PWR4011"
 			(at 113.03 78.74 0)
 			(effects
@@
 				(path
 					"/c2797150-7a6e-556a-82f5-fdda13c31368/9b6d3467-85dc-5090-91f7-911c52154366"
-					(reference "#PWR3011")
+					(reference "#PWR4011")
 					(unit 1)
 				)
@@
 		(property
 			"Reference"
-			"#PWR3012"
+			"#PWR4012"
 			(at 113.03 104.14 0)
 			(effects
@@
 				(path
 					"/c2797150-7a6e-556a-82f5-fdda13c31368/9b6d3467-85dc-5090-91f7-911c52154366"
-					(reference "#PWR3012")
+					(reference "#PWR4012")
 					(unit 1)
 				)
@@
 		(property
 			"Reference"
-			"#PWR3013"
+			"#PWR4013"
 			(at 74.93 123.19 0)
 			(effects
@@
 				(path
 					"/c2797150-7a6e-556a-82f5-fdda13c31368/9b6d3467-85dc-5090-91f7-911c52154366"
-					(reference "#PWR3013")
+					(reference "#PWR4013")
 					(unit 1)
 				)
@@
 		(property
 			"Reference"
-			"#PWR3014"
+			"#PWR4014"
 			(at 85.09 123.19 0)
 			(effects
@@
 				(path
 					"/c2797150-7a6e-556a-82f5-fdda13c31368/9b6d3467-85dc-5090-91f7-911c52154366"
-					(reference "#PWR3014")
+					(reference "#PWR4014")
 					(unit 1)
 				)
@@
 		(property
 			"Reference"
-			"#PWR3015"
+			"#PWR4015"
 			(at 95.25 123.19 0)
 			(effects
@@
 				(path
 					"/c2797150-7a6e-556a-82f5-fdda13c31368/9b6d3467-85dc-5090-91f7-911c52154366"
-					(reference "#PWR3015")
+					(reference "#PWR4015")
 					(unit 1)
 				)
@@
 		(property
 			"Reference"
-			"#PWR3016"
+			"#PWR4016"
 			(at 85.09 113.03 0)
 			(effects
@@
 				(path
 					"/c2797150-7a6e-556a-82f5-fdda13c31368/9b6d3467-85dc-5090-91f7-911c52154366"
-					(reference "#PWR3016")
-					(unit 1)
-				)
+					(reference "#PWR4016")
+					(unit 1)
+				)

Commit message: bom: sourcing risk+cost report + C1591->C14663 (Extended->Basic 100n)
Stream F — live JLCPCB/LCSC sourcing pass over all 95 distinct BOM parts.

Report: carrier/manufacturing/SOURCING.md — per-part stock / Basic-vs-Extended
/ unit price / risk + flagged second sources, and a rollup (94 parts post-swap,
64 Extended of which 2 Preferred -> 62 feeder fees = ~$186, 15 parts <5k stock,
6 procurement-critical <300). Data from the JLCPCB parts API (live).

Applied swap (only clean Basic drop-in on the board): 100 nF 0603 decoupling
C1591 (Samsung CL10B104KB8NNNC, Extended, 2.08M) -> C14663 (YAGEO
CC0603KRX7R9BB104, Basic, 17.8M). IDENTICAL 100nF/50V/X7R/+-10%/0603, same
footprint+symbol -> netlist & render byte-identical; ratings.py already carries
C14663 with matching ratings. Merges 71 Extended + 12 existing-Basic positions
onto one 83-piece Basic line: removes one Extended feeder fee, cheaper unit,
8.5x more stock.

Everything else is REPORT-ONLY: every other Extended part is
Extended-by-necessity (no JLC-Basic equivalent — precise E96 values, specialty
ICs/connectors) or has only a footprint-mismatched / MPN-ambiguous alternate.
Also flagged (not fixed): C25750 ("40.2k" power:R1) currently resolves on LCSC
to a 120k 0402 part — a data-integrity bug; recommend C12447 after intent check.

Gates: part-rules PASS (132 checks, 0 findings); board PASS (33 sheets, golden
renders 33/33 match, DRC 0); selftest 59/59; m1_rc PASS; pytest 219 passed.
BOM regen deterministic (md5 stable).

Co-Authored-By: Claude Opus 4.8 <noreply@anthropic.com>
Parts:
- C4001, C4002, C4003: LCSC C1591 -> C14663
Changed lines of the file:
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@@
 		(property
 			"LCSC"
-			"C1591"
+			"C14663"
 			(at 74.93 121.92 0)
 			(effects
@@
 		(property
 			"LCSC"
-			"C1591"
+			"C14663"
 			(at 85.09 121.92 0)
 			(effects
@@
 		(property
 			"LCSC"
-			"C1591"
+			"C14663"
 			(at 95.25 121.92 0)
 			(effects
