File: carrier/schematic/bringup_modules.kicad_sch (KiCad schematic)
At the start: 70 parts, among them U6001 SY6280AAC, U6002 SY6280AAC, U6003 SY6280AAC, U6004 SY6280AAC, U6005 SY6280AAC, U6006 SY6280AAC, U6007 SY6280AAC, U6008 SY6280AAC, U6009 SY6280AAC, U6010 SY6280AAC

Commit message: bom: sourcing risk+cost report + C1591->C14663 (Extended->Basic 100n)
Stream F — live JLCPCB/LCSC sourcing pass over all 95 distinct BOM parts.

Report: carrier/manufacturing/SOURCING.md — per-part stock / Basic-vs-Extended
/ unit price / risk + flagged second sources, and a rollup (94 parts post-swap,
64 Extended of which 2 Preferred -> 62 feeder fees = ~$186, 15 parts <5k stock,
6 procurement-critical <300). Data from the JLCPCB parts API (live).

Applied swap (only clean Basic drop-in on the board): 100 nF 0603 decoupling
C1591 (Samsung CL10B104KB8NNNC, Extended, 2.08M) -> C14663 (YAGEO
CC0603KRX7R9BB104, Basic, 17.8M). IDENTICAL 100nF/50V/X7R/+-10%/0603, same
footprint+symbol -> netlist & render byte-identical; ratings.py already carries
C14663 with matching ratings. Merges 71 Extended + 12 existing-Basic positions
onto one 83-piece Basic line: removes one Extended feeder fee, cheaper unit,
8.5x more stock.

Everything else is REPORT-ONLY: every other Extended part is
Extended-by-necessity (no JLC-Basic equivalent — precise E96 values, specialty
ICs/connectors) or has only a footprint-mismatched / MPN-ambiguous alternate.
Also flagged (not fixed): C25750 ("40.2k" power:R1) currently resolves on LCSC
to a 120k 0402 part — a data-integrity bug; recommend C12447 after intent check.

Gates: part-rules PASS (132 checks, 0 findings); board PASS (33 sheets, golden
renders 33/33 match, DRC 0); selftest 59/59; m1_rc PASS; pytest 219 passed.
BOM regen deterministic (md5 stable).

Co-Authored-By: Claude Opus 4.8 <noreply@anthropic.com>
Parts:
- C6001, C6002, C6003, C6004, C6005, C6006, C6007, C6008, C6009, C6010, C6011, C6012, C6013, C6014, C6015, C6016, C6017, C6018, C6019, C6020: LCSC C1591 -> C14663
Changed lines of the file:
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@@
 		(property
 			"LCSC"
-			"C1591"
+			"C14663"
 			(at 77.47 168.91 0)
 			(effects
@@
 		(property
 			"LCSC"
-			"C1591"
+			"C14663"
 			(at 87.63 168.91 0)
 			(effects
@@
 		(property
 			"LCSC"
-			"C1591"
+			"C14663"
 			(at 97.79 168.91 0)
 			(effects
@@
 		(property
 			"LCSC"
-			"C1591"
+			"C14663"
 			(at 107.95 168.91 0)
 			(effects
@@
 		(property
 			"LCSC"
-			"C1591"
+			"C14663"
 			(at 118.11 168.91 0)
 			(effects
@@
 		(property
 			"LCSC"
-			"C1591"
+			"C14663"
 			(at 128.27 168.91 0)
 			(effects
@@
 		(property
 			"LCSC"
-			"C1591"
+			"C14663"
 			(at 138.43 168.91 0)
 			(effects
@@
 		(property
 			"LCSC"
-			"C1591"
+			"C14663"
 			(at 149.86 168.91 0)
 			(effects
@@
 		(property
 			"LCSC"
-			"C1591"
+			"C14663"
 			(at 166.37 168.91 0)
 			(effects
@@
 		(property
 			"LCSC"
-			"C1591"
+			"C14663"
 			(at 180.34 168.91 0)
 			(effects
@@
 		(property
 			"LCSC"
-			"C1591"
+			"C14663"
 			(at 191.77 168.91 0)
 			(effects
@@
 		(property
 			"LCSC"
-			"C1591"
+			"C14663"
 			(at 203.2 168.91 0)
 			(effects
@@
 		(property
 			"LCSC"
-			"C1591"
+			"C14663"
 			(at 213.36 168.91 0)
 			(effects
@@
 		(property
 			"LCSC"
-			"C1591"
+			"C14663"
 			(at 223.52 168.91 0)
 			(effects
@@
 		(property
 			"LCSC"
-			"C1591"
+			"C14663"
 			(at 233.68 168.91 0)
 			(effects
@@
 		(property
 			"LCSC"
-			"C1591"
+			"C14663"
 			(at 243.84 168.91 0)
 			(effects
@@
 		(property
 			"LCSC"
-			"C1591"
+			"C14663"
 			(at 255.27 168.91 0)
 			(effects
@@
 		(property
 			"LCSC"
-			"C1591"
+			"C14663"
 			(at 270.51 168.91 0)
 			(effects
@@
 		(property
 			"LCSC"
-			"C1591"
+			"C14663"
 			(at 287.02 168.91 0)
 			(effects
@@
 		(property
 			"LCSC"
-			"C1591"
+			"C14663"
 			(at 299.72 168.91 0)
 			(effects
