File: carrier/schematic/board_aux.kicad_sch (KiCad schematic)
At the start: 17 parts, among them SW1001 DSHP04TSGER, U1001 SY6280AAC, U1002 PCA9306DCUR

Commit message: bom: sourcing risk+cost report + C1591->C14663 (Extended->Basic 100n)
Stream F — live JLCPCB/LCSC sourcing pass over all 95 distinct BOM parts.

Report: carrier/manufacturing/SOURCING.md — per-part stock / Basic-vs-Extended
/ unit price / risk + flagged second sources, and a rollup (94 parts post-swap,
64 Extended of which 2 Preferred -> 62 feeder fees = ~$186, 15 parts <5k stock,
6 procurement-critical <300). Data from the JLCPCB parts API (live).

Applied swap (only clean Basic drop-in on the board): 100 nF 0603 decoupling
C1591 (Samsung CL10B104KB8NNNC, Extended, 2.08M) -> C14663 (YAGEO
CC0603KRX7R9BB104, Basic, 17.8M). IDENTICAL 100nF/50V/X7R/+-10%/0603, same
footprint+symbol -> netlist & render byte-identical; ratings.py already carries
C14663 with matching ratings. Merges 71 Extended + 12 existing-Basic positions
onto one 83-piece Basic line: removes one Extended feeder fee, cheaper unit,
8.5x more stock.

Everything else is REPORT-ONLY: every other Extended part is
Extended-by-necessity (no JLC-Basic equivalent — precise E96 values, specialty
ICs/connectors) or has only a footprint-mismatched / MPN-ambiguous alternate.
Also flagged (not fixed): C25750 ("40.2k" power:R1) currently resolves on LCSC
to a 120k 0402 part — a data-integrity bug; recommend C12447 after intent check.

Gates: part-rules PASS (132 checks, 0 findings); board PASS (33 sheets, golden
renders 33/33 match, DRC 0); selftest 59/59; m1_rc PASS; pytest 219 passed.
BOM regen deterministic (md5 stable).

Co-Authored-By: Claude Opus 4.8 <noreply@anthropic.com>
Parts:
- C1001, C1002, C1003, C1004: LCSC C1591 -> C14663
Changed lines of the file:
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@@
 		(property
 			"LCSC"
-			"C1591"
+			"C14663"
 			(at 100.33 157.48 0)
 			(effects
@@
 		(property
 			"LCSC"
-			"C1591"
+			"C14663"
 			(at 116.84 157.48 0)
 			(effects
@@
 		(property
 			"LCSC"
-			"C1591"
+			"C14663"
 			(at 133.35 157.48 0)
 			(effects
@@
 		(property
 			"LCSC"
-			"C1591"
+			"C14663"
 			(at 149.86 157.48 0)
 			(effects

Commit message: fix(audit LOW): board_aux rail bulk cap + ethernet CT engineering-decision doc
- board_aux (implement): add a 10uF/25V (C15850) bulk hold-up cap on the gated
  +3V3_AUX rail at the SY6280 output — only a 100n was present and the DS
  recommends an output cap for the 200mA QWIIC load. Additive shunt (LAW-0 safe);
  .py + .cir + header updated; soft-start tolerates it. 538 footprints, BOARD PASS.
- ethernet CT (documented decision, not blind-implemented): the four chip-side
  magnetics centre taps stay open — the RTL8211F voltage-mode PHY self-biases
  (COMPLIANCE ETH-5 PASS). Realtek's CT->GND EMI cap is recorded as a DEFERRED
  EMC-tuning provision: this reusable magnetics library exposes only CHASSIS_GND
  (no signal GND), and CT-cap values are tuned against measured emissions — add at
  the EMC bring-up revision, not as a blind value in the library.

Verified: 148x137, DRC 0, BOARD PASS; board_aux + ethernet tests 34/34.

Co-Authored-By: Claude Opus 4.8 <noreply@anthropic.com>
Parts:
- added TP1003: AUX_I2C_SDA, TestPoint:TestPoint_Pad_D1.5mm, symbol Connector:TestPoint
- C1003: renamed from C1004; value 100n -> 10u; footprint Capacitor_SMD:C_0603_1608Metric -> Capacitor_SMD:C_0805_2012Metric; LCSC C14663 -> C15850
- C1004: renamed from D1001; value red -> 100n; footprint LED_SMD:LED_0603_1608Metric -> Capacitor_SMD:C_0603_1608Metric; symbol Device:LED -> Device:C; LCSC C2286 -> C14663
- D1001: renamed from R1003; value 330R -> red; footprint Resistor_SMD:R_0603_1608Metric -> LED_SMD:LED_0603_1608Metric; symbol Device:R -> Device:LED; LCSC C23138 -> C2286
- R1003: renamed from TP1001; value +3V3_AUX -> 330R; footprint TestPoint:TestPoint_Pad_D1.5mm -> Resistor_SMD:R_0603_1608Metric; symbol Connector:TestPoint -> Device:R; BOM exclude -> (none); LCSC (none) -> C23138
- TP1001: renamed from TP1002; value AUX_I2C_SCL -> +3V3_AUX
- TP1002: renamed from TP1003; value AUX_I2C_SDA -> AUX_I2C_SCL
- renumbered C1003 to C1005
Connections:
- net +3V3_AUX: now also C1005.1, D1001.2 (A), TP1001.1; no longer C1004.2 (A), R1003.1
- net +3V3_SC: now also C1004.1; no longer C1005.1
- net AUX_I2C_SCL: now also TP1002.1; no longer TP1001.1
- net AUX_I2C_SDA: now also TP1003.1; no longer TP1002.1
- net GND: now also C1004.2, R1003.2; no longer D1001.2
- net at D1001.1 (K): now also R1003.1; no longer C1004.1 (K)
Other:
- moved on the sheet: C1001, C1002, C1003, C1005, TP1001, TP1002
