File: carrier/schematic/som_j3.kicad_sch (KiCad schematic)
At the start: 1 part, among them J21003 DF40C-100DS-0.4V(51)

Commit message: board: four board-management HW blocks on a manually-gated +3V3_AUX (BOARDHW)
The four services the carrier was missing — all behind ONE manual power enable
(C1) on two new sheets split so neither defeats the placer's rail-stub router:

  board_aux       — the gate + I2C isolator (infrastructure)
  board_services  — ID-EEPROM + RTC + watchdog + QWIIC (the peripherals)

WHAT LANDED
  * 24AA025E48 (C129895)  ID-EEPROM with a factory EUI-48 **MAC** for the
      LAN8720/RJ45 — strapped 0x51 (0x50 is the FMC EEPROM).
  * RV-3028-C7 (C3019759) I2C RTC, integrated DTCXO (no crystal), CR1220 coin
      cell (KH-CR1220-2) with auto-switchover, 0x52.
  * TPS3823-33 (C7719)    supervisor + windowed watchdog.
  * ZX-SH1.0-4PWT (C7430446)  QWIIC / STEMMA-QT expansion (gated 3V3 + the
      isolated AUX I2C).
  * SY6280 gate + DSHP04 DIP + PCA9306 isolator complete the infrastructure.

CONSTRAINTS (the user's three standing requirements)
  C1 manual enable "like the previous": +3V3_AUX is a SY6280 load switch whose
     EN is a default-OFF DSHP04 DIP (100k pulldown) — the same gated-module
     idiom, self-contained so it touches none of the dense rail/EN sheets.
  C2 "no watchdog reset during power-up": THREE independent guards — (1) the
     supervisor's VDD is the default-OFF +3V3_AUX, so it is UNPOWERED through
     power-up; (2) the TPS3823 disables its watchdog while WDI floats, and WDI
     is driven only by the PL (WATCHDOG_KICK, Hi-Z until the fabric is up); (3)
     RESET# is a firmware-mediated PL EVENT (J3.31), never a rail/POR line.
  C3 Zynq-agnostic: the only SoM-side signals (the 2 watchdog lines) ride PL
     bank-35 IO by their contract net names (IO_L16_N/P_35 -> J3.29/31); xdc.py
     emits the constraints live — nothing hard-codes the Zynq part.

LAW 0 (electrical integrity): the peripherals sit on the GATED rail but their
bus is the always-on STM32_I2C2 management bus. A PCA9306 bridges them with EN
tied to +3V3_AUX, so the switch OPENS whenever the rail is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
Parts:
- renumbered J21003 to J23003
Changed lines of the file:
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@@
 		(property
 			"Reference"
-			"J21003"
+			"J23003"
 			(at 148.59 26.67 0)
 			(effects
@@
 				(path
 					"/c2797150-7a6e-556a-82f5-fdda13c31368/1a90d640-b359-59d8-a9ea-ed0f40ee4461"
-					(reference "J21003")
+					(reference "J23003")
 					(unit 1)
 				)
@@
 		(property
 			"Reference"
-			"#PWR21001"
+			"#PWR23001"
 			(at 133.35 25.4 0)
 			(effects
@@
 				(path
 					"/c2797150-7a6e-556a-82f5-fdda13c31368/1a90d640-b359-59d8-a9ea-ed0f40ee4461"
-					(reference "#PWR21001")
+					(reference "#PWR23001")
 					(unit 1)
 				)
@@
 		(property
 			"Reference"
-			"#PWR21002"
+			"#PWR23002"
 			(at 133.35 154.94 0)
 			(effects
@@
 				(path
 					"/c2797150-7a6e-556a-82f5-fdda13c31368/1a90d640-b359-59d8-a9ea-ed0f40ee4461"
-					(reference "#PWR21002")
+					(reference "#PWR23002")
 					(unit 1)
 				)
@@
 		(property
 			"Reference"
-			"#PWR21003"
+			"#PWR23003"
 			(at 83.82 149.86 0)
 			(effects
@@
 				(path
 					"/c2797150-7a6e-556a-82f5-fdda13c31368/1a90d640-b359-59d8-a9ea-ed0f40ee4461"
-					(reference "#PWR21003")
+					(reference "#PWR23003")
 					(unit 1)
 				)
@@
 		(property
 			"Reference"
-			"#PWR21004"
+			"#PWR23004"
 			(at 163.83 25.4 0)
 			(effects
@@
 				(path
 					"/c2797150-7a6e-556a-82f5-fdda13c31368/1a90d640-b359-59d8-a9ea-ed0f40ee4461"
-					(reference "#PWR21004")
+					(reference "#PWR23004")
 					(unit 1)
 				)
@@
 		(property
 			"Reference"
-			"#PWR21005"
+			"#PWR23005"
 			(at 213.36 154.94 0)
 			(effects
@@
 				(path
 					"/c2797150-7a6e-556a-82f5-fdda13c31368/1a90d640-b359-59d8-a9ea-ed0f40ee4461"
-					(reference "#PWR21005")
+					(reference "#PWR23005")
 					(unit 1)
 				)

Commit message: audit fixes: QWIIC ESD on its own sheet + firmware I2C-map completeness
Acting on a multi-agent adversarial re-audit of the 28-sheet board. Each
finding was independently re-verified before action — two confident "HIGH"
findings were FALSE POSITIVES whose proposed fixes would have INTRODUCED bugs,
and are documented-rejected, not applied:

  * "DSHP04 switches in parallel" — wrong. The footprint pads prove the pairing
    by physical opposition (switch n = pads n & 9-n): switch 1 = pads 1&8 is the
    only one on EN_AUX; the other even pins (2/4/6) are NC, identical to the
    proven bringup_rails SW6 idiom. The proposed "fix" (pins 1+2) wires two
    DIFFERENT switches and would leave EN_AUX permanently pulled down — the rail
    could never enable.
  * "PCA9306 EN floats when AUX is off" — wrong. A 100k to a 0 V rail pulls EN
    to 0 V (disabled), which is exactly TI's recommended "isolate when the gated
    side is unpowered" connection. No float.

REAL findings actioned:

1. QWIIC connector lacked ESD (every other external connector has it). Moved the
   QWIIC out of board_services onto its own sheet board_qwiic (the carrier's
   connectors-get-their-own-sheet idiom — rj45_connector, usb_uart_connector)
   and added a USBLC6-2SC6 low-cap ESD array at the connector (1<->6 / 3<->4
   passthrough, clamp ref +3V3_AUX). The dedicated sheet also keeps both sheets
   sparse enough for the rail-stub router. board_services drops to 9 parts.

2. schgen/firmware.py loaded only 7 sheets, so the SC-firmware contract + its
   I2C address-collision check were BLIND to the new devices. Added board_aux/
   board_services to SOURCES and three address rows: FMC-EEPROM 0x50, ID-EEPROM
   0x51 (DERIVED from the 24AA025E48 A1/A0 straps, so a mis-strap to 0x50 now
   trips the collision check against the FMC EEPROM), RTC 0x52. The firmware can
   now address the EUI-48 MAC EEPROM and the RTC. 114 -> 117 #defines.

3. board_services docstring clarified (EEPROM/RTC are on the PCA9306-i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
Parts:
- renumbered J23003 to J24003
Changed lines of the file:
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@@
 		(property
 			"Reference"
-			"J23003"
+			"J24003"
 			(at 148.59 26.67 0)
 			(effects
@@
 				(path
 					"/c2797150-7a6e-556a-82f5-fdda13c31368/1a90d640-b359-59d8-a9ea-ed0f40ee4461"
-					(reference "J23003")
+					(reference "J24003")
 					(unit 1)
 				)
@@
 		(property
 			"Reference"
-			"#PWR23001"
+			"#PWR24001"
 			(at 133.35 25.4 0)
 			(effects
@@
 				(path
 					"/c2797150-7a6e-556a-82f5-fdda13c31368/1a90d640-b359-59d8-a9ea-ed0f40ee4461"
-					(reference "#PWR23001")
+					(reference "#PWR24001")
 					(unit 1)
 				)
@@
 		(property
 			"Reference"
-			"#PWR23002"
+			"#PWR24002"
 			(at 133.35 154.94 0)
 			(effects
@@
 				(path
 					"/c2797150-7a6e-556a-82f5-fdda13c31368/1a90d640-b359-59d8-a9ea-ed0f40ee4461"
-					(reference "#PWR23002")
+					(reference "#PWR24002")
 					(unit 1)
 				)
@@
 		(property
 			"Reference"
-			"#PWR23003"
+			"#PWR24003"
 			(at 83.82 149.86 0)
 			(effects
@@
 				(path
 					"/c2797150-7a6e-556a-82f5-fdda13c31368/1a90d640-b359-59d8-a9ea-ed0f40ee4461"
-					(reference "#PWR23003")
+					(reference "#PWR24003")
 					(unit 1)
 				)
@@
 		(property
 			"Reference"
-			"#PWR23004"
+			"#PWR24004"
 			(at 163.83 25.4 0)
 			(effects
@@
 				(path
 					"/c2797150-7a6e-556a-82f5-fdda13c31368/1a90d640-b359-59d8-a9ea-ed0f40ee4461"
-					(reference "#PWR23004")
+					(reference "#PWR24004")
 					(unit 1)
 				)
@@
 		(property
 			"Reference"
-			"#PWR23005"
+			"#PWR24005"
 			(at 213.36 154.94 0)
 			(effects
@@
 				(path
 					"/c2797150-7a6e-556a-82f5-fdda13c31368/1a90d640-b359-59d8-a9ea-ed0f40ee4461"
-					(reference "#PWR23005")
+					(reference "#PWR24005")
 					(unit 1)
 				)

Commit message: buck U1 -> LMR33630 EP buck: power_som split + placer regulator-template generalization
LANDS the exposed-pad buck reselect (the whole point: U1 was a bare TSOT-23-6
TPS54302 with no thermal pad). U1 is now the LMR33630ADDAR (LCSC C841384): TI
SIMPLE SWITCHER, synchronous + internally compensated, 3.8-36 V / 3 A, HSOIC-8
PowerPAD with a REAL datasheet exposed pad, EP (pad 9) netted to GND. Uses the
KiCad STOCK symbol Regulator_Switching:LMR33640ADDA (same DDA pinout, proper
power_in VIN) + the faithful EP-bearing footprint — exactly the TPS54302/
AP2112K stock-symbol idiom. VFB 1.0 V -> 40.2k/10k FB divider = 5.02 V.

SHEET SPLIT (power -> power + power_som): the larger LMR33630 pushed the
4-converter power sheet past one A3 page. The +5V_SOM always-on stage (U4) is
the cleanly-separable unit (only +VIN/+5V_SOM/GND rails cross — they merge by
name; every signal net is internal) and moves to its own subsystem power_som.py.
An auto-paginator cannot split this sheet from the netlist alone (its regulators
chain-share input/output rails, so shared decoupling caps can't be assigned to a
stage); the human split assigns them explicitly. board LINK proves +5V_SOM
merges power_som<->som_j1 and +VIN across pd_input/power/power_mon/power_som.

PLACER GENERALIZATION (schgen/place.py, regulator template) so a richer buck
than the TPS54302's exact 6-pin pinout places — all verified byte-identical for
the 28 unchanged sheets (per-sheet), board gate PASS:
  - _detect_stages: a switch/output pin may be 'output' (LMR SW) not just
    'power_out' (TPS54302 SW); LDO branch stays strict to power_out.
  - _stage_row Edit 1+3: place an aux internal-LDO bias output (LMR VCC, pin 6)
    + its single bypass cap in its own left column (was the "U1_VCC islet, opens
    forbidden" open); emit ALL distinct bottom GND/EP points (not just the last);
    emit explicit NC markers for authored no-connects (the LMR open-collector PG
    pin 4 — was an ERC "Pin not connected").
  - _stage_row Edit 2: ro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
Parts:
- renumbered J24003 to J25003
Changed lines of the file:
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@@
 		(property
 			"Reference"
-			"J24003"
+			"J25003"
 			(at 148.59 26.67 0)
 			(effects
@@
 				(path
 					"/c2797150-7a6e-556a-82f5-fdda13c31368/1a90d640-b359-59d8-a9ea-ed0f40ee4461"
-					(reference "J24003")
+					(reference "J25003")
 					(unit 1)
 				)
@@
 		(property
 			"Reference"
-			"#PWR24001"
+			"#PWR25001"
 			(at 133.35 25.4 0)
 			(effects
@@
 				(path
 					"/c2797150-7a6e-556a-82f5-fdda13c31368/1a90d640-b359-59d8-a9ea-ed0f40ee4461"
-					(reference "#PWR24001")
+					(reference "#PWR25001")
 					(unit 1)
 				)
@@
 		(property
 			"Reference"
-			"#PWR24002"
+			"#PWR25002"
 			(at 133.35 154.94 0)
 			(effects
@@
 				(path
 					"/c2797150-7a6e-556a-82f5-fdda13c31368/1a90d640-b359-59d8-a9ea-ed0f40ee4461"
-					(reference "#PWR24002")
+					(reference "#PWR25002")
 					(unit 1)
 				)
@@
 		(property
 			"Reference"
-			"#PWR24003"
+			"#PWR25003"
 			(at 83.82 149.86 0)
 			(effects
@@
 				(path
 					"/c2797150-7a6e-556a-82f5-fdda13c31368/1a90d640-b359-59d8-a9ea-ed0f40ee4461"
-					(reference "#PWR24003")
+					(reference "#PWR25003")
 					(unit 1)
 				)
@@
 		(property
 			"Reference"
-			"#PWR24004"
+			"#PWR25004"
 			(at 163.83 25.4 0)
 			(effects
@@
 				(path
 					"/c2797150-7a6e-556a-82f5-fdda13c31368/1a90d640-b359-59d8-a9ea-ed0f40ee4461"
-					(reference "#PWR24004")
+					(reference "#PWR25004")
 					(unit 1)
 				)
@@
 		(property
 			"Reference"
-			"#PWR24005"
+			"#PWR25005"
 			(at 213.36 154.94 0)
 			(effects
@@
 				(path
 					"/c2797150-7a6e-556a-82f5-fdda13c31368/1a90d640-b359-59d8-a9ea-ed0f40ee4461"
-					(reference "#PWR24005")
+					(reference "#PWR25005")
 					(unit 1)
 				)

Commit message: feat: USB-JTAG/UART debug bridge (CH347T) + Pmod expansion (Stream C)
Two new feature sheets (board 30 -> 33):
- usb_jtag + usb_jtag_connector: a self-powered, isolated USB-JTAG/UART debug
  bridge. CH347T (chosen over FT2232H, whose 64-pin LQFP the placer cannot route)
  on its own USB-powered island (AP2112K-3.3 LDO, USBLC6 ESD, 8MHz xtal); JTAG
  isolated to the Zynq via an SN74LVC125 buffer with default-Hi-Z OE (100k pull +
  DIP) so the existing debug_boot header owns JTAG by default (zero contention,
  netlist-proven: ZYNQ_JTAG touches only the buffer). Can program a dead board.
- pmod_expansion: a Digilent Pmod (2x6, 3.3V) — 8 IO on verified-free bank-13 PL
  pins (via FUNCTION_MAP) + a manually-gated rail + TPD4E1U06 ESD.

Pin alloc verified free (XDC 146 -> 156, no double-claims). Regression green:
board 33 sheets, selftest 59/59, pytest 219. usb_jtag render inspected (LAW 1).

Co-Authored-By: Claude Opus 4.8 <noreply@anthropic.com>
Parts:
- renumbered J25003 to J26003
Changed lines of the file:
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@@
 		(property
 			"Reference"
-			"J25003"
+			"J26003"
 			(at 148.59 26.67 0)
 			(effects
@@
 				(path
 					"/c2797150-7a6e-556a-82f5-fdda13c31368/1a90d640-b359-59d8-a9ea-ed0f40ee4461"
-					(reference "J25003")
+					(reference "J26003")
 					(unit 1)
 				)
@@
 		(property
 			"Reference"
-			"#PWR25001"
+			"#PWR26001"
 			(at 133.35 25.4 0)
 			(effects
@@
 				(path
 					"/c2797150-7a6e-556a-82f5-fdda13c31368/1a90d640-b359-59d8-a9ea-ed0f40ee4461"
-					(reference "#PWR25001")
+					(reference "#PWR26001")
 					(unit 1)
 				)
@@
 		(property
 			"Reference"
-			"#PWR25002"
+			"#PWR26002"
 			(at 133.35 154.94 0)
 			(effects
@@
 				(path
 					"/c2797150-7a6e-556a-82f5-fdda13c31368/1a90d640-b359-59d8-a9ea-ed0f40ee4461"
-					(reference "#PWR25002")
+					(reference "#PWR26002")
 					(unit 1)
 				)
@@
 		(property
 			"Reference"
-			"#PWR25003"
+			"#PWR26003"
 			(at 83.82 149.86 0)
 			(effects
@@
 				(path
 					"/c2797150-7a6e-556a-82f5-fdda13c31368/1a90d640-b359-59d8-a9ea-ed0f40ee4461"
-					(reference "#PWR25003")
+					(reference "#PWR26003")
 					(unit 1)
 				)
@@
 		(property
 			"Reference"
-			"#PWR25004"
+			"#PWR26004"
 			(at 163.83 25.4 0)
 			(effects
@@
 				(path
 					"/c2797150-7a6e-556a-82f5-fdda13c31368/1a90d640-b359-59d8-a9ea-ed0f40ee4461"
-					(reference "#PWR25004")
+					(reference "#PWR26004")
 					(unit 1)
 				)
@@
 		(property
 			"Reference"
-			"#PWR25005"
+			"#PWR26005"
 			(at 213.36 154.94 0)
 			(effects
@@
 				(path
 					"/c2797150-7a6e-556a-82f5-fdda13c31368/1a90d640-b359-59d8-a9ea-ed0f40ee4461"
-					(reference "#PWR25005")
+					(reference "#PWR26005")
 					(unit 1)
 				)

Commit message: board_services: fix watchdog 3.3V->2.5V domain crossing — relocate WATCHDOG nets to a 3.3V bank (audit HIGH+MED)
The TPS3823-33 supervisor (U3, +3V3_AUX, 3.3V push-pull) drove WATCHDOG_RST_N +
WATCHDOG_KICK into Zynq bank 35 (VCCO=+2V5_VADJ): RESET# chronically forward-bit
the 2.5V input clamp diode (HIGH reliability), and the LVCMOS25 driver VOH ~2.1V
sat below the TPS3823 WDI VIH 2.31V (MED, kicks could miss).

Fix = Option A (relocate), keeping U3 on 3.3V: the TPS3823-33 MONITORS 3.3V
(VIT- 2.93V) so re-railing it to 2.5V would wedge it in reset — correctly
rejected. Moved both nets to spare bank-33 +3V3 (LVCMOS33) pins (J3.98 ball W20
RST_N, J3.96 ball W21 KICK) so they share U3's 3.3V domain: clamp gone (3.3V into
3.3V VCCO), WDI driven by LVCMOS33 VOH ~3.0V clears the 2.31V VIH.

- som_conn_gen.py: WATCHDOG_RST_N -> IO_L4_P_33, WATCHDOG_KICK -> IO_L4_N_33;
  + DO-NOT-LOAD guard comment for the on-SoM MIO VM0/VM1 straps.
- board_services.py: U3 binds the relocated nets; reset-RC waiver on the
  push-pull supervisor OUTPUT (rule not softened — LAW 4).
- XDC regenerated (LVCMOS33/bank33); manual.py + test_board_services.py updated.

Verify: LINK PASS (both nets bind board_services+som_j3); golden 33 match (only
board_services + som_j3 changed); BOARD PASS; selftest 61/61; board_services
pytest 17 passed. U3 VDD unchanged on +3V3_AUX.

Co-Authored-By: Claude Opus 4.8 <noreply@anthropic.com>
Connections:
- net IO_L4_N_33 renamed WATCHDOG_KICK
- net IO_L4_P_33 renamed WATCHDOG_RST_N
Changed lines of the file:
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@@
 	)
 	(hierarchical_label
-		"IO_L4_N_33"
+		"WATCHDOG_KICK"
 		(shape bidirectional)
 		(at 163.83 149.86 0)
@@
 	)
 	(hierarchical_label
-		"IO_L4_P_33"
+		"WATCHDOG_RST_N"
 		(shape bidirectional)
 		(at 185.42 152.4 0)
