File: carrier/schematic/usb_jtag.kicad_sch (KiCad schematic)
At the start: 19 parts, among them SW28001 DSHP04TSGER, U28001 CH347T, U28002 SN74LVC125ADR, U28004 AP2112K-3.3TRG1, Y28001 8MHz

Commit message: bom: sourcing risk+cost report + C1591->C14663 (Extended->Basic 100n)
Stream F — live JLCPCB/LCSC sourcing pass over all 95 distinct BOM parts.

Report: carrier/manufacturing/SOURCING.md — per-part stock / Basic-vs-Extended
/ unit price / risk + flagged second sources, and a rollup (94 parts post-swap,
64 Extended of which 2 Preferred -> 62 feeder fees = ~$186, 15 parts <5k stock,
6 procurement-critical <300). Data from the JLCPCB parts API (live).

Applied swap (only clean Basic drop-in on the board): 100 nF 0603 decoupling
C1591 (Samsung CL10B104KB8NNNC, Extended, 2.08M) -> C14663 (YAGEO
CC0603KRX7R9BB104, Basic, 17.8M). IDENTICAL 100nF/50V/X7R/+-10%/0603, same
footprint+symbol -> netlist & render byte-identical; ratings.py already carries
C14663 with matching ratings. Merges 71 Extended + 12 existing-Basic positions
onto one 83-piece Basic line: removes one Extended feeder fee, cheaper unit,
8.5x more stock.

Everything else is REPORT-ONLY: every other Extended part is
Extended-by-necessity (no JLC-Basic equivalent — precise E96 values, specialty
ICs/connectors) or has only a footprint-mismatched / MPN-ambiguous alternate.
Also flagged (not fixed): C25750 ("40.2k" power:R1) currently resolves on LCSC
to a 120k 0402 part — a data-integrity bug; recommend C12447 after intent check.

Gates: part-rules PASS (132 checks, 0 findings); board PASS (33 sheets, golden
renders 33/33 match, DRC 0); selftest 59/59; m1_rc PASS; pytest 219 passed.
BOM regen deterministic (md5 stable).

Co-Authored-By: Claude Opus 4.8 <noreply@anthropic.com>
Parts:
- C28003, C28004, C28007: LCSC C1591 -> C14663
Changed lines of the file:
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@@
 		(property
 			"LCSC"
-			"C1591"
+			"C14663"
 			(at 93.98 105.41 0)
 			(effects
@@
 		(property
 			"LCSC"
-			"C1591"
+			"C14663"
 			(at 104.14 105.41 0)
 			(effects
@@
 		(property
 			"LCSC"
-			"C1591"
+			"C14663"
 			(at 114.3 105.41 0)
 			(effects

Commit message: carrier: 4 confirmed datasheet-audit fixes (crystal CL, LED Vf, SY6280 Cin, LVC125 doc)
All four adversarially re-verified against the datasheet + schematic before
applying:

- usb_jtag-1 (crystal load caps): Y1 (KDS DSX321G, CL=12pF) had two 22pF load
  caps presenting ~15pF -> 8MHz pulled ~-50..-90ppm (outside ±20ppm). 22p->16p
  C0G 0603 (Cext = 2·(CL-~4pF stray)); LCSC C162205 (Murata GRM1885C1H160JA01D,
  16pF C0G 50V 0603, live-verified).
- usb_jtag-2 (SN74LVC125A): removed the false "Ioff partial-power-down" docstring
  claim (TI SCAS290T has no such spec); powered-rail Hi-Z holds via the normal
  3-state OE pull-up. Series back-feed Rs documented as a DNP/layout reservation
  (forcing them overflows the A3 sheet; not fitted).
- io_misc-1 (user LED current): +3V3_USER_LED through 1k gave ~0.2mA (invisible)
  for the high-Vf (~3.1V) green/blue/white LEDs. Per-colour Rs: red keeps 1k
  (~1.3mA); green/blue/white -> 200R (C8218), ~1-3.5mA, within the 5mA rating.
- expansion-1 (SY6280 Cin): the load-switch IN pin had only 100n; added the
  datasheet-mandated 10uF (C15850) bulk at U1.IN, kept the 100n.

BOM VALUES now 0 unverified (white LED C2290 catalogued). Regression: board 33
+ golden match, all gates PASS, selftest 59, m1_rc, pytest 242 — green.

Co-Authored-By: Claude Opus 4.8 <noreply@anthropic.com>
Parts:
- C28005, C28006: value 22p -> 16p; LCSC C1653 -> C162205
Changed lines of the file:
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@@
 		(property
 			"Value"
-			"22p"
+			"16p"
 			(at 116.022 59.69 0)
 			(effects
@@
 		(property
 			"LCSC"
-			"C1653"
+			"C162205"
 			(at 111.76 58.42 0)
 			(effects
@@
 		(property
 			"Value"
-			"22p"
+			"16p"
 			(at 98.242 59.69 0)
 			(effects
@@
 		(property
 			"LCSC"
-			"C1653"
+			"C162205"
 			(at 93.98 58.42 0)
 			(effects

Commit message: fix: 3 CRITICAL electrical defects from the multi-agent audit (SW2 / LCD D1 / JTAG TDI-TDO)
A 69-agent electrical audit (35 per-subsystem + 7 cross-cutting, every finding
adversarially refuted) surfaced 3 board-dead CRITICAL defects that passed DRC/ERC/
netlist-equivalence. Each independently re-verified from the source artifacts before
fixing (per the "audits over-confirm; fixes can introduce bugs" rule):

1. SW2 (DSHP08) module DIP shorted all enables. Each DIP rocker bridges the two
   pads in the SAME COLUMN; the DSHP08 footprint numbers its bottom row 9..16
   (UNLIKE DSHP04's 8..5), so positions pair (n, n+8) — but the adapter re-used
   DSHP04's (n,17-n) diagonal, shorting +3V3_SC to itself on 1/3/5/7 and tying two
   enable nets on 2/4/6/8. All 7 module enables stuck off. FIX in the ADAPTER
   (+3V3_SC on top pins 1-8, BU_DIP nets on bottom pins 9-16) — NOT by renumbering
   the faithful EasyEDA footprint as the audit suggested (that would corrupt the
   real-part mapping; "never redraw parts"). DSHP08 is used only by SW2.
   + footprint-aware regression test (reads same-column pairs, asserts each rocker
     bridges +3V3_SC -> one unique BU_DIP enable) for SW2 and SW1.

2. LCD SY7201 boost catch diode D1 (SS34) reversed — cathode on LX, anode on the
   output, so the boost could never pump VLED+ (dead backlight). Device:D_Schottky
   is pin1=K/pin2=A; put K (D1.1) on the output, A (D1.2) on LX. The dossier was
   already correct; the netlist contradicted it.

3. usb_jtag CH347T TDI/TDO swapped — pin7=RTS0/MISO/TDO (bridge input), pin8=
   TXD0/MOSI/TDI (bridge output). DBG_FT_TDI sat on the input pin (buffer 2A had
   no driver) and DBG_FT_TDO on the output pin (collides with buffer 3Y when the
   bridge enables). Swapped to U1.8/U1.7; doc table corrected.

Verified: 148x137, DRC 0, netlist-equivalence PASS on all 35 sheets, every LAW gate
green, 68 subsystem tests pass.

Co-Authored-By: Claude Opus 4.8 <noreply@anthropic.com>
Connections:
- net DBG_FT_TDI: now also U28001.8 (TXD0/MOSI/TDI); no longer U28001.7 (RTS0/GPIO1/MISO/TDO)
- net DBG_FT_TDO: now also U28001.7 (RTS0/GPIO1/MISO/TDO); no longer U28001.8 (TXD0/MOSI/TDI)
Changed lines of the file:
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@@
+	(wire
+		(pts
+			(xy 179.07 67.31)
+			(xy 208.28 67.31)
+		)
+		(stroke
+			(width 0)
+			(type default)
+		)
+	)
+	(wire
+		(pts
+			(xy 304.8 80.01)
+			(xy 294.64 80.01)
+		)
+		(stroke
+			(width 0)
+			(type default)
+		)
+	)
 	(wire
 		(pts
@@
 	(wire
 		(pts
-			(xy 304.8 80.01)
-			(xy 294.64 80.01)
-		)
-		(stroke
-			(width 0)
-			(type default)
-		)
-	)
-	(wire
-		(pts
-			(xy 179.07 67.31)
-			(xy 208.28 67.31)
-		)
-		(stroke
-			(width 0)
-			(type default)
-		)
-	)
-	(wire
-		(pts
 			(xy 326.39 69.85)
 			(xy 354.33 69.85)
@@
 	)
 	(label
+		"DBG_FT_TDO"
+		(at 189.23 69.85 0)
+		(effects
+			(font
+				(size 1.27 1.27)
+			)
+			(justify left bottom)
+		)
+	)
+	(label
 		"DBG_FT_TDI"
-		(at 189.23 69.85 0)
-		(effects
-			(font
-				(size 1.27 1.27)
-			)
-			(justify left bottom)
-		)
-	)
-	(label
-		"DBG_FT_TDO"
 		(at 208.28 67.31 0)
 		(effects

Commit message: fix(silk): tighten 6 sheet titles overflowing the title-block cell (M6)
The audit flagged 6 sheet titles whose text overflowed the KiCad title-block
Title cell, crossing the border/zone rules (LAW 1). Root cause: the authored
Circuit titles were longer than the cell renders (the fit boundary is ~58 chars
of typical text; these were 55-73). Tightened all 6 at the source (display-only
strings, no info-loss of the essentials, cannot affect netlist/routing — board
.kicad_pcb byte-unchanged):
- board_services 73->47, pmod_expansion 65->45, mechanical 60->50,
  usb_jtag 59->38, usb_jtag_connector 58->42, power_som 55->37.
Render-confirmed: board_services + mechanical (the longest) now end well inside
the cell. The gallery description table (carrier/README.md) regenerated to match.
666 tests pass at HEAD; the 3 title-asserting tests (som_j1/j2/j3) are untouched.

Co-Authored-By: Claude Opus 4.8 <noreply@anthropic.com>
Other:
- title: USB-JTAG/UART debug bridge: CH347T, self-powered + isolated -> USB-JTAG/UART bridge: CH347T, isolated
Changed lines of the file:
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@@
 	(paper "A3")
 	(title_block
-		(title "USB-JTAG/UART debug bridge: CH347T, self-powered + isolated")
+		(title "USB-JTAG/UART bridge: CH347T, isolated")
 		(company "Zynq SoM Carrier")
 		(comment 1 "usb_jtag — generated by schgen (do not hand-edit)")
