File: carrier/schematic/usb_jtag_connector.kicad_sch (KiCad schematic)
At the start: 6 parts, among them J29001 TYPE-C-31-M-12, U29001 USBLC6-2SC6

Commit message: fix(silk): tighten 6 sheet titles overflowing the title-block cell (M6)
The audit flagged 6 sheet titles whose text overflowed the KiCad title-block
Title cell, crossing the border/zone rules (LAW 1). Root cause: the authored
Circuit titles were longer than the cell renders (the fit boundary is ~58 chars
of typical text; these were 55-73). Tightened all 6 at the source (display-only
strings, no info-loss of the essentials, cannot affect netlist/routing — board
.kicad_pcb byte-unchanged):
- board_services 73->47, pmod_expansion 65->45, mechanical 60->50,
  usb_jtag 59->38, usb_jtag_connector 58->42, power_som 55->37.
Render-confirmed: board_services + mechanical (the longest) now end well inside
the cell. The gallery description table (carrier/README.md) regenerated to match.
666 tests pass at HEAD; the 3 title-asserting tests (som_j1/j2/j3) are untouched.

Co-Authored-By: Claude Opus 4.8 <noreply@anthropic.com>
Other:
- title: USB-C UFP debug port -> CH347T (VBUS + protected USB pair) -> USB-C UFP debug port -> CH347T (protected)
Changed lines of the file:
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@@
 	(paper "A4")
 	(title_block
-		(title "USB-C UFP debug port -> CH347T (VBUS + protected USB pair)")
+		(title "USB-C UFP debug port -> CH347T (protected)")
 		(company "Zynq SoM Carrier")
 		(comment 1 "usb_jtag_connector — generated by schgen (do not hand-edit)")
