File: carrier/schematic/board_qwiic.kicad_sch (KiCad schematic)
At the start: 2 parts, among them J2001 ZX-SH1.0-4PWT, U2001 USBLC6-2SC6

Commit message: Publish current carrier and devkit placement release with fresh renders
Other:
- title: QWIIC / STEMMA-QT expansion connector + USBLC6 ESD array -> QWIIC / STEMMA-QT expansion connector +
Changed lines of the file:
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@@
 	(paper "A4")
 	(title_block
-		(title "QWIIC / STEMMA-QT expansion connector + USBLC6 ESD array")
+		(title "QWIIC / STEMMA-QT expansion connector +")
 		(company "Zynq SoM Carrier")
 		(comment 1 "board_qwiic — generated by schgen (do not hand-edit)")
+		(comment 2 "USBLC6 ESD array")
 	)
 	(wire
