File: carrier/schematic/som_decoupling.kicad_sch (KiCad schematic)
At the start: 18 parts

Commit message: Publish current carrier and devkit placement release with fresh renders
Other:
- title: SoM power-entry decoupling under the DF40 mezzanine -> SoM power-entry decoupling under the
Changed lines of the file:
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@@
 	(paper "A3")
 	(title_block
-		(title "SoM power-entry decoupling under the DF40 mezzanine")
+		(title "SoM power-entry decoupling under the")
 		(company "Zynq SoM Carrier")
 		(comment 1 "som_decoupling — generated by schgen (do not hand-edit)")
+		(comment 2 "DF40 mezzanine")
 	)
 	(symbol
