File: devkit_mini/schematic/mechanical.kicad_sch (KiCad schematic)
At the start: 4 parts

Commit message: Publish current carrier and devkit placement release with fresh renders
Other:
- company: Zynq SoM Carrier -> Zynq SoM Devkit Mini
- title: Mechanical: M3 mounts + chassis-GND bond (fiducials are PCB-only, emitted by the placer) -> Mechanical: M3 mounts + chassis-GND
Changed lines of the file:
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@@
 	(paper "A4")
 	(title_block
-		(title
-			"Mechanical: M3 mounts + chassis-GND bond (fiducials are PCB-only, emitted by the placer)"
-		)
-		(company "Zynq SoM Carrier")
+		(title "Mechanical: M3 mounts + chassis-GND")
+		(company "Zynq SoM Devkit Mini")
 		(comment 1 "mechanical — generated by schgen (do not hand-edit)")
+		(comment 2 "bond (fiducials are PCB-only, emitted by the placer)")
 	)
 	(wire
