File: devkit_mini/schematic/power_mon.kicad_sch (KiCad schematic)
At the start: 10 parts, among them U5001 INA3221AIRGVR, U5002 INA3221AIRGVR

Commit message: feat(native): migrate schematic pipeline and fix devkit electrical coverage
Parts:
- added TP5001: +3V3_SC, TestPoint:TestPoint_Pad_D1.5mm, symbol Connector:TestPoint
- added TP5002: STM32_I2C2_SCL, TestPoint:TestPoint_Pad_D1.5mm, symbol Connector:TestPoint
- added TP5003: STM32_I2C2_SDA, TestPoint:TestPoint_Pad_D1.5mm, symbol Connector:TestPoint
Connections:
- net +3V3_SC: now also TP5001.1
- net STM32_I2C2_SCL: now also TP5002.1
- net STM32_I2C2_SDA: now also TP5003.1
Other:
- moved on the sheet: C5001, C5002, C5003, R5001, RS5001, RS5002, RS5003, RS5004, U5001, U5002

Commit message: Publish current carrier and devkit placement release with fresh renders
Other:
- company: Zynq SoM Carrier -> Zynq SoM Devkit Mini
- title: Rail telemetry: 2x INA3221 + shunts (I2C 0x40/41) -> Rail telemetry: 2x INA3221 + shunts
Changed lines of the file:
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@@
 	(paper "A4")
 	(title_block
-		(title "Rail telemetry: 2x INA3221 + shunts (I2C 0x40/41)")
-		(company "Zynq SoM Carrier")
+		(title "Rail telemetry: 2x INA3221 + shunts")
+		(company "Zynq SoM Devkit Mini")
 		(comment 1 "power_mon — generated by schgen (do not hand-edit)")
+		(comment 2 "(I2C 0x40/41)")
 	)
 	(wire
