File: devkit_mini/schematic/som_j3.kicad_sch (KiCad schematic)
At the start: 1 part, among them J10003 DF40C-100DP-0.4V(51)

Commit message: Publish current carrier and devkit placement release with fresh renders
Other:
- company: Zynq SoM Carrier -> Zynq SoM Devkit Mini
- title: SoM J3: FPGA bank 33/34/35 IO + VCCO rails -> SoM J3: FPGA bank 33/34/35 IO + VCCO
Changed lines of the file:
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@@
 	(paper "A4")
 	(title_block
-		(title "SoM J3: FPGA bank 33/34/35 IO + VCCO rails")
-		(company "Zynq SoM Carrier")
+		(title "SoM J3: FPGA bank 33/34/35 IO + VCCO")
+		(company "Zynq SoM Devkit Mini")
 		(comment 1 "som_j3 — generated by schgen (do not hand-edit)")
+		(comment 2 "rails")
 	)
 	(wire
