File: devkit_mini/schematic/uart_bridge.kicad_sch (KiCad schematic)
At the start: 10 parts, among them U11001 CP2102N-A02

Commit message: Publish current carrier and devkit placement release with fresh renders
Other:
- company: Zynq SoM Carrier -> Zynq SoM Devkit Mini
Changed lines of the file:
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@@
 	(title_block
 		(title "UART bridge: CP2102N USB-UART")
-		(company "Zynq SoM Carrier")
+		(company "Zynq SoM Devkit Mini")
 		(comment 1 "uart_bridge — generated by schgen (do not hand-edit)")
 	)
