File: devkit_mini/schematic/usb_uart_connector.kicad_sch (KiCad schematic)
At the start: 5 parts, among them J12001 TYPE-C-31-M-12, U12001 USBLC6-2SC6

Commit message: Publish current carrier and devkit placement release with fresh renders
Other:
- company: Zynq SoM Carrier -> Zynq SoM Devkit Mini
Changed lines of the file:
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@@
 	(title_block
 		(title "USB-C UFP console port -> CP2102N")
-		(company "Zynq SoM Carrier")
+		(company "Zynq SoM Devkit Mini")
 		(comment 1 "usb_uart_connector — generated by schgen (do not hand-edit)")
 	)
